File: pcb/PCB_V1/PCB_V1.kicad_sch (KiCad schematic)
At the start: 13 parts, among them U101 TPS54202DDCR

Commit message: Add RTC, microSD and protected sensor interfaces to PCB schematic
Other:
- note added: "Ревизия 0.2: RTC, microSD и датчики добавлены; силовая часть ещё не разработана."
- note removed: "Черновик 0.1: входная защита и силовые нагрузки будут добавлены отдельно."

Commit message: pcb: add fan pump and PTC output stages
Other:
- added sheet Outputs (Outputs.kicad_sch)
- note added: "Ревизия 0.3: выходы FAN/PUMP/PTC добавлены. Входная защита и LED-драйверы ещё не разработаны."
- note removed: "Ревизия 0.2: RTC, microSD и датчики добавлены; силовая часть ещё не разработана."
Changed lines of the file:
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@@
 		(title "01 - Logic power / 12 V to 3.3 V")
 		(date "2026-09-26")
-		(rev "0.2-DRAFT")
+		(rev "0.3-DRAFT")
 		(company "GrowBox controller")
-		(comment 1 "Logic first; power loads not yet implemented")
+		(comment 1 "Draft: input protection and LED drivers pending")
 	)
 	(text "Vout = 0.596 x (1 + 100k/22k) = 3.305 V\n500 kHz; L = 10 uH; ripple ~0.48 A at 12 V (nominal).\n2 A IC rating; target logic budget <= 1 A continuous.\nL101: footprint candidate; exact MPN / DCR / Isat to verify.\nC104/C105: verify effective capacitance under DC bias.\nC106 is NOT fitted until loop/transient verification."
@@
 		)
 	)
-	(text "Ревизия 0.2: RTC, microSD и датчики добавлены; силовая часть ещё не разработана."
+	(text "Ревизия 0.3: выходы FAN/PUMP/PTC добавлены. Входная защита и LED-драйверы ещё не разработаны."
 		(exclude_from_sim no)
 		(at 20.32 25.4 0)
@@
 		)
 	)
-	(label "+12V_PROTECTED"
-		(at 25.4 170.18 0)
-		(effects
-			(font
-				(size 1 1)
-			)
-			(justify left bottom)
-		)
-	)
 	(label "BUCK_FB"
 		(at 243.84 85.09 0)
@@
 	(label "BUCK_FB"
 		(at 111.76 66.04 0)
-		(effects
-			(font
-				(size 1 1)
-			)
-			(justify left bottom)
-		)
-	)
-	(label "+12V_PROTECTED"
-		(at 25.4 50.8 0)
 		(effects
 			(font
@@
 		)
 	)
+	(global_label "+12V_PROTECTED"
+		(shape bidirectional)
+		(at 25.4 170.18 0)
+		(effects
+			(font
+				(size 1 1)
+			)
+			(justify left bottom)
+		)
+		(property "Intersheetrefs" "${INTERSHEET_REFS}"
+			(at 25.4 170.18 0)
+			(hide yes)
+			(show_name no)
+			(do_not_autoplace no)
+			(effects
+				(font
+					(size 1.27 1.27)
+				)
+			)
+		)
+	)
 	(global_label "GND"
 		(shape bidirectional)
@@
 		(property "Intersheetrefs" "${INTERSHEET_REFS}"
 			(at 149.86 170.18 0)
+			(hide yes)
+			(show_name no)
+			(do_not_autoplace no)
+			(effects
+				(font
+					(size 1.27 1.27)
+				)
+			)
+		)
+	)
+	(global_label "+12V_PROTECTED"
+		(shape bidirectional)
+		(at 25.4 50.8 0)
+		(effects
+			(font
+				(size 1 1)
+			)
+			(justify left bottom)
+		)
+		(property "Intersheetrefs" "${INTERSHEET_REFS}"
+			(at 25.4 50.8 0)
 			(hide yes)
 			(show_name no)
@@
 	)
 	(sheet
-		(at 200.66 132.08)
-		(size 66.04 22.86)
+		(at 200.66 151.13)
+		(size 66.04 7.62)
 		(exclude_from_sim no)
 		(in_bom yes)
@@
 			(color 0 0 0 0)
 		)
+		(property "Sheetname" "Outputs"
+			(at 200.66 150.495 0)
+			(show_name no)
+			(do_not_autoplace no)
+			(effects
+				(font
+					(size 1.27 1.27)
+				)
+				(justify left bottom)
+			)
+		)
+		(property "Sheetfile" "Outputs.kicad_sch"
+			(at 200.66 159.385 0)
+			(show_name no)
+			(do_not_autoplace no)
+			(effects
+				(font
+					(size 1.27 1.27)
+				)
+				(justify left top)
+			)
+		)
+		(instances
+			(project "PCB_V1"
+				(path "/7c30e6d8-4e60-4647-b4d3-d05e639d6467"
+					(page "4")
+				)
+			)
+		)
+	)
+	(sheet
+		(at 200.66 132.08)
+		(size 66.04 7.62)
+		(exclude_from_sim no)
+		(in_bom yes)
+		(on_board yes)
+		(dnp no)
+		(fields_autoplaced yes)
+		(stroke
+			(width 0.254)
+			(type solid)
+		)
+		(fill
+			(color 0 0 0 0)
+		)
 		(property "Sheetname" "MCU / ESP32"
 			(at 200.66 131.445 0)
@@
 		)
 		(property "Sheetfile" "MCU.kicad_sch"
-			(at 200.66 155.575 0)
-			(show_name no)
-			(do_not_autoplace no)
+			(at 200.66 140.335 0)
+			(show_name no)
+			(do_not_autoplace no)
