File: pcb/PCB_V1/PCB_V1.kicad_sch (KiCad schematic)
At the start: 13 parts, among them U101 TPS54202DDCR

Commit message: pcb: use low-leakage RTC supply diode for revision 0.21
Other:
- note added: "0.21 DRAFT: cost-down (PCF8563 RTC, DPAK/TO-277A boost parts, 7 mm inductors); routing and prototype validation pending."
- note removed: "0.20 DRAFT: cost-down (PCF8563 RTC, DPAK/TO-277A boost parts, 7 mm inductors); routing and prototype validation pending."
Changed lines of the file:
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@@
 	(title_block
 		(title "01 - Logic power / 12 V aux to 3.3 V")
-		(date "2026-09-29")
-		(rev "0.20-DRAFT")
+		(date "2026-09-30")
+		(rev "0.21-DRAFT")
 		(company "GrowBox controller")
 		(comment 1 "Simplified prototype; unrouted; hardware qualification pending")
@@
 		)
 	)
-	(text "0.20 DRAFT: cost-down (PCF8563 RTC, DPAK/TO-277A boost parts, 7 mm inductors); routing and prototype validation pending."
+	(text "0.21 DRAFT: cost-down (PCF8563 RTC, DPAK/TO-277A boost parts, 7 mm inductors); routing and prototype validation pending."
 		(exclude_from_sim no)
 		(at 20.32 25.4 0)
