File: pcb/PCB_V1/PCB_V1.kicad_sch (KiCad schematic)
At the start: 13 parts, among them U101 TPS54202DDCR

Commit message: pcb: revision 0.22 routing preparation
- Stack confirmed by the user: 1.6 mm, 1 oz outer, 0.5 oz inner.
- LED output MLCCs: Murata GRM32EC72A106KE05L (X7S, 50k in stock) instead
  of TDK; DC-bias digitised from Murata data (2.60 uF at 49 V, model
  2.55 uF), CH1 bank 6.44 uF effective.
- microSD: HRO TF-01A (push-push, C91145) on a project footprint from the
  HRO drawing, checked against the LCSC land; SD passives re-placed.
- TP301 on the PCF8563 CLKOUT for crystal trimming.
- Kelvin net ties NT711/NT712/NT721/NT722 at the LED-driver shunts
  (LED*_CS_K, LED*_FB_K); net ties are excluded from the BOM export.
- analyze_copper.py: IPC-2221 copper screen for the confirmed stack
  (main 24 V path needs pours on both outer layers, via counts).
- L711 and XT60PW-M re-checked and kept; reports v22 and ROUTING_PREP.md.
  USD 30.04 per board (28.42 for five), ERC 0, DRC 0.

Co-Authored-By: Claude Opus 5.5 <noreply@anthropic.com>
Other:
- note added: "0.22 DRAFT: pre-routing (Murata LED output MLCCs, HRO TF-01A microSD, CLKOUT test pad; stack 1.6 mm, 1 oz outer / 0.5 oz inner); routing and prototype validation pending."
- note removed: "0.21 DRAFT: cost-down (PCF8563 RTC, DPAK/TO-277A boost parts, 7 mm inductors); routing and prototype validation pending."
Changed lines of the file:
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@@
 		(title "01 - Logic power / 12 V aux to 3.3 V")
 		(date "2026-09-30")
-		(rev "0.21-DRAFT")
+		(rev "0.22-DRAFT")
 		(company "GrowBox controller")
 		(comment 1 "Simplified prototype; unrouted; hardware qualification pending")
@@
 		)
 	)
-	(text "0.21 DRAFT: cost-down (PCF8563 RTC, DPAK/TO-277A boost parts, 7 mm inductors); routing and prototype validation pending."
+	(text "0.22 DRAFT: pre-routing (Murata LED output MLCCs, HRO TF-01A microSD, CLKOUT test pad; stack 1.6 mm, 1 oz outer / 0.5 oz inner); routing and prototype validation pending."
 		(exclude_from_sim no)
 		(at 20.32 25.4 0)
