File: pcb/PCB_V1/Peripherals.kicad_sch (KiCad schematic)
At the start: 32 parts, among them J301 SHT4x / XH 2.50, J302 FLOAT / WAGO 2601, J401 Molex 104031-0811, U301 DS3231SN#

Commit message: pcb: adopt DS3231MZ RTC and compact TI strip MOSFETs
Parts:
- U301: value DS3231SN# -> DS3231MZ+TRL; footprint Package_SO:SOIC-16W_7.5x10.3mm_P1.27mm -> Package_SO:SOIC-8_3.9x4.9mm_P1.27mm; symbol GrowBox:DS3231SN -> GrowBox:DS3231MZ
Connections:
- net GND: no longer U301.10 (GND_NC), U301.11 (GND_NC), U301.12 (GND_NC), U301.13 (GND), U301.6 (GND_NC), U301.7 (GND_NC), U301.8 (GND_NC), U301.9 (GND_NC)
- net I2C_SCL: now also U301.8 (SCL); no longer U301.16 (SCL)
- net I2C_SDA: now also U301.7 (SDA); no longer U301.15 (SDA)
- net RTC_VBAT: now also U301.6 (VBAT); no longer U301.14 (VBAT)
Other:
- note added: "0.11 DRAFT — схема для проверки; разводка и испытания ещё не выполнены."
- note added: "01 DS3231MZ / I2C 0x68 / CR2032"
- note added: "SOIC-8: VCC=2, GND=5, VBAT=6, SDA=7, SCL=8. 32kHz, INT/SQW, RST не используются. CR2032 -> VBAT; без зарядки. RTC-код совместим."
- note removed: "0.2 DRAFT — схема для проверки; разводка и испытания ещё не выполнены."
- note removed: "01 DS3231SN / I2C 0x68 / CR2032"
- note removed: "NC 5..12 соединены с GND — требование datasheet. 32kHz, INT/SQW, RST не используются. Батарейка питает только VBAT; цепи зарядки нет."
Changed lines of the file:
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@@
 		(title "03 - RTC / microSD / external sensors")
 		(date "2026-09-26")
-		(rev "0.2-DRAFT")
+		(rev "0.11-DRAFT")
 		(company "GrowBox controller")
 		(comment 1 "Draft: input protection and LED drivers pending")
@@
 		)
 	)
-	(text "01  DS3231SN / I2C 0x68 / CR2032"
+	(text "01  DS3231MZ / I2C 0x68 / CR2032"
 		(exclude_from_sim no)
 		(at 20.32 35.56 0)
@@
 		)
 	)
-	(text "NC 5..12 соединены с GND — требование datasheet.\n32kHz, INT/SQW, RST не используются.\nБатарейка питает только VBAT; цепи зарядки нет."
+	(text "SOIC-8: VCC=2, GND=5, VBAT=6, SDA=7, SCL=8.\n32kHz, INT/SQW, RST не используются.\nCR2032 -> VBAT; без зарядки. RTC-код совместим."
 		(exclude_from_sim no)
 		(at 20.32 101.6 0)
@@
 		)
 	)
-	(text "0.2 DRAFT — схема для проверки; разводка и испытания ещё не выполнены."
+	(text "0.11 DRAFT — схема для проверки; разводка и испытания ещё не выполнены."
 		(exclude_from_sim no)
 		(at 20.32 24.13 0)
@@
 	)
 	(symbol
-		(lib_id "GrowBox:DS3231SN")
+		(lib_id "GrowBox:DS3231MZ")
 		(at 78.74 73.66 0)
 		(unit 1)
@@
 			)
 		)
-		(property "Value" "DS3231SN#"
+		(property "Value" "DS3231MZ+TRL"
 			(at 66.04 54.61 0)
 			(show_name no)
@@
 			)
 		)
-		(property "Footprint" "Package_SO:SOIC-16W_7.5x10.3mm_P1.27mm"
+		(property "Footprint" "Package_SO:SOIC-8_3.9x4.9mm_P1.27mm"
 			(at 78.74 73.66 0)
 			(hide yes)
@@
 			)
 		)
-		(property "Datasheet" "https://www.analog.com/media/en/technical-documentation/data-sheets/DS3231.pdf"
+		(property "Datasheet" "https://www.analog.com/media/en/technical-documentation/data-sheets/DS3231M.pdf"
 			(at 78.74 73.66 0)
 			(hide yes)
@@
 				)
 			)
-		)
-		(pin "1"
-		)
-		(pin "2"
-		)
-		(pin "3"
-		)
-		(pin "4"
-		)
-		(pin "13"
-		)
-		(pin "14"
-		)
-		(pin "15"
-		)
-		(pin "16"
-		)
-		(pin "5"
-		)
-		(pin "6"
-		)
-		(pin "7"
-		)
-		(pin "8"
-		)
-		(pin "9"
-		)
-		(pin "10"
-		)
-		(pin "11"
-		)
-		(pin "12"
 		)
 		(instances
@@
 			)
 		)
-	)
+		(pin "1"
+		)
+		(pin "2"
+		)
+		(pin "3"
+		)
+		(pin "4"
+		)
+		(pin "5"
+		)
+		(pin "6"
+		)
+		(pin "7"
+		)
+		(pin "8"
+		)
+	)
