File: pcb/PCB_V1/Peripherals.kicad_sch (KiCad schematic)
At the start: 32 parts, among them J301 SHT4x / XH 2.50, J302 FLOAT / 3.5 mm, J401 Molex 104031-0811, U301 PCF8563T/5, Y301 32.768k 12.5pF

Commit message: pcb: revision 0.22 routing preparation
- Stack confirmed by the user: 1.6 mm, 1 oz outer, 0.5 oz inner.
- LED output MLCCs: Murata GRM32EC72A106KE05L (X7S, 50k in stock) instead
  of TDK; DC-bias digitised from Murata data (2.60 uF at 49 V, model
  2.55 uF), CH1 bank 6.44 uF effective.
- microSD: HRO TF-01A (push-push, C91145) on a project footprint from the
  HRO drawing, checked against the LCSC land; SD passives re-placed.
- TP301 on the PCF8563 CLKOUT for crystal trimming.
- Kelvin net ties NT711/NT712/NT721/NT722 at the LED-driver shunts
  (LED*_CS_K, LED*_FB_K); net ties are excluded from the BOM export.
- analyze_copper.py: IPC-2221 copper screen for the confirmed stack
  (main 24 V path needs pours on both outer layers, via counts).
- L711 and XT60PW-M re-checked and kept; reports v22 and ROUTING_PREP.md.
  USD 30.04 per board (28.42 for five), ERC 0, DRC 0.

Co-Authored-By: Claude Opus 5.5 <noreply@anthropic.com>
Parts:
- added TP301: CLKOUT, TestPoint:TestPoint_Pad_D1.0mm, symbol Connector:TestPoint
- J401: value Molex 104031-0811 -> HRO TF-01A; footprint Connector_Card:microSD_HC_Molex_104031-0811 -> GrowBox:microSD_HRO_TF-01A; symbol Connector:Micro_SD_Card_Det2 -> Connector:Micro_SD_Card_Det1; LCSC C585350 -> C91145; MPN 1040310811 -> TF-01A; Manufacturer Molex -> Korean Hroparts Elec
Connections:
- net RTC_CLKOUT: now reaches U301.7 (CLKO)
- net RTC_CLKOUT: now also TP301.1
- no-connect marks 5 -> 3
Other:
- note added: "0.22 DRAFT — схема для проверки; разводка и испытания ещё не выполнены."
- note added: "R401..403 у ESP32; R404 у карты.\nJ401 HRO TF-01A (push-push); DET 9 не используется; SH -> GND.\nНачальная частота SPI 4 MHz; проверка фронтов до повышения."
- note added: "SOIC-8: OSCI=1, OSCO=2, VSS=4, SDA=5, SCL=6, VDD=8; INT unused; CLKOUT -> TP301 (firmware turns it off unless RTC_CLKOUT_TRIM).\nY301 FC-135 CL 12.5 pF: OSCO has 25 pF inside (15..35), OSCI needs ~25 pF -> C304 18p + pin/stray.\nTrim C304 on the prototype by the 32.768 kHz CLKOUT frequency after power-on (NXP method 1).\nD303 BAV170: +3V3 or CR2032 via R307 -> RTC_VDD (C301).\nVerify VF/leakage a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"
- note removed: "0.21 DRAFT — схема для проверки; разводка и испытания ещё не выполнены."
- note removed: "R401..403 у ESP32; R404 у карты. DET 9/10 не используется; SH -> GND. Начальная частота SPI 4 MHz; проверка фронтов до повышения."
- note removed: "SOIC-8: OSCI=1, OSCO=2, VSS=4, SDA=5, SCL=6, VDD=8; INT, CLKOUT unused (firmware turns CLKOUT off). Y301 FC-135 CL 12.5 pF: OSCO has 25 pF inside (15..35), OSCI needs ~25 pF -> C304 18p + pin/stray. Trim C304 on the prototype by the 32.768 kHz CLKOUT frequency after power-on (NXP method 1). D303 BAV170: +3V3 or CR2032 via R307 -> RTC_VDD (C301). Verify VF/leakage at temperature. R307 is not quali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"
Changed lines of the file:
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@@
 		(title "03 - RTC / microSD / external sensors")
 		(date "2026-09-30")
-		(rev "0.21-DRAFT")
+		(rev "0.22-DRAFT")
 		(company "GrowBox controller")
 		(comment 1 "Simplified prototype; unrouted; hardware qualification pending")
@@
 		)
 	)
-	(text "R401..403 у ESP32; R404 у карты.\nDET 9/10 не используется; SH -> GND.\nНачальная частота SPI 4 MHz; проверка фронтов до повышения."
+	(text "R401..403 у ESP32; R404 у карты.\\nJ401 HRO TF-01A (push-push); DET 9 не используется; SH -> GND.\\nНачальная частота SPI 4 MHz; проверка фронтов до повышения."
 		(exclude_from_sim no)
 		(at 218.44 114.3 0)
@@
 		)
 	)
-	(text "SOIC-8: OSCI=1, OSCO=2, VSS=4, SDA=5, SCL=6, VDD=8; INT, CLKOUT unused (firmware turns CLKOUT off).\nY301 FC-135 CL 12.5 pF: OSCO has 25 pF inside (15..35), OSCI needs ~25 pF -> C304 18p + pin/stray.\nTrim C304 on the prototype by the 32.768 kHz CLKOUT frequency after power-on (NXP method 1).\nD303 BAV170: +3V3 or CR2032 via R307 -> RTC_VDD (C301).\nVerify VF/leakage at temperature. R307 is not qualified fault/charging protection."
+	(text "SOIC-8: OSCI=1, OSCO=2, VSS=4, SDA=5, SCL=6, VDD=8; INT unused; CLKOUT -> TP301 (firmware turns it off unless RTC_CLKOUT_TRIM).\\nY301 FC-135 CL 12.5 pF: OSCO has 25 pF inside (15..35), OSCI needs ~25 pF -> C304 18p + pin/stray.\\nTrim C304 on the prototype by the 32.768 kHz CLKOUT frequency after power-on (NXP method 1).\\nD303 BAV170: +3V3 or CR2032 via R307 -> RTC_VDD (C301).\\nVerify VF/leakage at temperature. R307 is not qualified fault/charging protection."
 		(exclude_from_sim no)
 		(at 20.32 101.6 0)
@@
 		)
 	)
-	(text "0.21 DRAFT — схема для проверки; разводка и испытания ещё не выполнены."
+	(text "0.22 DRAFT — схема для проверки; разводка и испытания ещё не выполнены."
 		(exclude_from_sim no)
 		(at 20.32 24.13 0)
@@
 		(at 347.98 86.36)
 	)
-	(no_connect
-		(at 347.98 83.82)
-	)
 	(wire
 		(pts
@@
 	)
 	(symbol
-		(lib_id "Connector:Micro_SD_Card_Det2")
+		(lib_id "Connector:Micro_SD_Card_Det1")
 		(at 370.84 73.66 0)
 		(unit 1)
@@
 			)
 		)
-		(property "Value" "Molex 104031-0811"
+		(property "Value" "HRO TF-01A"
 			(at 347.98 52.07 0)
 			(show_name no)
@@
 			)
 		)
-		(property "Footprint" "Connector_Card:microSD_HC_Molex_104031-0811"
+		(property "Footprint" "GrowBox:microSD_HRO_TF-01A"
 			(at 370.84 73.66 0)
 			(hide yes)
@@
 			)
 		)
-		(property "Datasheet" "https://www.molex.com/content/dam/molex/molex-dot-com/products/automated/en-us/salesdrawingpdf/104/104031/1040310811_sd.pdf"
+		(property "Datasheet" "https://www.lcsc.com/product-detail/C91145.html"
 			(at 370.84 73.66 0)
 			(hide yes)
@@
 			)
 		)
-		(property "Manufacturer" "Molex"
+		(property "Manufacturer" "Korean Hroparts Elec"
 			(at 370.84 73.66 0)
 			(hide yes)
@@
 			)
 		)
-		(property "MPN" "1040310811"
+		(property "MPN" "TF-01A"
 			(at 370.84 73.66 0)
 			(hide yes)
@@
 			)
 		)
-		(property "LCSC" "C585350"
+		(property "LCSC" "C91145"
 			(at 370.84 73.66 0)
 			(hide yes)
@@
 		)
 	)
-	(no_connect
-		(at 88.9 76.2)
-	)
 	(wire
 		(pts
@@
 		)
 	)
+	(wire
+		(pts
+			(xy 88.9 76.2) (xy 99.06 76.2)
+		)
+		(stroke
+			(width 0)
+			(type default)
+		)
+	)
+	(label "RTC_CLKOUT"
+		(at 91.44 76.2 0)
+		(effects
+			(font
+				(size 1.0 1.0)
+			)
+			(justify left bottom)
+		)
+	)
+	(symbol
+		(lib_id "Connector:TestPoint")
+		(at 99.06 76.2 0)
+		(unit 1)
+		(exclude_from_sim no)
+		(in_bom yes)
+		(on_board yes)
+		(dnp no)
+		(property "Reference" "TP301"
+			(at 102.87 74.93 0)
+			(effects
+				(font
+					(size 1 1)
+				)
+				(justify left)
+			)
+		)
+		(property "Value" "CLKOUT"
+			(at 102.87 77.47 0)
+			(effects
+				(font
+					(size 1 1)
+				)
+				(justify left)
+			)
+		)
+		(property "Footprint" "TestPoint:TestPoint_Pad_D1.0mm"
+			(at 99.06 76.2 0)
+			(effects
+				(font
+					(size 1 1)
+				)
+				(hide yes)
+				(justify left)
+			)
+		)
+		(property "Datasheet" ""
+			(at 99.06 76.2 0)
+			(effects
+				(font
+					(size 1 1)
+				)
+				(hide yes)
+				(justify left)
+			)
+		)
+		(property "Description" "PCF8563 CLKOUT (open drain): 32.768 kHz for C304 trimming, add a pull-up while measuring"
+			(at 99.06 76.2 0)
+			(effects
+				(font
+					(size 1 1)
+				)
+				(hide yes)
+				(justify left)
+			)
+		)
+		(pin "1"
+		)
+		(instances
+			(project "PCB_V1"
+				(path "/7c30e6d8-4e60-4647-b4d3-d05e639d6467/6b08d5d1-f5dd-51d1-a612-b10717fdf3b0/bcf5e9ab-329b-5115-ad03-190ffcafae19"
+					(reference "TP301")
+					(unit 1)
+				)
+			)
+		)
+	)
