File: pcb/PCB_V1/Heater.kicad_sch (KiCad schematic)
At the start: 8 parts, among them J601 PTC + / switched -, Q601 NTMFS5C628NLT1G, U601 UCC27524ADR

Commit message: pcb: add protected input and independent LED boost drivers
Connections:
- net +12V_PROTECTED renamed +12V_LOADS
Changed lines of the file:
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@@
 		(title "05 - PTC heater switch")
 		(date "2026-09-26")
-		(rev "0.3-DRAFT")
+		(rev "0.4-DRAFT")
 		(company "GrowBox controller")
 		(comment 1 "Draft: input protection and LED drivers pending")
@@
 		)
 	)
-	(global_label "+12V_PROTECTED"
+	(global_label "+12V_LOADS"
 		(shape bidirectional)
 		(at 30.48 92.71 0)
@@
 		)
 	)
-	(global_label "+12V_PROTECTED"
+	(global_label "+12V_LOADS"
 		(shape bidirectional)
 		(at 88.9 48.26 0)
@@
 		)
 	)
-	(global_label "+12V_PROTECTED"
+	(global_label "+12V_LOADS"
 		(shape bidirectional)
 		(at 30.48 57.15 0)
@@
 		)
 	)
-	(global_label "+12V_PROTECTED"
+	(global_label "+12V_LOADS"
 		(shape bidirectional)
 		(at 228.6 48.26 0)

Commit message: pcb: select ideal-diode input protection and regulate heater gate supply
Parts:
- added C603: 2.2u / 50V X7R, Capacitor_SMD:C_0805_2012Metric, symbol Device:C
- added C604: 10u / 16V X7R, Capacitor_SMD:C_0805_2012Metric, symbol Device:C
- added U602: TPS70950DBVR, Package_TO_SOT_SMD:SOT-23-5, symbol GrowBox:TPS70950
- C602: value 1u / 25V -> 2.2u / 25V X7R
- Q601: LCSC (none) -> C145537; MPN (none) -> NTMFS5C628NLT1G; Manufacturer (none) -> onsemi
Connections:
- net +12V_LOADS: now also C603.1, U602.1 (VIN); no longer C601.1, C602.1, U601.6 (V_{DD})
- net +3V3: now also U602.3 (EN)
- net GND: now also C603.2, C604.2, U602.2 (GND)
- new net +5V_GATE: C601.1, C602.1, C604.1, U601.6 (V_{DD}), U602.5 (VOUT)
- no-connect marks 1 -> 2
Other:
- note added: "0.13 DRAFT: power/thermal limits remain subject to prototype validation."
- note added: "EN = +3V3; do not connect EN to 12 V. TPS70950 has reverse-current protection. C604: >=2.2 uF effective at 5 V; ESR <=0.2 ohm. C602 >=1 uF effective, directly at driver. C603/C604 directly at LDO. Gate supply budget <=5 mA; PTC ON/OFF <=1 Hz."
- note added: "LOCAL 5 V GATE SUPPLY"
- note added: "Q601: G=4, S=1/2/3, D=5; SO-8FL exposed drain is not GND. RDS(on) max 3.3 mOhm at VGS=4.5 V, Tj=25 C. Conduction ~0.229 W at 8.33 A / ~0.303 W at 9.58 A. Hot resistance and switching overshoot still require thermal/scope checks."
- note added: "U601: ENA=3.3 V, INA=HEATER_EN. Channel B disabled. VDD from local +5V_GATE. C601/C602 close to VDD/GND. Short OUTA-G-S-GND loop. MCU R210=10k pull-down; R602 discharges the gate when unpowered. Verify 5 V startup/droop: SOIC start threshold up to 4.65 V; never power directly from 12 V."
- note removed: "0.3 DRAFT: номинальный ток не является подтверждённым допустимым током платы."
- note removed: "Q601: G=4, S=1/2/3, D=5; SO-8FL, площадка D не GND. Rds(on) max 2.4mOhm при Vgs=10V, Tj=25C. Проводимость: ~0.167W при 8.33A; ~0.220W при 9.58A. При нагреве Rds возрастает; проверить тепло и выбросы на реальной PCB."
- note removed: "U601: ENA от 3.3V, INA=HEATER_EN. Канал B отключён. C601/C602 вплотную к VDD/GND. Короткий контур OUTA-G-S-GND. R210 на MCU = 10k pull-down; R602 удерживает затвор без питания. Питание драйвера 4.5..18V; входная OVP должна обеспечить этот предел."
