File: pcb/PCB_V1/Heater.kicad_sch (KiCad schematic)
At the start: 11 parts, among them J601 PTC + / switched -, Q601 NTMFS5C628NLT1G, U601 UCC27524ADR, U602 TPS70950DBVR

Commit message: pcb: move board to 24 V input with 12 V aux buck and merged LED bar channel
Revision 0.14 of PCB_V1 (see pcb/PCB_V1/REDESIGN_24V.md):
- 24 V input on keyed XT60PW-M (pin 1 GND, pin 2 +24V); LM74700, input
  MOSFET and F901 removed; SMBJ26CA TVS; 220 uF/50 V bulk
- ATM mini-blade fuses in XF-508P-B-B holders: F902 10 A loads, F903 7.5 A LED
- new LMR16020 24 V -> 12 V aux buck (500 kHz) feeding PC fans, the
  UCC27524A heater gate driver and the TPS54202 3.3 V buck; TPS70950 removed
- heater and pump on 24 V: SMBJ30A drain TVS, AO3422 + SS36 pump stage
- LED CH1 panel keeps SRP1770TA/0.027 R/1k, switch now CSD19534Q5A;
  CH2 drives both identical bars in parallel (J721 || J731, 0.40 R);
  third AL8853 channel removed
- TS-1187A buttons, DORABO/KANGNEX terminals
- project library: LMR16020 and CSD19534Q5A symbols, TI DQJ and XF-508P
  footprints
- verify_netlist.py / verify_board.py / analyze_*.py updated for 24 V;
  new sync_board.py updates the unrouted staging board from the netlist
- ERC 0/0; netlist, board and sizing checks pass; DRC only the 12 known
  ESP32 drill sizes plus unrouted connections; 163 components

Co-Authored-By: Claude Opus 5.5 <noreply@anthropic.com>
Parts:
- removed C603: 2.2u / 50V X7R, Capacitor_SMD:C_0805_2012Metric, symbol Device:C
- removed C604: 10u / 16V X7R, Capacitor_SMD:C_0805_2012Metric, symbol Device:C
- removed U602: TPS70950DBVR, Package_TO_SOT_SMD:SOT-23-5, symbol GrowBox:TPS70950
- D601: value SMBJ18A-E3/52 -> SMBJ30A-E3/52; LCSC (none) -> C1973126; MPN (none) -> SMBJ30A-E3/52; Manufacturer (none) -> Vishay
- J601: value PTC + / switched - -> PTC + / switched - (3.5 mm); footprint TerminalBlock_WAGO:TerminalBlock_WAGO_2601-1102_1x02_P3.50mm_Horizontal -> TerminalBlock_Phoenix:TerminalBlock_Phoenix_PT-1,5-2-3.5-H_1x02_P3.50mm_Horizontal; LCSC (none) -> C466970; MPN (none) -> DB125-3.5-2P-GN-S; Manufacturer (none) -> DORABO
Connections:
- net +12V_LOADS renamed +24V_LOADS
- net +5V_GATE renamed +12V
- no-connect marks 2 -> 1
Other:
- note added: "GATE DRIVER SUPPLY = +12V AUX"
- note added: "PTC / 24 V / 100 W / 4.17 A, ПУСК ~4.8 A"
- note added: "Q601: G=4, S=1/2/3, D=5; SO-8FL exposed drain is not GND. RDS(on) max 2.4 mOhm at VGS=10 V, 25 C; gate now ~12 V. Conduction ~0.042 W at 4.17 A / ~0.055 W at 4.8 A (25 C). D601 SMBJ30A: standoff 30 V > 25 V supply, clamp 48.4 V < 60 V VDS."
- note added: "TPS70950 removed in 0.14: UCC27524A VDD is the regulated +12V aux rail (4.5-18 V range, isolated from 24 V input transients by the buck)."
- note added: "U601: ENA=3.3 V, INA=HEATER_EN. Channel B disabled. VDD = +12V from the aux buck (sheet 06). C601/C602 close to VDD/GND. Short OUTA-G-S-GND loop. MCU R210=10k pull-down; R602 discharges the gate."
- note removed: "EN = +3V3; do not connect EN to 12 V. TPS70950 has reverse-current protection. C604: >=2.2 uF effective at 5 V; ESR <=0.2 ohm. C602 >=1 uF effective, directly at driver. C603/C604 directly at LDO. Gate supply budget <=5 mA; PTC ON/OFF <=1 Hz."
- note removed: "LOCAL 5 V GATE SUPPLY"
- note removed: "PTC / 12 V / 100 W / 8.33 A, ПУСК ~9.58 A"
- note removed: "Q601: G=4, S=1/2/3, D=5; SO-8FL exposed drain is not GND. RDS(on) max 3.3 mOhm at VGS=4.5 V, Tj=25 C. Conduction ~0.229 W at 8.33 A / ~0.303 W at 9.58 A. Hot resistance and switching overshoot still require thermal/scope checks."
- note removed: "U601: ENA=3.3 V, INA=HEATER_EN. Channel B disabled. VDD from local +5V_GATE. C601/C602 close to VDD/GND. Short OUTA-G-S-GND loop. MCU R210=10k pull-down; R602 discharges the gate when unpowered. Verify 5 V startup/droop: SOIC start threshold up to 4.65 V; never power directly from 12 V."
- title: 05 - PTC heater switch -> 05 - PTC heater switch (24 V)
