File: pcb/PCB_V1/Heater.kicad_sch (KiCad schematic)
At the start: 8 parts, among them J601 PTC + / switched - (3.5 mm), Q601 NTMFS5C628NLT1G, U601 UCC27524ADR

Commit message: pcb: refine 24 V bias, branch protection and auxiliary supply
Parts:
- C602: value 2.2u / 25V X7R -> 4.7u / 25V X7R
Other:
- note added: "0.15 DRAFT: 24 V / 100 W PTC; power/thermal limits require prototype validation."
- note added: "PTC: низкочастотное ON/OFF. Внешний термостат/термопредохранитель последовательно с +PTC, с DC-рейтингом по току; температуру выбрать по механике нагревателя. На этой схеме он НЕ установлен. TVS — от выбросов на проводах, не защита от КЗ. Ветвь защищена F902; отключение при КЗ требует проверки."
- note removed: "0.13 DRAFT: power/thermal limits remain subject to prototype validation."
- note removed: "PTC: низкочастотное ON/OFF. Внешний термостат/термопредохранитель последовательно с +PTC, с DC-рейтингом по току; температуру выбрать по механике нагревателя. На этой схеме он НЕ установлен. TVS — от выбросов на проводах, не защита от КЗ. Предохранитель ещё нужен."
Changed lines of the file:
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@@
 		(title "05 - PTC heater switch (24 V)")
 		(date "2026-09-27")
-		(rev "0.14-DRAFT")
+		(rev "0.15-DRAFT")
 		(company "GrowBox controller")
-		(comment 1 "Prototype design; protection and thermal qualification pending")
+		(comment 1 "Engineering draft; startup, thermal and fault qualification pending")
 	)
 	(text "U601: ENA=3.3 V, INA=HEATER_EN. Channel B disabled. VDD = +12V from the aux buck (sheet 06).\nC601/C602 close to VDD/GND. Short OUTA-G-S-GND loop.\nMCU R210=10k pull-down; R602 discharges the gate."
@@
 		)
 	)
-	(text "PTC: низкочастотное ON/OFF. Внешний термостат/термопредохранитель\nпоследовательно с +PTC, с DC-рейтингом по току; температуру выбрать\nпо механике нагревателя. На этой схеме он НЕ установлен.\nTVS — от выбросов на проводах, не защита от КЗ. Предохранитель ещё нужен."
+	(text "PTC: низкочастотное ON/OFF. Внешний термостат/термопредохранитель\nпоследовательно с +PTC, с DC-рейтингом по току; температуру выбрать\nпо механике нагревателя. На этой схеме он НЕ установлен.\nTVS — от выбросов на проводах, не защита от КЗ. Ветвь защищена F902; отключение при КЗ требует проверки."
 		(exclude_from_sim no)
 		(at 20.32 175.26 0)
@@
 		)
 	)
-	(text "0.13 DRAFT: power/thermal limits remain subject to prototype validation."
+	(text "0.15 DRAFT: 24 V / 100 W PTC; power/thermal limits require prototype validation."
 		(exclude_from_sim no)
 		(at 20.32 24.13 0)
@@
 			)
 		)
-		(property "Value" "2.2u / 25V X7R"
+		(property "Value" "4.7u / 25V X7R"
 			(at 33.48 102.87 0)
 			(show_name no)
