File: pcb/PCB_V1/Heater.kicad_sch (KiCad schematic)
At the start: 8 parts, among them J601 PTC + / switched - (3.5 mm), Q601 NTMFS5C628NLT1G, U601 UCC27524ADR

Commit message: pcb: revision 0.16 - drop redundant F903, restore CH1 inductor margin, clean DRC and docs
Schematic/board:
- remove F903 (7.5 A LED blade fuse): F711 6.3 A and F721 3 A already fuse
  each LED channel and F903 had the smallest margin; TP903/#FLG0603 removed,
  LED channel fuses and C710 now sit on +24V
- L711 back to Bourns SRP1770TA-470M with R715 0.027 ohm: CH1 OCP headroom
  3.17 A (was 0.34 A), worst-case winding loss 0.77 W (was 1.22 W)
- ESP32 footprint GrowBox:ESP32-WROOM-32E_NoVias without the 12 in-pad
  0.2 mm vias: DRC now 0 violations (only unrouted connections remain)
- 167 components; ERC 0/0

Checks and docs:
- new check_all.py runs ERC, netlist/board verification, sizing reports,
  BOM export and DRC; --write refreshes review/*_v16 and sheet images
- verify_netlist.py, verify_board.py, analyze_*.py updated for 0.16
- REDESIGN_24V.md -> DESIGN.md (current design only), new CHANGELOG.md,
  superseded 12 V documents in PCB_V1/history/, older reports in
  review/history/, README files rewritten as entry points
- cost estimation paused; v0.15 price audit kept as history

Co-Authored-By: Claude Opus 5.5 <noreply@anthropic.com>
Other:
- note added: "0.16 DRAFT: 24 V / 100 W PTC; power/thermal limits require prototype validation."
- note removed: "0.15 DRAFT: 24 V / 100 W PTC; power/thermal limits require prototype validation."
Changed lines of the file:
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@@
 		(title "05 - PTC heater switch (24 V)")
 		(date "2026-09-27")
-		(rev "0.15-DRAFT")
+		(rev "0.16-DRAFT")
 		(company "GrowBox controller")
 		(comment 1 "Engineering draft; startup, thermal and fault qualification pending")
@@
 		)
 	)
-	(text "0.15 DRAFT: 24 V / 100 W PTC; power/thermal limits require prototype validation."
+	(text "0.16 DRAFT: 24 V / 100 W PTC; power/thermal limits require prototype validation."
 		(exclude_from_sim no)
 		(at 20.32 24.13 0)
