File: pcb/PCB_V1/Heater.kicad_sch (KiCad schematic)
At the start: 8 parts, among them J601 PTC + / switched - (3.5 mm), Q601 NTMFS5C628NLT1G, U601 UCC27524ADR

Commit message: pcb: integrate reviewed parts and validate initial 100mm placement
Parts:
- C602: LCSC (none) -> C98195; MPN (none) -> CL21B475KAFNNNE; Manufacturer (none) -> Samsung Electro-Mechanics
- J601: footprint TerminalBlock_Phoenix:TerminalBlock_Phoenix_PT-1,5-2-3.5-H_1x02_P3.50mm_Horizontal -> GrowBox:TerminalBlock_DORABO_DB125-3.5_1x02_P3.50mm_Horizontal
Other:
- note added: "0.17 DRAFT: 24 V / 100 W PTC; power/thermal limits require prototype validation."
- note removed: "0.16 DRAFT: 24 V / 100 W PTC; power/thermal limits require prototype validation."
Changed lines of the file:
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@@
 	(title_block
 		(title "05 - PTC heater switch (24 V)")
-		(date "2026-09-27")
-		(rev "0.16-DRAFT")
+		(date "2026-09-28")
+		(rev "0.17-DRAFT")
 		(company "GrowBox controller")
 		(comment 1 "Engineering draft; startup, thermal and fault qualification pending")
@@
 		)
 	)
-	(text "0.16 DRAFT: 24 V / 100 W PTC; power/thermal limits require prototype validation."
+	(text "0.17 DRAFT: 24 V / 100 W PTC; power/thermal limits require prototype validation."
 		(exclude_from_sim no)
 		(at 20.32 24.13 0)
@@
 			)
 		)
-		(property "Datasheet" ""
+		(property "Datasheet" "https://product.samsungsem.com/mlcc/CL21B475KAFNNN.do"
 			(at 30.48 101.6 0)
 			(hide yes)
@@
 					(unit 1)
 				)
+			)
+		)
+		(property "Manufacturer" "Samsung Electro-Mechanics"
+			(at 30.48 101.6 0)
+			(hide yes)
+			(show_name no)
+			(do_not_autoplace no)
+			(effects
+				(font
+					(size 1 1)
+				)
+				(justify left)
+			)
+		)
+		(property "MPN" "CL21B475KAFNNNE"
+			(at 30.48 101.6 0)
+			(hide yes)
+			(show_name no)
+			(do_not_autoplace no)
+			(effects
+				(font
+					(size 1 1)
+				)
+				(justify left)
+			)
+		)
+		(property "LCSC" "C98195"
+			(at 30.48 101.6 0)
+			(hide yes)
+			(show_name no)
+			(do_not_autoplace no)
+			(effects
+				(font
+					(size 1 1)
+				)
+				(justify left)
 			)
 		)
@@
 			)
 		)
-		(property "Footprint" "TerminalBlock_Phoenix:TerminalBlock_Phoenix_PT-1,5-2-3.5-H_1x02_P3.50mm_Horizontal"
+		(property "Footprint" "GrowBox:TerminalBlock_DORABO_DB125-3.5_1x02_P3.50mm_Horizontal"
 			(at 254 48.26 0)
 			(hide yes)

Commit message: pcb: simplify passives and microSD circuitry for revision 0.18
Parts:
- C601: value 100n / 25V -> 100n 50V X7R; LCSC (none) -> C1591; MPN (none) -> CL10B104KB8NNNC; Manufacturer (none) -> Samsung
- R602: value 100k -> 100k 1%; LCSC (none) -> C25803; MPN (none) -> 0603WAF1003T5E; Manufacturer (none) -> UNI-ROYAL
Other:
- note added: "0.18 DRAFT: 24 V / 100 W PTC; power/thermal limits require prototype validation."
- note removed: "0.17 DRAFT: 24 V / 100 W PTC; power/thermal limits require prototype validation."
Changed lines of the file:
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@@
 	(title_block
 		(title "05 - PTC heater switch (24 V)")
-		(date "2026-09-28")
-		(rev "0.17-DRAFT")
+		(date "2026-09-29")
+		(rev "0.18-DRAFT")
 		(company "GrowBox controller")
-		(comment 1 "Engineering draft; startup, thermal and fault qualification pending")
+		(comment 1 "Simplified prototype; unrouted; hardware qualification pending")
 	)
 	(text "U601: ENA=3.3 V, INA=HEATER_EN. Channel B disabled. VDD = +12V from the aux buck (sheet 06).\nC601/C602 close to VDD/GND. Short OUTA-G-S-GND loop.\nMCU R210=10k pull-down; R602 discharges the gate."
@@
 		)
 	)
-	(text "0.17 DRAFT: 24 V / 100 W PTC; power/thermal limits require prototype validation."
+	(text "0.18 DRAFT: 24 V / 100 W PTC; power/thermal limits require prototype validation."
 		(exclude_from_sim no)
 		(at 20.32 24.13 0)
@@
 			)
 		)
-		(property "Value" "100k"
+		(property "Value" "100k 1%"
 			(at 152.86 99.06 0)
 			(show_name no)
@@
 					(unit 1)
 				)
+			)
+		)
+		(property "Manufacturer" "UNI-ROYAL"
+			(at 149.86 97.79 0)
+			(hide yes)
+			(show_name no)
+			(do_not_autoplace no)
+			(effects
+				(font
+					(size 1 1)
+				)
+				(justify left)
+			)
+		)
+		(property "MPN" "0603WAF1003T5E"
+			(at 149.86 97.79 0)
+			(hide yes)
+			(show_name no)
+			(do_not_autoplace no)
+			(effects
+				(font
+					(size 1 1)
+				)
+				(justify left)
+			)
+		)
+		(property "LCSC" "C25803"
+			(at 149.86 97.79 0)
+			(hide yes)
+			(show_name no)
+			(do_not_autoplace no)
+			(effects
+				(font
+					(size 1 1)
+				)
+				(justify left)
 			)
 		)
@@
 			)
 		)
-		(property "Value" "100n / 25V"
+		(property "Value" "100n 50V X7R"
 			(at 33.48 67.31 0)
 			(show_name no)
@@
 			)
 		)
+		(property "Manufacturer" "Samsung"
+			(at 30.48 66.04 0)
+			(hide yes)
+			(show_name no)
+			(do_not_autoplace no)
+			(effects
+				(font
+					(size 1 1)
+				)
+				(justify left)
+			)
+		)
+		(property "MPN" "CL10B104KB8NNNC"
+			(at 30.48 66.04 0)
+			(hide yes)
+			(show_name no)
+			(do_not_autoplace no)
+			(effects
+				(font
+					(size 1 1)
+				)
+				(justify left)
+			)
+		)
+		(property "LCSC" "C1591"
+			(at 30.48 66.04 0)
+			(hide yes)
+			(show_name no)
+			(do_not_autoplace no)
+			(effects
+				(font
+					(size 1 1)
+				)
+				(justify left)
+			)
+		)
