File: pcb/PCB_V1/Heater.kicad_sch (KiCad schematic)
At the start: 8 parts, among them J601 PTC + / switched - (3.5 mm), Q601 NTMFS5C628NLT1G, U601 UCC27524ADR

Commit message: pcb: revision 0.19 cost-down in the schematic, same footprints
Schematic and calculations only; PCB_V1.kicad_pcb is untouched on the
user's request. All substitutions keep footprints and nets.

- C716-C719, C726-C728: TDK C3225X7R2A106K250AC (X7R, published DC-bias
  curve 2.35 uF at 49 V) instead of Samsung CL32Y106KCV6PNE.
- C104/C105/C401: Samsung CL21A226MPQNNNE X5R; C521/C710/C715/C725/
  C905/C906: Taiyo Yuden UMK325AB7106KMHP.
- C602 shares CL21A106KAYNNNE with C201 (1.41 uF screen >= 1 uF);
  D601 shares SMBJ26CA with D901 (D_TVS symbol, 42.1 V clamp);
  R501/R511/R521 33R; F904 3 A shared with F721.
- analyze_led_power/analyze_power_path/verify_netlist updated; price and
  JLC snapshots v19; reports, sheet images and checks log v19.
- COST_DOWN.md: USD 37.50 per board (was 39.82), 65 purchase codes,
  rejected candidates and board status.

verify_board.py reports value differences for 17 parts until the board
is synced (footprints and nets already match); all other checks pass.

Co-Authored-By: Claude Opus 5.5 <noreply@anthropic.com>
Parts:
- C602: value 4.7u / 25V X7R -> 10u / 25V X5R; LCSC C98195 -> C15850; MPN CL21B475KAFNNNE -> CL21A106KAYNNNE
- D601: value SMBJ30A-E3/52 -> SMBJ26CA-E3/52; symbol Device:D_Zener -> Device:D_TVS; LCSC C1973126 -> C515606; MPN SMBJ30A-E3/52 -> SMBJ26CA-E3/52
Changed lines of the file:
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@@
 			)
 		)
-		(property "Value" "4.7u / 25V X7R"
+		(property "Value" "10u / 25V X5R"
 			(at 33.48 102.87 0)
 			(show_name no)
@@
 			)
 		)
-		(property "Datasheet" "https://product.samsungsem.com/mlcc/CL21B475KAFNNN.do"
+		(property "Datasheet" "https://product.samsungsem.com/mlcc/CL21A106KAYNNN.do"
 			(at 30.48 101.6 0)
 			(hide yes)
@@
 			)
 		)
-		(property "MPN" "CL21B475KAFNNNE"
-			(at 30.48 101.6 0)
-			(hide yes)
-			(show_name no)
-			(do_not_autoplace no)
-			(effects
-				(font
-					(size 1 1)
-				)
-				(justify left)
-			)
-		)
-		(property "LCSC" "C98195"
+		(property "MPN" "CL21A106KAYNNNE"
+			(at 30.48 101.6 0)
+			(hide yes)
+			(show_name no)
+			(do_not_autoplace no)
+			(effects
+				(font
+					(size 1 1)
+				)
+				(justify left)
+			)
+		)
+		(property "LCSC" "C15850"
 			(at 30.48 101.6 0)
 			(hide yes)
@@
 	)
 	(symbol
-		(lib_id "Device:D_Zener")
+		(lib_id "Device:D_TVS")
 		(at 259.08 104.14 90)
 		(unit 1)
@@
 			)
 		)
-		(property "Value" "SMBJ30A-E3/52"
+		(property "Value" "SMBJ26CA-E3/52"
 			(at 259.08 99.06 90)
 			(show_name no)
@@
 			)
 		)
-		(property "LCSC" "C1973126"
+		(property "LCSC" "C515606"
 			(at 259.08 104.14 0)
 			(effects
@@
 			)
 		)
-		(property "MPN" "SMBJ30A-E3/52"
+		(property "MPN" "SMBJ26CA-E3/52"
 			(at 259.08 104.14 0)
 			(effects
