File: pcb/PCB_V1/LEDDrivers.kicad_sch (KiCad schematic)
At the start: 67 parts, among them J711 LED +/- (return isolated), J721 LED +/- (return isolated), J731 LED +/- (return isolated), Q711 SiR106ADP-T1-RE3, Q721 CSD19538Q3A, Q731 CSD19538Q3A, U700 SN74LVC1G08DBVR, U710 AL8853S-13, U720 AL8853S-13, U730 AL8853S-13

Commit message: pcb: move board to 24 V input with 12 V aux buck and merged LED bar channel
Revision 0.14 of PCB_V1 (see pcb/PCB_V1/REDESIGN_24V.md):
- 24 V input on keyed XT60PW-M (pin 1 GND, pin 2 +24V); LM74700, input
  MOSFET and F901 removed; SMBJ26CA TVS; 220 uF/50 V bulk
- ATM mini-blade fuses in XF-508P-B-B holders: F902 10 A loads, F903 7.5 A LED
- new LMR16020 24 V -> 12 V aux buck (500 kHz) feeding PC fans, the
  UCC27524A heater gate driver and the TPS54202 3.3 V buck; TPS70950 removed
- heater and pump on 24 V: SMBJ30A drain TVS, AO3422 + SS36 pump stage
- LED CH1 panel keeps SRP1770TA/0.027 R/1k, switch now CSD19534Q5A;
  CH2 drives both identical bars in parallel (J721 || J731, 0.40 R);
  third AL8853 channel removed
- TS-1187A buttons, DORABO/KANGNEX terminals
- project library: LMR16020 and CSD19534Q5A symbols, TI DQJ and XF-508P
  footprints
- verify_netlist.py / verify_board.py / analyze_*.py updated for 24 V;
  new sync_board.py updates the unrouted staging board from the netlist
- ERC 0/0; netlist, board and sizing checks pass; DRC only the 12 known
  ESP32 drill sizes plus unrouted connections; 163 components

Co-Authored-By: Claude Opus 5.5 <noreply@anthropic.com>
Parts:
- removed C731: 1u 25V X7R, Capacitor_SMD:C_0805_2012Metric, symbol Device:C
- removed C732: 100p / comp tune, Capacitor_SMD:C_0603_1608Metric, symbol Device:C
- removed C733: 100p / CS tune, Capacitor_SMD:C_0603_1608Metric, symbol Device:C
- removed C734: 220n / comp tune, Capacitor_SMD:C_0603_1608Metric, symbol Device:C
- removed C735: 22u 25V X7R, Capacitor_SMD:C_1210_3225Metric, symbol Device:C
- removed C736, C737: 10u 100V X7S, Capacitor_SMD:C_1210_3225Metric, symbol Device:C
- removed D731: STPS2H100AFY, Diode_SMD:D_SOD-128, symbol Device:D_Schottky
- removed L731: 47u SRP1265A-470M, GrowBox:L_Bourns_SRP1265A, symbol Device:L
- removed Q731: CSD19538Q3A, GrowBox:TI_DNH0008A_CSD19538Q3A, symbol GrowBox:CSD19538Q3A
- removed R731: 10R, Resistor_SMD:R_0603_1608Metric, symbol Device:R
- removed R732: 2.7k 1% / slope tune, Resistor_SMD:R_0603_1608Metric, symbol Device:R
- removed R733: 100k, Resistor_SMD:R_0603_1608Metric, symbol Device:R
- removed R734: 10k / comp tune, Resistor_SMD:R_0603_1608Metric, symbol Device:R
- removed R735: 0.047 1% >=1W, Resistor_SMD:R_2512_6332Metric, symbol Device:R
- removed R736: 0.80 1% >=0.25W, Resistor_SMD:R_1206_3216Metric, symbol Device:R
- removed R737: 316k 1%, Resistor_SMD:R_0603_1608Metric, symbol Device:R
- removed R738: 10k 1%, Resistor_SMD:R_0603_1608Metric, symbol Device:R
- removed U730: AL8853S-13, Package_SO:SOIC-8_3.9x4.9mm_P1.27mm, symbol GrowBox:AL8853
- added C710: 10u 50V X7R, Capacitor_SMD:C_1210_3225Metric, symbol Device:C
- added C728: 10u 100V X7S, Capacitor_SMD:C_1210_3225Metric, symbol Device:C
- C711, C721: value 1u 25V X7R -> 1u 50V X7R; LCSC (none) -> C28323; MPN (none) -> CL21B105KBFNNNE; Manufacturer (none) -> Samsung
- C715, C725: value 22u 25V X7R -> 10u 50V X7R; LCSC (none) -> C77102; MPN (none) -> GRM32ER71H106KA12L; Manufacturer (none) -> Murata
- J711, J721, J731: LCSC (none) -> C8465; MPN (none) -> WJ500V-5.08-2P; Manufacturer (none) -> KANGNEX
- Q711: value SiR106ADP-T1-RE3 -> CSD19534Q5A; footprint Package_SO:PowerPAK_SO-8_Single -> GrowBox:TI_DQJ0008A_CSD19534Q5A; symbol GrowBox:NMOS_PowerPAK_Candidate -> GrowBox:CSD19534Q5A; LCSC (none) -> C114200; MPN (none) -> CSD19534Q5A; Manufacturer (none) -> Texas Instruments
- R715: value 0.027 1% >=2W -> 0.027 1% >=1W
- R726: value 0.80 1% >=0.25W -> 0.40 1% >=0.25W
Connections:
- net LED3_OUT is gone; now on net LED2_OUT: J731.1 (Pin_1)
- net LED3_RETURN is gone; now on net LED2_RETURN: J731.2 (Pin_2)
- net GND: now also C710.2, C728.2
- net LED2_OUT: now also C728.1
- net +12V_LED renamed +24V_LED
- net +24V_LED: now also C710.1
Other:
- note added: "0.14 DRAFT: 24 V input. CH1 panel 1.099 A; CH2 two bars 0.5 A total. AL8853 / CSD19534Q5A / CSD19538Q3A."
- note added: "144 sizing cases at 24 V (2 ch x 72); typical ramp only. Startup/OCP, outer-loop stability, hot magnetics and thermal tests remain required."
- note added: "CH2: 0.500 A nominal / two identical bars in parallel (J721 + J731)"
- note added: "Do not connect LED- to GND. Only J721/J731 (same channel) share LED2_RETURN; never join CH1 and CH2 returns. Output short protection needs branch fuses/disconnect; boost diode conducts at shutdown."
- note added: "J731: second bar on CH2, parallel with J721. Former CH3 removed in 0.14."
- note added: "TWO CONSTANT-CURRENT BOOST CHANNELS FROM +24V_LED / COMMON DIMMING"
- note removed: "0.12 DRAFT; component budget around USD 30 is a guide, not a hard cap. AL8853 / CSD19538Q3A."
- note removed: "216 sizing cases checked; typical ramp only. Startup/OCP, outer-loop stability, hot magnetics and thermal tests remain required."
- note removed: "CH2: 0.250 A nominal / strip"
- note removed: "CH3: 0.250 A nominal / strip"
- note removed: "Do not connect LED- to GND or join LED returns. Output short protection needs branch fuses/disconnect; boost diode conducts at shutdown."
- note removed: "THREE INDEPENDENT CONSTANT-CURRENT BOOST CHANNELS / COMMON DIMMING"
- title: 07 - AL8853 cost-down LED drivers -> 07 - AL8853 LED drivers, 24 V input, 2 channels
