File: pcb/PCB_V1/LEDDrivers.kicad_sch (KiCad schematic)
At the start: 50 parts, among them J711 LED +/- (return isolated), J721 LED +/- (return isolated), J731 LED +/- (return isolated), Q711 CSD19534Q5A, Q721 CSD19538Q3A, U700 SN74LVC1G08DBVR, U710 AL8853S-13, U720 AL8853S-13

Commit message: pcb: refine 24 V bias, branch protection and auxiliary supply
Parts:
- added F711: 6.3A / 045106.3MRL, GrowBox:Fuse_Littelfuse_451, symbol Device:Fuse
- added F721: 3A / 0451003.MRL, GrowBox:Fuse_Littelfuse_451, symbol Device:Fuse
- L711: value 47u SRP1770TA-470M -> 47u SRP1265A-470M; footprint Inductor_SMD:L_Bourns_SRP1770TA_16.9x16.9mm -> GrowBox:L_Bourns_SRP1265A; LCSC C2041872 -> C840530; MPN SRP1770TA-470M -> SRP1265A-470M
- R715: value 0.027 1% >=1W -> 0.043 1% >=1W
- R726: value 0.40 1% >=0.25W -> 0.43 1% >=0.25W
Connections:
- net +24V_LED: now also F711.1, F721.1; no longer C711.1, C715.1, C721.1, C725.1, L711.1, L721.1, U710.1 (VIN), U720.1 (VIN)
- new net +12V: C711.1, C721.1, U710.1 (VIN), U720.1 (VIN)
- new net LED1_VIN: C715.1, F711.2, L711.1
- new net LED2_VIN: C725.1, F721.2, L721.1
Other:
- note added: "0.15 DRAFT: power input 24 V; AL8853 bias 12 V. CH1 1.099 A; CH2 0.465 A total. Qualification pending."
- note added: "144 sizing cases: 24 V power / 12 V IC bias. Typical ramp only; startup, compensation, hot magnetics and fault clearing require tests."
- note added: "CH2: 0.465 A nominal TOTAL / J721 + J731 parallel; <=0.484 A at FB/R tolerance corner"
- note added: "DRAFT: 120 kHz; OVP nominal 65.2 V. 100 V output parts. Current calculations: REDESIGN_24V.md / LED_power_v15.txt."
- note added: "J731: second bar on CH2, parallel with J721. Sharing need not be equal; one open bar leaves the other below 0.5 A (steady-state)."
- note added: "LED-: J721/J731 share CH2; never join CH1 to CH2 or GND. F711/F721 protect INPUT paths; boost diodes conduct at shutdown."
- note removed: "0.14 DRAFT: 24 V input. CH1 panel 1.099 A; CH2 two bars 0.5 A total. AL8853 / CSD19534Q5A / CSD19538Q3A."
- note removed: "144 sizing cases at 24 V (2 ch x 72); typical ramp only. Startup/OCP, outer-loop stability, hot magnetics and thermal tests remain required."
- note removed: "CH2: 0.500 A nominal / two identical bars in parallel (J721 + J731)"
- note removed: "DRAFT: 120 kHz; OVP nominal 65.2 V. 100 V power parts; selected MPNs and sizing: LED_POWER_COMPONENTS.md."
- note removed: "Do not connect LED- to GND. Only J721/J731 (same channel) share LED2_RETURN; never join CH1 and CH2 returns. Output short protection needs branch fuses/disconnect; boost diode conducts at shutdown."
- note removed: "J731: second bar on CH2, parallel with J721. Former CH3 removed in 0.14."
