File: pcb/PCB_V1/LEDDrivers.kicad_sch (KiCad schematic)
At the start: 52 parts, among them J711 LED +/- (return isolated), J721 LED +/- (return isolated), J731 LED +/- (return isolated), Q711 CSD19534Q5A, Q721 CSD19538Q3A, U700 SN74LVC1G08DBVR, U710 AL8853S-13, U720 AL8853S-13

Commit message: pcb: revision 0.16 - drop redundant F903, restore CH1 inductor margin, clean DRC and docs
Schematic/board:
- remove F903 (7.5 A LED blade fuse): F711 6.3 A and F721 3 A already fuse
  each LED channel and F903 had the smallest margin; TP903/#FLG0603 removed,
  LED channel fuses and C710 now sit on +24V
- L711 back to Bourns SRP1770TA-470M with R715 0.027 ohm: CH1 OCP headroom
  3.17 A (was 0.34 A), worst-case winding loss 0.77 W (was 1.22 W)
- ESP32 footprint GrowBox:ESP32-WROOM-32E_NoVias without the 12 in-pad
  0.2 mm vias: DRC now 0 violations (only unrouted connections remain)
- 167 components; ERC 0/0

Checks and docs:
- new check_all.py runs ERC, netlist/board verification, sizing reports,
  BOM export and DRC; --write refreshes review/*_v16 and sheet images
- verify_netlist.py, verify_board.py, analyze_*.py updated for 0.16
- REDESIGN_24V.md -> DESIGN.md (current design only), new CHANGELOG.md,
  superseded 12 V documents in PCB_V1/history/, older reports in
  review/history/, README files rewritten as entry points
- cost estimation paused; v0.15 price audit kept as history

Co-Authored-By: Claude Opus 5.5 <noreply@anthropic.com>
Parts:
- L711: value 47u SRP1265A-470M -> 47u SRP1770TA-470M; footprint GrowBox:L_Bourns_SRP1265A -> Inductor_SMD:L_Bourns_SRP1770TA_16.9x16.9mm; LCSC C840530 -> C2041872; MPN SRP1265A-470M -> SRP1770TA-470M
- R715: value 0.043 1% >=1W -> 0.027 1% >=1W
Connections:
- net +24V_LED renamed +24V
Other:
- note added: "0.16 DRAFT: power input 24 V; AL8853 bias 12 V. CH1 back to SRP1770TA-470M / 0.027 ohm (OCP headroom). CH1 1.099 A; CH2 0.465 A total. Qualification pending."
- note added: "TWO CONSTANT-CURRENT BOOST CHANNELS FROM +24V (EACH CHANNEL FUSED: F711, F721) / COMMON DIMMING"
- note removed: "0.15 DRAFT: power input 24 V; AL8853 bias 12 V. CH1 1.099 A; CH2 0.465 A total. Qualification pending."
- note removed: "TWO CONSTANT-CURRENT BOOST CHANNELS FROM +24V_LED / COMMON DIMMING"
Changed lines of the file:
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@@
 		(title "07 - AL8853 LED drivers, 24 V input, 2 channels")
 		(date "2026-09-27")
-		(rev "0.15-DRAFT")
+		(rev "0.16-DRAFT")
 		(company "GrowBox controller")
 		(comment 1 "Engineering draft; startup, thermal and fault qualification pending")
@@
 		)
 	)
-	(text "TWO CONSTANT-CURRENT BOOST CHANNELS FROM +24V_LED / COMMON DIMMING"
+	(text "TWO CONSTANT-CURRENT BOOST CHANNELS FROM +24V (EACH CHANNEL FUSED: F711, F721) / COMMON DIMMING"
 		(exclude_from_sim no)
 		(at 20.32 15.24 0)
@@
 		)
 	)
-	(text "0.15 DRAFT: power input 24 V; AL8853 bias 12 V. CH1 1.099 A; CH2 0.465 A total. Qualification pending."
+	(text "0.16 DRAFT: power input 24 V; AL8853 bias 12 V. CH1 back to SRP1770TA-470M / 0.027 ohm (OCP headroom). CH1 1.099 A; CH2 0.465 A total. Qualification pending."
 		(exclude_from_sim no)
 		(at 20.32 22.86 0)
@@
 			)
 		)
-		(property "Value" "0.043 1% >=1W"
+		(property "Value" "0.027 1% >=1W"
 			(at 252.73 157.48 0)
 			(show_name no)
@@
 			)
 		)
-		(property "Value" "47u SRP1265A-470M"
+		(property "Value" "47u SRP1770TA-470M"
 			(at 149.86 87.63 90)
 			(show_name no)
@@
 			)
 		)
-		(property "Footprint" "GrowBox:L_Bourns_SRP1265A"
+		(property "Footprint" "Inductor_SMD:L_Bourns_SRP1770TA_16.9x16.9mm"
 			(at 165.1 97.79 90)
 			(hide yes)
@@
 			)
 		)
-		(property "MPN" "SRP1265A-470M"
+		(property "MPN" "SRP1770TA-470M"
 			(at 165.1 97.79 90)
 			(hide yes)
@@
 			)
 		)
-		(property "LCSC" "C840530"
+		(property "LCSC" "C2041872"
 			(at 165.1 97.79 90)
 			(hide yes)
@@
 		)
 	)
-	(global_label "+24V_LED"
+	(global_label "+24V"
 		(shape bidirectional)
 		(at 40.64 142.24 90)
@@
 		)
 	)
-	(global_label "+24V_LED"
+	(global_label "+24V"
 		(shape bidirectional)
 		(at 455.93 153.67 180)
@@
 		)
 	)
-	(global_label "+24V_LED"
+	(global_label "+24V"
 		(shape bidirectional)
 		(at 455.93 254.0 180)
