File: pcb/PCB_V1/LEDDrivers.kicad_sch (KiCad schematic)
At the start: 50 parts, among them J711 LED +/- (return isolated), J721 LED +/- (return isolated), J731 LED +/- (return isolated), Q711 AOD66923, Q721 AOD66923, U700 SN74LVC1G08DBVR, U710 AL8853S-13, U720 AL8853S-13

Commit message: pcb: revision 0.22 routing preparation
- Stack confirmed by the user: 1.6 mm, 1 oz outer, 0.5 oz inner.
- LED output MLCCs: Murata GRM32EC72A106KE05L (X7S, 50k in stock) instead
  of TDK; DC-bias digitised from Murata data (2.60 uF at 49 V, model
  2.55 uF), CH1 bank 6.44 uF effective.
- microSD: HRO TF-01A (push-push, C91145) on a project footprint from the
  HRO drawing, checked against the LCSC land; SD passives re-placed.
- TP301 on the PCF8563 CLKOUT for crystal trimming.
- Kelvin net ties NT711/NT712/NT721/NT722 at the LED-driver shunts
  (LED*_CS_K, LED*_FB_K); net ties are excluded from the BOM export.
- analyze_copper.py: IPC-2221 copper screen for the confirmed stack
  (main 24 V path needs pours on both outer layers, via counts).
- L711 and XT60PW-M re-checked and kept; reports v22 and ROUTING_PREP.md.
  USD 30.04 per board (28.42 for five), ERC 0, DRC 0.

Co-Authored-By: Claude Opus 5.5 <noreply@anthropic.com>
Parts:
- added NT711, NT712, NT721, NT722: Kelvin, NetTie:NetTie-2_SMD_Pad0.5mm, symbol Device:NetTie_2
- C716, C717, C718, C719, C726, C727, C728: value 10u 100V X7R -> 10u 100V X7S; LCSC C49296968 -> C576517; MPN C3225X7R2A106K250AC -> GRM32EC72A106KE05L; Manufacturer TDK -> Murata
Connections:
- net LED1_RETURN: now also NT712.1; no longer U710.5 (FB)
- net LED1_SOURCE: now also NT711.1; no longer R712.1
- net LED2_RETURN: now also NT722.1; no longer U720.5 (FB)
- net LED2_SOURCE: now also NT721.1; no longer R722.1
- new net LED1_CS_K: NT711.2, R712.1
- new net LED1_FB_K: NT712.2, U710.5 (FB)
- new net LED2_CS_K: NT721.2, R722.1
- new net LED2_FB_K: NT722.2, U720.5 (FB)
Other:
- note added: "0.22 DRAFT: Q711/Q721 AOD66923 DPAK, D711/D721 SS5P10 TO-277A. Power input 24 V; AL8853 bias 12 V. CH1 back to SRP1770TA-470M / 0.027 ohm (OCP headroom). CH1 1.111 A; CH2 0.465 A total. Qualification pending."
- note removed: "0.21 DRAFT: Q711/Q721 AOD66923 DPAK, D711/D721 SS5P10 TO-277A. Power input 24 V; AL8853 bias 12 V. CH1 back to SRP1770TA-470M / 0.027 ohm (OCP headroom). CH1 1.111 A; CH2 0.465 A total. Qualification pending."
