File: pcb/PCB_V1/PCB_V1.kicad_pcb (KiCad board)
At the start: 4 copper layers, 100 x 100 mm, 175 parts, among them J201 UART / 3V3 logic, J301 SHT4x / XH 2.50, J302 FLOAT / WAGO 2601, J401 Molex 104031-0811, J501 FAN1 / WAGO 2601, J511 FAN2 / WAGO 2601, J521 PUMP + / switched -, J601 PTC + / switched -, J711 LED +/- (return isolated), J721 LED +/- (return isolated), J731 LED +/- (return isolated), J901 12 V IN / 25 A design, Q501 AO3400A, Q511 AO3400A, Q521 AO3400A, Q601 NTMFS5C628NLT1G, Q711 SiR106ADP-T1-RE3, Q721 CSD19538Q3A, Q731 CSD19538Q3A, Q901 NTMFS5C628NLT1G, SW201 RESET, SW202 BOOT, U101 TPS54202DDCR, U201 ESP32-WROOM-32E-N4, U301 DS3231MZ+TRL, U601 UCC27524ADR, U602 TPS70950DBVR, U700 SN74LVC1G08DBVR, U710 AL8853S-13, U720 AL8853S-13, U730 AL8853S-13, U901 LM74700QDBVRQ1

Commit message: pcb: move board to 24 V input with 12 V aux buck and merged LED bar channel
Revision 0.14 of PCB_V1 (see pcb/PCB_V1/REDESIGN_24V.md):
- 24 V input on keyed XT60PW-M (pin 1 GND, pin 2 +24V); LM74700, input
  MOSFET and F901 removed; SMBJ26CA TVS; 220 uF/50 V bulk
- ATM mini-blade fuses in XF-508P-B-B holders: F902 10 A loads, F903 7.5 A LED
- new LMR16020 24 V -> 12 V aux buck (500 kHz) feeding PC fans, the
  UCC27524A heater gate driver and the TPS54202 3.3 V buck; TPS70950 removed
- heater and pump on 24 V: SMBJ30A drain TVS, AO3422 + SS36 pump stage
- LED CH1 panel keeps SRP1770TA/0.027 R/1k, switch now CSD19534Q5A;
  CH2 drives both identical bars in parallel (J721 || J731, 0.40 R);
  third AL8853 channel removed
- TS-1187A buttons, DORABO/KANGNEX terminals
- project library: LMR16020 and CSD19534Q5A symbols, TI DQJ and XF-508P
  footprints
- verify_netlist.py / verify_board.py / analyze_*.py updated for 24 V;
  new sync_board.py updates the unrouted staging board from the netlist
- ERC 0/0; netlist, board and sizing checks pass; DRC only the 12 known
  ESP32 drill sizes plus unrouted connections; 163 components

Co-Authored-By: Claude Opus 5.5 <noreply@anthropic.com>
Parts:
- removed C603: 2.2u / 50V X7R, Capacitor_SMD:C_0805_2012Metric
- removed C604: 10u / 16V X7R, Capacitor_SMD:C_0805_2012Metric
- removed C731: 1u 25V X7R, Capacitor_SMD:C_0805_2012Metric
- removed C732: 100p / comp tune, Capacitor_SMD:C_0603_1608Metric
- removed C733: 100p / CS tune, Capacitor_SMD:C_0603_1608Metric
- removed C734: 220n / comp tune, Capacitor_SMD:C_0603_1608Metric
- removed C735: 22u 25V X7R, Capacitor_SMD:C_1210_3225Metric
- removed C736, C737: 10u 100V X7S, Capacitor_SMD:C_1210_3225Metric
- removed C903: 100n / 50V X7R, Capacitor_SMD:C_0805_2012Metric
- removed C904: 220n / 50V X7R, Capacitor_SMD:C_0805_2012Metric
- removed D731: STPS2H100AFY, Diode_SMD:D_SOD-128
- removed F901: 25 A preliminary / verify I2t, Fuse:Fuse_2920_7451Metric
- removed L731: 47u SRP1265A-470M, GrowBox:L_Bourns_SRP1265A
- removed Q731: CSD19538Q3A, GrowBox:TI_DNH0008A_CSD19538Q3A
- removed Q901: NTMFS5C628NLT1G, Package_SO:ONSemi_SO-8FL_488AA
- removed R731: 10R, Resistor_SMD:R_0603_1608Metric
- removed R732: 2.7k 1% / slope tune, Resistor_SMD:R_0603_1608Metric
- removed R733: 100k, Resistor_SMD:R_0603_1608Metric
- removed R734: 10k / comp tune, Resistor_SMD:R_0603_1608Metric
- removed R735: 0.047 1% >=1W, Resistor_SMD:R_2512_6332Metric
- removed R736: 0.80 1% >=0.25W, Resistor_SMD:R_1206_3216Metric
- removed R737: 316k 1%, Resistor_SMD:R_0603_1608Metric
- removed R738: 10k 1%, Resistor_SMD:R_0603_1608Metric
- removed R903: 0 / gate link, Resistor_SMD:R_0603_1608Metric
- removed U602: TPS70950DBVR, Package_TO_SOT_SMD:SOT-23-5
- removed U730: AL8853S-13, Package_SO:SOIC-8_3.9x4.9mm_P1.27mm
- removed U901: LM74700QDBVRQ1, Package_TO_SOT_SMD:SOT-23-6
- added C710: 10u 50V X7R, Capacitor_SMD:C_1210_3225Metric, F.Cu at (175.0, 1810.0)
- added C728: 10u 100V X7S, Capacitor_SMD:C_1210_3225Metric, F.Cu at (225.0, 1810.0)
- added C905: 10u 50V X7R, Capacitor_SMD:C_1210_3225Metric, F.Cu at (275.0, 1810.0)
- added C906: 10u 50V X7R, Capacitor_SMD:C_1210_3225Metric, F.Cu at (325.0, 1810.0)
- added C907: 100n 50V X7R, Capacitor_SMD:C_0603_1608Metric, F.Cu at (375.0, 1810.0)
- added C908: 100n 50V X7R, Capacitor_SMD:C_0603_1608Metric, F.Cu at (175.0, 1860.0)
- added C909: 22u 25V X7R, Capacitor_SMD:C_1210_3225Metric, F.Cu at (225.0, 1860.0)
- added C910: 22u 25V X7R, Capacitor_SMD:C_1210_3225Metric, F.Cu at (275.0, 1860.0)
- added D902: SS36-E3/57T, Diode_SMD:D_SMC, F.Cu at (325.0, 1860.0)
- added L902: 22u SRP1265A-220M, GrowBox:L_Bourns_SRP1265A, F.Cu at (375.0, 1860.0)
- added R904: 100k 1%, Resistor_SMD:R_0603_1608Metric, F.Cu at (175.0, 1910.0)
- added R905: 6.65k 1%, Resistor_SMD:R_0603_1608Metric, F.Cu at (225.0, 1910.0)
- added R906: 49.9k 1%, Resistor_SMD:R_0603_1608Metric, F.Cu at (275.0, 1910.0)
- added R907: 560k 1%, Resistor_SMD:R_0603_1608Metric, F.Cu at (325.0, 1910.0)
- added R908: 47k 1%, Resistor_SMD:R_0603_1608Metric, F.Cu at (375.0, 1910.0)
- added U902: LMR16020PDDAR, Package_SO:SOIC-8-1EP_3.9x4.9mm_P1.27mm_EP2.95x4.9mm_Mask2.71x3.4mm, F.Cu at (175.0, 1960.0)
- C521: value 10u / 25V X7R -> 10u / 50V X7R
- C711, C721: value 1u 25V X7R -> 1u 50V X7R
- C715, C725: value 22u 25V X7R -> 10u 50V X7R
- C901: value 220u / 35V low ESR -> 220u / 50V
- D521: value SS34-E3/57T -> SS36-E3/57T
- D601: value SMBJ18A-E3/52 -> SMBJ30A-E3/52
- D901: value SMBJ14CA-E3/52 -> SMBJ26CA-E3/52
- F902: value 20 A loads / verify -> 10A mini blade (ATM); footprint Fuse:Fuse_2920_7451Metric -> GrowBox:Fuseholder_Blade_Mini_XFCN_XF-508P
- F903: value 10 A LED / verify -> 7.5A mini blade (ATM); footprint Fuse:Fuse_2920_7451Metric -> GrowBox:Fuseholder_Blade_Mini_XFCN_XF-508P
- J302: value FLOAT / WAGO 2601 -> FLOAT / 3.5 mm; footprint TerminalBlock_WAGO:TerminalBlock_WAGO_2601-1102_1x02_P3.50mm_Horizontal -> TerminalBlock_Phoenix:TerminalBlock_Phoenix_PT-1,5-2-3.5-H_1x02_P3.50mm_Horizontal
- J501: value FAN1 / WAGO 2601 -> FAN1 / 3.5 mm; footprint TerminalBlock_WAGO:TerminalBlock_WAGO_2601-1104_1x04_P3.50mm_Horizontal -> TerminalBlock_Phoenix:TerminalBlock_Phoenix_PT-1,5-4-3.5-H_1x04_P3.50mm_Horizontal
- J511: value FAN2 / WAGO 2601 -> FAN2 / 3.5 mm; footprint TerminalBlock_WAGO:TerminalBlock_WAGO_2601-1104_1x04_P3.50mm_Horizontal -> TerminalBlock_Phoenix:TerminalBlock_Phoenix_PT-1,5-4-3.5-H_1x04_P3.50mm_Horizontal
- J521: value PUMP + / switched - -> PUMP + / switched - (3.5 mm); footprint TerminalBlock_WAGO:TerminalBlock_WAGO_2601-1102_1x02_P3.50mm_Horizontal -> TerminalBlock_Phoenix:TerminalBlock_Phoenix_PT-1,5-2-3.5-H_1x02_P3.50mm_Horizontal
- J601: value PTC + / switched - -> PTC + / switched - (3.5 mm); footprint TerminalBlock_WAGO:TerminalBlock_WAGO_2601-1102_1x02_P3.50mm_Horizontal -> TerminalBlock_Phoenix:TerminalBlock_Phoenix_PT-1,5-2-3.5-H_1x02_P3.50mm_Horizontal
- J901: value 12 V IN / 25 A design -> XT60PW-M 24V IN; footprint TerminalBlock_Phoenix:TerminalBlock_Phoenix_MKDS-1,5-2-5.08_1x02_P5.08mm_Horizontal -> Connector_AMASS:AMASS_XT60PW-M_1x02_P7.20mm_Horizontal
- Q521: value AO3400A -> AO3422
- Q711: value SiR106ADP-T1-RE3 -> CSD19534Q5A; footprint Package_SO:PowerPAK_SO-8_Single -> GrowBox:TI_DQJ0008A_CSD19534Q5A
- R715: value 0.027 1% >=2W -> 0.027 1% >=1W
- R726: value 0.80 1% >=0.25W -> 0.40 1% >=0.25W
- SW201, SW202: footprint Button_Switch_SMD:SW_SPST_TL3342 -> Button_Switch_SMD:SW_Push_1P1T_XKB_TS-1187A
- TP101: value +12V_PROTECTED -> +12V
- TP901: value +12V_PROTECTED -> +24V
- TP902: value +12V_LOADS -> +24V_LOADS
- TP903: value +12V_LED -> +24V_LED
Connections:
- net +12V_LED renamed +24V_LED
- C101 pad 1: +12V_PROTECTED -> +12V
- C102 pad 1: +12V_PROTECTED -> +12V
- C521 pad 1: +12V_LOADS -> +24V_LOADS
- C601 pad 1: +5V_GATE -> +12V
- C602 pad 1: +5V_GATE -> +12V
- C901 pad 1: +12V_PROTECTED -> +24V
- C902 pad 1: +12V_PROTECTED -> +24V
- D521 pad 1: +12V_LOADS -> +24V_LOADS
- D901 pad 1: +12V_FUSED -> +24V
- F902 pad 1: +12V_PROTECTED -> +24V
- F902 pad 2: +12V_LOADS -> +24V_LOADS
- F903 pad 1: +12V_PROTECTED -> +24V
- J501 pad 2: +12V_LOADS -> +12V
- J511 pad 2: +12V_LOADS -> +12V
- J521 pad 1: +12V_LOADS -> +24V_LOADS
- J601 pad 1: +12V_LOADS -> +24V_LOADS
- J731 pad 1: /LEDDrivers/LED3_OUT -> /LEDDrivers/LED2_OUT
- J731 pad 2: /LEDDrivers/LED3_RETURN -> /LEDDrivers/LED2_RETURN
- J901 pad 1: +12V_IN -> GND
- J901 pad 2: GND -> +24V
- TP101 pad 1: +12V_PROTECTED -> +12V
- TP901 pad 1: +12V_PROTECTED -> +24V
- TP902 pad 1: +12V_LOADS -> +24V_LOADS
- U101 pad 3: +12V_PROTECTED -> +12V
- U601 pad 6: +5V_GATE -> +12V
