File: pcb/PCB_V1/PCB_V1.kicad_pcb (KiCad board)
At the start: 4 copper layers, 100 x 100 mm, 163 parts, among them J201 UART / 3V3 logic, J301 SHT4x / XH 2.50, J302 FLOAT / 3.5 mm, J401 Molex 104031-0811, J501 FAN1 / 3.5 mm, J511 FAN2 / 3.5 mm, J521 PUMP + / switched - (3.5 mm), J601 PTC + / switched - (3.5 mm), J711 LED +/- (return isolated), J721 LED +/- (return isolated), J731 LED +/- (return isolated), J901 XT60PW-M 24V IN, Q501 AO3400A, Q511 AO3400A, Q521 AO3422, Q601 NTMFS5C628NLT1G, Q711 CSD19534Q5A, Q721 CSD19538Q3A, SW201 RESET, SW202 BOOT, U101 TPS54202DDCR, U201 ESP32-WROOM-32E-N4, U301 DS3231MZ+TRL, U601 UCC27524ADR, U700 SN74LVC1G08DBVR, U710 AL8853S-13, U720 AL8853S-13, U902 LMR16020PDDAR

Commit message: pcb: refine 24 V bias, branch protection and auxiliary supply
Parts:
- added F501: 1A / 0451001.MRL, GrowBox:Fuse_Littelfuse_451, F.Cu at (175.0, 2020.0)
- added F511: 1A / 0451001.MRL, GrowBox:Fuse_Littelfuse_451, F.Cu at (225.0, 2020.0)
- added F521: 1A / 0451001.MRL, GrowBox:Fuse_Littelfuse_451, F.Cu at (275.0, 2020.0)
- added F711: 6.3A / 045106.3MRL, GrowBox:Fuse_Littelfuse_451, F.Cu at (325.0, 2020.0)
- added F721: 3A / 0451003.MRL, GrowBox:Fuse_Littelfuse_451, F.Cu at (375.0, 2020.0)
- added F904: 2A / 0451002.MRL, GrowBox:Fuse_Littelfuse_451, F.Cu at (175.0, 2070.0)
- C602: value 2.2u / 25V X7R -> 4.7u / 25V X7R
- C909: value 22u 25V X7R -> 100u 25V polymer; footprint Capacitor_SMD:C_1210_3225Metric -> Capacitor_SMD:CP_Elec_8x6.9
- J521: value PUMP + / switched - (3.5 mm) -> PUMP 24V / 6W
- L711: value 47u SRP1770TA-470M -> 47u SRP1265A-470M; footprint Inductor_SMD:L_Bourns_SRP1770TA_16.9x16.9mm -> GrowBox:L_Bourns_SRP1265A
- R715: value 0.027 1% >=1W -> 0.043 1% >=1W
- R726: value 0.40 1% >=0.25W -> 0.43 1% >=0.25W
- R904: value 100k 1% -> 150k 0.1%
- R905: value 6.65k 1% -> 10k 0.1%
Connections:
- C521 pad 1: +24V_LOADS -> /Outputs/PUMP_24V
- C711 pad 1: +24V_LED -> +12V
- C715 pad 1: +24V_LED -> /LEDDrivers/LED1_VIN
- C721 pad 1: +24V_LED -> +12V
- C725 pad 1: +24V_LED -> /LEDDrivers/LED2_VIN
- C905 pad 1: +24V -> /InputPower/AUX_VIN
- C906 pad 1: +24V -> /InputPower/AUX_VIN
- C907 pad 1: +24V -> /InputPower/AUX_VIN
- D521 pad 1: +24V_LOADS -> /Outputs/PUMP_24V
- J501 pad 2: +12V -> /Outputs/FAN1_12V
- J511 pad 2: +12V -> /Outputs/FAN2_12V
- J521 pad 1: +24V_LOADS -> /Outputs/PUMP_24V
- L711 pad 1: +24V_LED -> /LEDDrivers/LED1_VIN
- L721 pad 1: +24V_LED -> /LEDDrivers/LED2_VIN
- R907 pad 1: +24V -> /InputPower/AUX_VIN
- U710 pad 1: +24V_LED -> +12V
- U720 pad 1: +24V_LED -> +12V
- U902 pad 2: +24V -> /InputPower/AUX_VIN
