File: pcb/PCB_V1/PCB_V1.kicad_pcb (KiCad board)
At the start: 4 copper layers, 100 x 100 mm, 169 parts, among them J201 UART / 3V3 logic, J301 SHT4x / XH 2.50, J302 FLOAT / 3.5 mm, J401 Molex 104031-0811, J501 FAN1 / 3.5 mm, J511 FAN2 / 3.5 mm, J521 PUMP 24V / 6W, J601 PTC + / switched - (3.5 mm), J711 LED +/- (return isolated), J721 LED +/- (return isolated), J731 LED +/- (return isolated), J901 XT60PW-M 24V IN, Q501 AO3400A, Q511 AO3400A, Q521 AO3422, Q601 NTMFS5C628NLT1G, Q711 CSD19534Q5A, Q721 CSD19538Q3A, SW201 RESET, SW202 BOOT, U101 TPS54202DDCR, U201 ESP32-WROOM-32E-N4, U301 DS3231MZ+TRL, U601 UCC27524ADR, U700 SN74LVC1G08DBVR, U710 AL8853S-13, U720 AL8853S-13, U902 LMR16020PDDAR

Commit message: pcb: revision 0.16 - drop redundant F903, restore CH1 inductor margin, clean DRC and docs
Schematic/board:
- remove F903 (7.5 A LED blade fuse): F711 6.3 A and F721 3 A already fuse
  each LED channel and F903 had the smallest margin; TP903/#FLG0603 removed,
  LED channel fuses and C710 now sit on +24V
- L711 back to Bourns SRP1770TA-470M with R715 0.027 ohm: CH1 OCP headroom
  3.17 A (was 0.34 A), worst-case winding loss 0.77 W (was 1.22 W)
- ESP32 footprint GrowBox:ESP32-WROOM-32E_NoVias without the 12 in-pad
  0.2 mm vias: DRC now 0 violations (only unrouted connections remain)
- 167 components; ERC 0/0

Checks and docs:
- new check_all.py runs ERC, netlist/board verification, sizing reports,
  BOM export and DRC; --write refreshes review/*_v16 and sheet images
- verify_netlist.py, verify_board.py, analyze_*.py updated for 0.16
- REDESIGN_24V.md -> DESIGN.md (current design only), new CHANGELOG.md,
  superseded 12 V documents in PCB_V1/history/, older reports in
  review/history/, README files rewritten as entry points
- cost estimation paused; v0.15 price audit kept as history

Co-Authored-By: Claude Opus 5.5 <noreply@anthropic.com>
Parts:
- removed F903: 7.5A mini blade (ATM), GrowBox:Fuseholder_Blade_Mini_XFCN_XF-508P
- removed TP903: +24V_LED, TestPoint:TestPoint_Pad_D2.0mm
- L711: value 47u SRP1265A-470M -> 47u SRP1770TA-470M; footprint GrowBox:L_Bourns_SRP1265A -> Inductor_SMD:L_Bourns_SRP1770TA_16.9x16.9mm
- R715: value 0.043 1% >=1W -> 0.027 1% >=1W
- U201: footprint RF_Module:ESP32-WROOM-32E -> GrowBox:ESP32-WROOM-32E_NoVias
Connections:
- C710 pad 1: +24V_LED -> +24V
- F711 pad 1: +24V_LED -> +24V
- F721 pad 1: +24V_LED -> +24V
