File: pcb/PCB_V1/PCB_V1.kicad_pcb (KiCad board)
At the start: 4 copper layers, 100 x 100 mm, 167 parts, among them J201 UART / 3V3 logic, J301 SHT4x / XH 2.50, J302 FLOAT / 3.5 mm, J401 Molex 104031-0811, J501 FAN1 / 3.5 mm, J511 FAN2 / 3.5 mm, J521 PUMP 24V / 6W, J601 PTC + / switched - (3.5 mm), J711 LED +/- (return isolated), J721 LED +/- (return isolated), J731 LED +/- (return isolated), J901 XT60PW-M 24V IN, Q501 AO3400A, Q511 AO3400A, Q521 AO3422, Q601 NTMFS5C628NLT1G, Q711 CSD19534Q5A, Q721 CSD19538Q3A, SW201 RESET, SW202 BOOT, U101 TPS54202DDCR, U201 ESP32-WROOM-32E-N4, U301 DS3231MZ+TRL, U601 UCC27524ADR, U700 SN74LVC1G08DBVR, U710 AL8853S-13, U720 AL8853S-13, U902 LMR16020PDDAR

Commit message: pcb: place 167 components and establish four-layer routing rules
Parts:
- BT301: moved to B.Cu
- moved F904 1986.4 mm to (89.0, 85.5)
- moved F521 1937.7 mm to (81.0, 92.0)
- moved F721 1934.0 mm to (108.0, 104.5)
- moved F711 1931.3 mm to (60.0, 107.0), turned to 90 degrees
- moved F511 1883.7 mm to (133.0, 138.5)
- moved F501 1882.5 mm to (113.0, 138.5)
- moved U902 1878.6 mm to (98.0, 83.0)
- moved R908 1841.1 mm to (92.0, 90.8)
- moved R907 1836.2 mm to (89.0, 89.0)
- moved R906 1831.9 mm to (94.5, 87.0)
- moved R905 1824.7 mm to (101.8, 89.5)
- moved R904 1815.4 mm to (104.0, 96.0)
- moved D902 1795.6 mm to (106.8, 77.7)
- moved L902 1791.1 mm to (111.0, 88.5)
- moved C908 1783.0 mm to (97.0, 78.7)
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Other:
- board text added: "24V IN"
- board text added: "BOOT"
- board text added: "CR2032 / NO CHARGE"
- board text added: "FAN1"
- board text added: "FAN2"
- board text added: "FLOAT"
- board text added: "GROWBOX 24V / P1"
- board text added: "GROWBOX P1 / BOTTOM"
- board text added: "LED1"
- board text added: "LED2"
- board text added: "LED3"
- board text added: "PTC 24V"
- board text added: "PUMP 24V"
- board text added: "RESET"
- board text added: "SD"
- board text added: "SHT4x"
- board text added: "UART"
- board text removed: "/"
- board text removed: "/InputPower/"
- board text removed: "/LEDDrivers/"
- board text removed: "/MCU / ESP32/"
- board text removed: "/MCU / ESP32/Peripherals/"
- board text removed: "/Outputs/"
- board text removed: "/Outputs/Heater/"
- board text removed: "100 x 100 mm / 4 Cu layers / UNROUTED DRAFT"
- board text removed: "Candidate footprints staged outside outline"

Commit message: pcb: integrate reviewed parts and validate initial 100mm placement
Parts:
- BT301: footprint Battery:BatteryHolder_Keystone_3002_1x2032 -> Battery:BatteryHolder_MYOUNG_BS-07-A1BJ001_CR2032
- J302, J521, J601: footprint TerminalBlock_Phoenix:TerminalBlock_Phoenix_PT-1,5-2-3.5-H_1x02_P3.50mm_Horizontal -> GrowBox:TerminalBlock_DORABO_DB125-3.5_1x02_P3.50mm_Horizontal
- J501, J511: footprint TerminalBlock_Phoenix:TerminalBlock_Phoenix_PT-1,5-4-3.5-H_1x04_P3.50mm_Horizontal -> GrowBox:TerminalBlock_DORABO_DB125-3.5_1x04_P3.50mm_Horizontal
- J711, J721, J731: footprint TerminalBlock_Phoenix:TerminalBlock_Phoenix_MKDS-1,5-2-5.08_1x02_P5.08mm_Horizontal -> GrowBox:TerminalBlock_KANGNEX_WJ500V-5.08_1x02_P5.08mm_Horizontal
- J901: footprint Connector_AMASS:AMASS_XT60PW-M_1x02_P7.20mm_Horizontal -> GrowBox:AMASS_XT60PW-M_1x02_P7.20mm_Horizontal
- L101: value 10uH / Isat >= 4.5A -> 10u SRP7050TA-100M; footprint Inductor_SMD:L_Coilcraft_XAL7050-XXX -> Inductor_SMD:L_Bourns_SRP7028A_7.3x6.6mm
- R716: value 0.182 1% >=1W -> 0.18 1% 2W 50ppm
- moved J302 1.60 mm to (146.0, 120.0)
- moved BT301 1.50 mm to (115.5, 102.0)
- moved J501 1.50 mm to (109.0, 145.9)
- moved J511 1.50 mm to (129.0, 145.9)
- moved J521 1.40 mm to (54.1, 92.0)
- moved J601 1.40 mm to (54.1, 78.0)
- moved L101 1.00 mm to (90.0, 99.5)
- moved J711 0.10 mm to (60.0, 144.1)
- moved J721 0.10 mm to (77.0, 144.1)
- moved J731 0.10 mm to (94.0, 144.1)
Other:
- board text added: "GROWBOX 0.17 / BOTTOM"
- board text added: "GROWBOX 24V / 0.17"
- board text removed: "GROWBOX 24V / P1"
- board text removed: "GROWBOX P1 / BOTTOM"

Commit message: pcb: simplify passives and microSD circuitry for revision 0.18
Parts:
- removed D401, D402, D403: TPD2E2U06DCKR, Package_TO_SOT_SMD:SOT-323_SC-70
- removed R409: 0 / SD supply, Resistor_SMD:R_0805_2012Metric
- removed R701, R702: 47k, Resistor_SMD:R_0603_1608Metric
- C101: value 22u 50V -> 22u 25V X7R
- C102: value 100n / 50V -> 100n 50V X7R
- C103, C202, C301, C303, C402: value 100n / 16V -> 100n 50V X7R
- C601: value 100n / 25V -> 100n 50V X7R
- C700: value 100n 16V -> 100n 50V X7R
- L101: value 10u SRP7050TA-100M -> 10u SRP7028A-100M
- R101: value 100k 0.1% -> 100k 1%
- R102: value 22k 0.1% -> 22k 1%
- R204: value 1k / VREF only -> 1k 1%
- R205, R206: value 470 -> 1k 1%
- R305, R503, R513: value 1k -> 1k 1%
- R502, R512, R522, R602, R713, R723: value 100k -> 100k 1%
- R703: value 47k -> 47k 1%
- R712: value 1k 1% / slope tune -> 1k 1%
- R906: value 49.9k 1% -> 47k 1%
Connections:
- C401 pad 1: /MCU / ESP32/Peripherals/+3V3_SD -> +3V3
- C402 pad 1: /MCU / ESP32/Peripherals/+3V3_SD -> +3V3
- J401 pad 4: /MCU / ESP32/Peripherals/+3V3_SD -> +3V3
- R405 pad 1: /MCU / ESP32/Peripherals/+3V3_SD -> +3V3
- R406 pad 1: /MCU / ESP32/Peripherals/+3V3_SD -> +3V3
- R407 pad 1: /MCU / ESP32/Peripherals/+3V3_SD -> +3V3
- R408 pad 1: /MCU / ESP32/Peripherals/+3V3_SD -> +3V3
- R410 pad 1: /MCU / ESP32/Peripherals/+3V3_SD -> +3V3
Other:
- board text added: "GROWBOX 0.18 / BOTTOM"
- board text added: "GROWBOX 24V / 0.18"
- board text removed: "GROWBOX 0.17 / BOTTOM"
- board text removed: "GROWBOX 24V / 0.17"
