File: pcb/PCB_V1/PCB_V1.kicad_pcb (KiCad board)
At the start: 4 copper layers, 100 x 100 mm, 161 parts, among them J201 UART / 3V3 logic, J301 SHT4x / XH 2.50, J302 FLOAT / 3.5 mm, J401 Molex 104031-0811, J501 FAN1 / 3.5 mm, J511 FAN2 / 3.5 mm, J521 PUMP 24V / 6W, J601 PTC + / switched - (3.5 mm), J711 LED +/- (return isolated), J721 LED +/- (return isolated), J731 LED +/- (return isolated), J901 XT60PW-M 24V IN, Q501 AO3400A, Q511 AO3400A, Q521 AO3422, Q601 NTMFS5C628NLT1G, Q711 CSD19534Q5A, Q721 CSD19538Q3A, SW201 RESET, SW202 BOOT, U101 TPS54202DDCR, U201 ESP32-WROOM-32E-N4, U301 DS3231MZ+TRL, U601 UCC27524ADR, U700 SN74LVC1G08DBVR, U710 AL8853S-13, U720 AL8853S-13, U902 LMR16020PDDAR

Commit message: pcb: sync board values for revision 0.19
sync_board.py applied the 17 schematic value/field changes of 0.19 to
PCB_V1.kicad_pcb (C104/C105/C401, C201, C602, C716-C719, C726-C728,
R501/R511/R521, D601, F904). A before/after comparison shows no moved,
rotated or flipped part, no footprint change and no net change.
check_all.py now passes completely; docs and v19 check log updated.

Co-Authored-By: Claude Opus 5.5 <noreply@anthropic.com>
Parts:
- C104, C105, C401: value 22u / 10V X7R -> 22u / 10V X5R
- C201: value 10u / 10V -> 10u / 25V X5R
- C602: value 4.7u / 25V X7R -> 10u / 25V X5R
- C716, C717, C718, C719, C726, C727, C728: value 10u 100V X7S -> 10u 100V X7R
- D601: value SMBJ30A-E3/52 -> SMBJ26CA-E3/52
- F904: value 2A / 0451002.MRL -> 3A / 0451003.MRL
- R501, R511, R521: value 100 -> 33

Commit message: pcb: revision 0.20 cost-down with new footprints and placement
- RTC: DS3231MZ replaced by NXP PCF8563T/5 with an Epson FC-135 crystal
  (CL 12.5 pF), C304 18 pF C0G on OSCI, BAT54C supply OR (D303) and R307
  1k from the CR2032.
- Boost switches Q711/Q721: AOS AOD66923 (DPAK) on a project footprint
  that keeps the S1/2/3 G4 D5 numbering; diodes D711/D721: Vishay SS5P10
  (TO-277A).
- L101 cjiang FXL0630-100-M and L902 PROD PSPMAA0604-220M-ANP on the
  KiCad FXL0630 land.
- LED switch areas and the RTC cluster re-placed (29 parts moved);
  ERC 0, DRC 0, 340 unrouted links.
- Checks, price/JLC snapshots v20, reports, placement images and docs
  updated: USD 31.62 per board (29.52 for five boards).

Co-Authored-By: Claude Opus 5.5 <noreply@anthropic.com>
Parts:
- added C304: 18p 50V C0G, Capacitor_SMD:C_0603_1608Metric, F.Cu at (120.4, 77.9)
- added D303: BAT54C, Package_TO_SOT_SMD:SOT-23, F.Cu at (117.3, 82.0)
- added R307: 1k 1%, Resistor_SMD:R_0603_1608Metric, F.Cu at (117.3, 85.4)
- added Y301: 32.768k 12.5pF, Crystal:Crystal_SMD_3215-2Pin_3.2x1.5mm, F.Cu at (120.4, 80.9)
- D711: value STPS5H100B-TR -> SS5P10-M3/86A; footprint Package_TO_SOT_SMD:TO-252-2 -> GrowBox:Vishay_TO-277A_D_K1_A2
- D721: value STPS2H100AFY -> SS5P10-M3/86A; footprint Diode_SMD:D_SOD-128 -> GrowBox:Vishay_TO-277A_D_K1_A2
- L101: value 10u SRP7028A-100M -> 10u FXL0630-100-M; footprint Inductor_SMD:L_Bourns_SRP7028A_7.3x6.6mm -> Inductor_SMD:L_Changjiang_FXL0630
- L902: value 22u SRP1265A-220M -> 22u PSPMAA0604-220M; footprint GrowBox:L_Bourns_SRP1265A -> Inductor_SMD:L_Changjiang_FXL0630
- Q711: value CSD19534Q5A -> AOD66923; footprint GrowBox:TI_DQJ0008A_CSD19534Q5A -> GrowBox:TO-252-2_NMOS_S123_G4_D5
- Q721: value CSD19538Q3A -> AOD66923; footprint GrowBox:TI_DNH0008A_CSD19538Q3A -> GrowBox:TO-252-2_NMOS_S123_G4_D5
- U301: value DS3231MZ+TRL -> PCF8563T/5
- moved R721 11.3 mm to (122.3, 125.2), turned to 90 degrees
- moved R723 7.22 mm to (122.7, 122.4)
- moved R713 6.03 mm to (83.7, 124.3)
- moved C728 5.73 mm to (130.0, 111.9)
- moved C719 5.61 mm to (95.9, 109.7)
- moved C718 5.60 mm to (95.9, 106.2)
- moved C717 5.51 mm to (91.0, 109.7)
- moved C716 5.50 mm to (91.0, 106.2)
- moved C727 5.38 mm to (130.0, 108.4)
- moved D711 5.12 mm to (85.0, 108.3), turned to 180 degrees
- moved C726 5.06 mm to (130.0, 104.9)
- moved R722 4.77 mm to (130.0, 128.4)
- moved C723 4.62 mm to (133.1, 128.4)
- moved C721 4.57 mm to (131.8, 119.9)
- moved D721 4.21 mm to (124.0, 106.3), turned to 180 degrees
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Connections:
- C301 pad 1: +3V3 -> /MCU / ESP32/Peripherals/RTC_VDD
- D711 pad 1: unconnected-(D711-NC-Pad1) -> /LEDDrivers/LED1_OUT
- D711 pad 2: /LEDDrivers/LED1_OUT -> /LEDDrivers/LED1_SW
- U301 pad 1: unconnected-(U301-32kHz-Pad1) -> /MCU / ESP32/Peripherals/RTC_OSCI
- U301 pad 2: +3V3 -> /MCU / ESP32/Peripherals/RTC_OSCO
- U301 pad 4: unconnected-(U301-~{RST}-Pad4) -> GND
- U301 pad 5: GND -> I2C_SDA
- U301 pad 6: /MCU / ESP32/Peripherals/RTC_VBAT -> I2C_SCL
- U301 pad 7: I2C_SDA -> unconnected-(U301-CLKO-Pad7)
- U301 pad 8: I2C_SCL -> /MCU / ESP32/Peripherals/RTC_VDD
Other:
- board text added: "GROWBOX 0.20 / BOTTOM"
- board text added: "GROWBOX 24V / 0.20"
- board text removed: "GROWBOX 0.18 / BOTTOM"
- board text removed: "GROWBOX 24V / 0.18"
