File: pcb/PCB_V1/InputPower.kicad_sch (KiCad schematic)
At the start: 23 parts, among them J901 XT60PW-M 24V IN, U902 LMR16020PDDAR

Commit message: pcb: refine 24 V bias, branch protection and auxiliary supply
Parts:
- added F904: 2A / 0451002.MRL, GrowBox:Fuse_Littelfuse_451, symbol Device:Fuse
- C909: value 22u 25V X7R -> 100u 25V polymer; footprint Capacitor_SMD:C_1210_3225Metric -> Capacitor_SMD:CP_Elec_8x6.9; symbol Device:C -> Device:C_Polarized; LCSC C309062 -> C136279; MPN CL32B226KAJNNNE -> 25SVPF100M; Manufacturer Samsung -> Panasonic
- R904: value 100k 1% -> 150k 0.1%
- R905: value 6.65k 1% -> 10k 0.1%
Connections:
- net +24V: now also F904.1; no longer C905.1, C906.1, C907.1, R907.1, U902.2 (VIN)
- new net AUX_VIN: C905.1, C906.1, C907.1, F904.2, R907.1, U902.2 (VIN)
Other:
- note added: "12 V AUX: two fans, UCC27524A, TPS54202 and both AL8853 VIN pins. LMR16020, 500 kHz, 22 uH. Vout = 0.75 x (1 + 150k/10k) = 12.00 V; 0.1% divider, static range 11.74..12.26 V. Budget 1.2 A. EN divider 560k/47k retained. C909 100u polymer + C910 22u ceramic; verify startup/load steps and thermal vias. F904 and downstream fuses do not qualify fault clearing; test against the actual PSU and cables."
- note added: "External PSU: 24.0 V set point, <=25 V. D901 SMBJ26CA: 26 V standoff, 42.1 V clamp at 14.3 A (25 C). AL8853 VIN pins now use 12 V aux; their power inductors still use 24 V. F902 10 A loads; F903 7.5 A LED; F904 2 A aux. PSU must protect the unfused XT60/TVS input segment."
- note removed: "12 V AUX BUCK: fans, UCC27524A VDD, TPS54202 3.3 V input. LMR16020 500 kHz (RT 49.9k). Vout = 0.75 V x (1 + 100k/6.65k) = 12.03 V. EN divider 560k/47k: start ~14.9 V (<=17.3 V), stop ~12.9 V. L902 22 uH: ripple ~0.57 App at 25 V in. Budget 1.5 A; IC current limit 2.5-3.8 A. D902 SS36 60 V/3 A. Keep the VIN-C907/C905-GND and SW-D902 loops short; EP to GND with vias."
- note removed: "External PSU: 24.0 V set point, never above 25 V. D901 SMBJ26CA: standoff 26 V, VBR 28.9 V min, clamp 42.1 V at 14.3 A (10/1000 us) <= AL8853 43 V abs max; LMR16020 65 V. F902 10 A ATM: PTC 4.2 A (+15% cold) + pump. F903 7.5 A ATM: LED boost input 3.6 A nom / 4.5 A worst est. Holders XF-508P-B-B (<=5 mOhm). Fuse interrupt rating and cable I2t to be checked with the real PSU."
- moved on the sheet: C910
