File: pcb/PCB_V1/InputPower.kicad_sch (KiCad schematic)
At the start: 24 parts, among them J901 XT60PW-M 24V IN, U902 LMR16020PDDAR

Commit message: pcb: revision 0.16 - drop redundant F903, restore CH1 inductor margin, clean DRC and docs
Schematic/board:
- remove F903 (7.5 A LED blade fuse): F711 6.3 A and F721 3 A already fuse
  each LED channel and F903 had the smallest margin; TP903/#FLG0603 removed,
  LED channel fuses and C710 now sit on +24V
- L711 back to Bourns SRP1770TA-470M with R715 0.027 ohm: CH1 OCP headroom
  3.17 A (was 0.34 A), worst-case winding loss 0.77 W (was 1.22 W)
- ESP32 footprint GrowBox:ESP32-WROOM-32E_NoVias without the 12 in-pad
  0.2 mm vias: DRC now 0 violations (only unrouted connections remain)
- 167 components; ERC 0/0

Checks and docs:
- new check_all.py runs ERC, netlist/board verification, sizing reports,
  BOM export and DRC; --write refreshes review/*_v16 and sheet images
- verify_netlist.py, verify_board.py, analyze_*.py updated for 0.16
- REDESIGN_24V.md -> DESIGN.md (current design only), new CHANGELOG.md,
  superseded 12 V documents in PCB_V1/history/, older reports in
  review/history/, README files rewritten as entry points
- cost estimation paused; v0.15 price audit kept as history

Co-Authored-By: Claude Opus 5.5 <noreply@anthropic.com>
Parts:
- removed F903: 7.5A mini blade (ATM), GrowBox:Fuseholder_Blade_Mini_XFCN_XF-508P, symbol Device:Fuse
- removed TP903: +24V_LED, TestPoint:TestPoint_Pad_D2.0mm, symbol Connector:TestPoint
Other:
- note added: "External PSU: 24.0 V set point, <=25 V. D901 SMBJ26CA: 26 V standoff, 42.1 V clamp at 14.3 A (25 C).\nAL8853 VIN pins now use 12 V aux; their power inductors still use 24 V.\nF902 10 A loads; LED channels fused individually on sheet 07 (F711 6.3 A, F721 3 A); F904 2 A aux. PSU must protect the unfused XT60/TVS input segment."
- note removed: "External PSU: 24.0 V set point, <=25 V. D901 SMBJ26CA: 26 V standoff, 42.1 V clamp at 14.3 A (25 C). AL8853 VIN pins now use 12 V aux; their power inductors still use 24 V. F902 10 A loads; F903 7.5 A LED; F904 2 A aux. PSU must protect the unfused XT60/TVS input segment."
- title: 06 - 24 V input, branch fuses, 12 V auxiliary buck -> 06 - 24 V input, fuses, 12 V auxiliary buck
