File: pcb/PCB_V1/InputPower.kicad_sch (KiCad schematic)
At the start: 22 parts, among them J901 XT60PW-M 24V IN, U902 LMR16020PDDAR

Commit message: pcb: integrate reviewed parts and validate initial 100mm placement
Parts:
- C902: LCSC (none) -> C40708; MPN (none) -> CL32B105KBHNNNE; Manufacturer (none) -> Samsung Electro-Mechanics
- J901: footprint Connector_AMASS:AMASS_XT60PW-M_1x02_P7.20mm_Horizontal -> GrowBox:AMASS_XT60PW-M_1x02_P7.20mm_Horizontal
- R904: LCSC (none) -> C326734; MPN (none) -> RT0603BRD07150KL; Manufacturer (none) -> Yageo
- R905: LCSC (none) -> C95204; MPN (none) -> RT0603BRD0710KL; Manufacturer (none) -> Yageo
- R906: LCSC (none) -> C23184; MPN (none) -> 0603WAF4992T5E; Manufacturer (none) -> UNI-ROYAL
- R907: LCSC (none) -> C23203; MPN (none) -> 0603WAF5603T5E; Manufacturer (none) -> UNI-ROYAL
- R908: LCSC (none) -> C105579; MPN (none) -> RC0603FR-0747KL; Manufacturer (none) -> Yageo
Changed lines of the file:
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@@
 	(title_block
 		(title "06 - 24 V input, fuses, 12 V auxiliary buck")
-		(date "2026-09-27")
-		(rev "0.16-DRAFT")
+		(date "2026-09-28")
+		(rev "0.17-DRAFT")
 		(company "GrowBox controller")
 		(comment 1 "Engineering draft; startup, thermal and fault qualification pending")
@@
 			)
 		)
-		(property "Footprint" "Connector_AMASS:AMASS_XT60PW-M_1x02_P7.20mm_Horizontal"
+		(property "Footprint" "GrowBox:AMASS_XT60PW-M_1x02_P7.20mm_Horizontal"
 			(at 38.1 50.8 0)
 			(effects
@@
 			)
 		)
-		(property "Datasheet" ""
+		(property "Datasheet" "https://product.samsungsem.com/mlcc/CL32B105KBHNNN.do"
 			(at 101.6 50.8 0)
 			(effects
@@
 					(unit 1)
 				)
+			)
+		)
+		(property "Manufacturer" "Samsung Electro-Mechanics"
+			(at 101.6 50.8 0)
+			(effects
+				(font
+					(size 1 1)
+				)
+				(hide yes)
+				(justify left)
+			)
+		)
+		(property "MPN" "CL32B105KBHNNNE"
+			(at 101.6 50.8 0)
+			(effects
+				(font
+					(size 1 1)
+				)
+				(hide yes)
+				(justify left)
+			)
+		)
+		(property "LCSC" "C40708"
+			(at 101.6 50.8 0)
+			(effects
+				(font
+					(size 1 1)
+				)
+				(hide yes)
+				(justify left)
 			)
 		)
@@
 			)
 		)
+		(property "Manufacturer" "UNI-ROYAL"
+			(at 91.44 111.76 0)
+			(effects
+				(font
+					(size 1 1)
+				)
+				(hide yes)
+				(justify left)
+			)
+		)
+		(property "MPN" "0603WAF5603T5E"
+			(at 91.44 111.76 0)
+			(effects
+				(font
+					(size 1 1)
+				)
+				(hide yes)
+				(justify left)
+			)
+		)
+		(property "LCSC" "C23203"
+			(at 91.44 111.76 0)
+			(effects
+				(font
+					(size 1 1)
+				)
+				(hide yes)
+				(justify left)
+			)
+		)
 	)
 	(wire
@@
 			)
 		)
+		(property "Manufacturer" "Yageo"
+			(at 91.44 149.86 0)
+			(effects
+				(font
+					(size 1 1)
+				)
+				(hide yes)
+				(justify left)
+			)
+		)
+		(property "MPN" "RC0603FR-0747KL"
+			(at 91.44 149.86 0)
+			(effects
+				(font
+					(size 1 1)
+				)
+				(hide yes)
+				(justify left)
+			)
+		)
+		(property "LCSC" "C105579"
+			(at 91.44 149.86 0)
+			(effects
+				(font
+					(size 1 1)
+				)
+				(hide yes)
+				(justify left)
+			)
+		)
 	)
 	(wire
@@
 			)
 		)
+		(property "Manufacturer" "UNI-ROYAL"
+			(at 109.22 152.4 0)
+			(effects
+				(font
+					(size 1 1)
+				)
+				(hide yes)
+				(justify left)
+			)
+		)
+		(property "MPN" "0603WAF4992T5E"
+			(at 109.22 152.4 0)
+			(effects
+				(font
+					(size 1 1)
+				)
+				(hide yes)
+				(justify left)
+			)
+		)
+		(property "LCSC" "C23184"
+			(at 109.22 152.4 0)
+			(effects
+				(font
+					(size 1 1)
+				)
+				(hide yes)
+				(justify left)
+			)
+		)
 	)
 	(wire
@@
 			)
 		)
+		(property "Manufacturer" "Yageo"
+			(at 220.98 114.3 0)
+			(effects
+				(font
+					(size 1 1)
+				)
+				(hide yes)
+				(justify left)
+			)
+		)
+		(property "MPN" "RT0603BRD07150KL"
+			(at 220.98 114.3 0)
+			(effects
+				(font
+					(size 1 1)
+				)
+				(hide yes)
+				(justify left)
+			)
+		)
+		(property "LCSC" "C326734"
+			(at 220.98 114.3 0)
+			(effects
+				(font
+					(size 1 1)
+				)
+				(hide yes)
+				(justify left)
+			)
+		)
 	)
 	(wire
@@
 			)
 		)
+		(property "Manufacturer" "Yageo"
+			(at 220.98 152.4 0)
+			(effects
+				(font
+					(size 1 1)
+				)
+				(hide yes)
+				(justify left)
+			)
+		)
+		(property "MPN" "RT0603BRD0710KL"
+			(at 220.98 152.4 0)
+			(effects
+				(font
+					(size 1 1)
+				)
+				(hide yes)
+				(justify left)
+			)
+		)
+		(property "LCSC" "C95204"
+			(at 220.98 152.4 0)
+			(effects
+				(font
+					(size 1 1)
+				)
+				(hide yes)
+				(justify left)
+			)
+		)

Commit message: pcb: simplify passives and microSD circuitry for revision 0.18
Parts:
- R906: value 49.9k 1% -> 47k 1%; LCSC C23184 -> C105579; MPN 0603WAF4992T5E -> RC0603FR-0747KL; Manufacturer UNI-ROYAL -> Yageo
Other:
- note added: "12 V AUX: two fans, UCC27524A, TPS54202 and both AL8853 VIN pins. LMR16020, ~526 kHz (RT 47k), 22 uH. Vout = 0.75 x (1 + 150k/10k) = 12.00 V; 0.1% divider, static range 11.74..12.26 V. Budget 1.2 A. EN divider 560k/47k retained. C909 100u polymer + C910 22u ceramic; verify startup/load steps and thermal vias. F904 and downstream fuses do not qualify fault clearing; test against the actual PSU and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"
- note added: "External PSU: 24.0 V set point, <=25 V. D901 SMBJ26CA: 26 V standoff, 42.1 V clamp at 14.3 A (25 C). AL8853 VIN pins now use 12 V aux; their power inductors still use 24 V. F902 10 A loads; LED channels fused individually on sheet 07 (F711 6.3 A, F721 3 A); F904 2 A aux. PSU must protect the unfused XT60/TVS input segment."
- note removed: "12 V AUX: two fans, UCC27524A, TPS54202 and both AL8853 VIN pins. LMR16020, 500 kHz, 22 uH. Vout = 0.75 x (1 + 150k/10k) = 12.00 V; 0.1% divider, static range 11.74..12.26 V. Budget 1.2 A. EN divider 560k/47k retained. C909 100u polymer + C910 22u ceramic; verify startup/load steps and thermal vias. F904 and downstream fuses do not qualify fault clearing; test against the actual PSU and cables."
- note removed: "External PSU: 24.0 V set point, <=25 V. D901 SMBJ26CA: 26 V standoff, 42.1 V clamp at 14.3 A (25 C).\nAL8853 VIN pins now use 12 V aux; their power inductors still use 24 V.\nF902 10 A loads; LED channels fused individually on sheet 07 (F711 6.3 A, F721 3 A); F904 2 A aux. PSU must protect the unfused XT60/TVS input segment."
Changed lines of the file:
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@@
 	(title_block
 		(title "06 - 24 V input, fuses, 12 V auxiliary buck")
-		(date "2026-09-28")
-		(rev "0.17-DRAFT")
+		(date "2026-09-29")
+		(rev "0.18-DRAFT")
 		(company "GrowBox controller")
-		(comment 1 "Engineering draft; startup, thermal and fault qualification pending")
+		(comment 1 "Simplified prototype; unrouted; hardware qualification pending")
 	)
 	(symbol
@@
 			)
 		)
-		(property "Value" "49.9k 1%"
+		(property "Value" "47k 1%"
 			(at 113.03 153.67 0)
 			(effects
@@
 			)
 		)
-		(property "Manufacturer" "UNI-ROYAL"
+		(property "Manufacturer" "Yageo"
 			(at 109.22 152.4 0)
 			(effects
@@
 			)
 		)
-		(property "MPN" "0603WAF4992T5E"
+		(property "MPN" "RC0603FR-0747KL"
 			(at 109.22 152.4 0)
 			(effects
@@
 			)
 		)
-		(property "LCSC" "C23184"
+		(property "LCSC" "C105579"
 			(at 109.22 152.4 0)
 			(effects
@@
 		)
 	)
-	(text "External PSU: 24.0 V set point, <=25 V. D901 SMBJ26CA: 26 V standoff, 42.1 V clamp at 14.3 A (25 C).\\nAL8853 VIN pins now use 12 V aux; their power inductors still use 24 V.\\nF902 10 A loads; LED channels fused individually on sheet 07 (F711 6.3 A, F721 3 A); F904 2 A aux. PSU must protect the unfused XT60/TVS input segment."
+	(text "External PSU: 24.0 V set point, <=25 V. D901 SMBJ26CA: 26 V standoff, 42.1 V clamp at 14.3 A (25 C).\nAL8853 VIN pins now use 12 V aux; their power inductors still use 24 V.\nF902 10 A loads; LED channels fused individually on sheet 07 (F711 6.3 A, F721 3 A); F904 2 A aux. PSU must protect the unfused XT60/TVS input segment."
 		(exclude_from_sim no)
 		(at 20.32 83.82 0)
@@
 		)
 	)
-	(text "12 V AUX: two fans, UCC27524A, TPS54202 and both AL8853 VIN pins. LMR16020, 500 kHz, 22 uH.\nVout = 0.75 x (1 + 150k/10k) = 12.00 V; 0.1% divider, static range 11.74..12.26 V. Budget 1.2 A.\nEN divider 560k/47k retained. C909 100u polymer + C910 22u ceramic; verify startup/load steps and thermal vias.\nF904 and downstream fuses do not qualify fault clearing; test against the actual PSU and cables."
+	(text "12 V AUX: two fans, UCC27524A, TPS54202 and both AL8853 VIN pins. LMR16020, ~526 kHz (RT 47k), 22 uH.\nVout = 0.75 x (1 + 150k/10k) = 12.00 V; 0.1% divider, static range 11.74..12.26 V. Budget 1.2 A.\nEN divider 560k/47k retained. C909 100u polymer + C910 22u ceramic; verify startup/load steps and thermal vias.\nF904 and downstream fuses do not qualify fault clearing; test against the actual PSU and cables."
 		(exclude_from_sim no)
 		(at 20.32 172.72 0)
