File: pcb/PCB_V1/MCU.kicad_sch (KiCad schematic)
At the start: 19 parts, among them J201 UART / 3V3 logic, SW201 RESET, SW202 BOOT, U201 ESP32-WROOM-32E-N4

Commit message: pcb: revision 0.16 - drop redundant F903, restore CH1 inductor margin, clean DRC and docs
Schematic/board:
- remove F903 (7.5 A LED blade fuse): F711 6.3 A and F721 3 A already fuse
  each LED channel and F903 had the smallest margin; TP903/#FLG0603 removed,
  LED channel fuses and C710 now sit on +24V
- L711 back to Bourns SRP1770TA-470M with R715 0.027 ohm: CH1 OCP headroom
  3.17 A (was 0.34 A), worst-case winding loss 0.77 W (was 1.22 W)
- ESP32 footprint GrowBox:ESP32-WROOM-32E_NoVias without the 12 in-pad
  0.2 mm vias: DRC now 0 violations (only unrouted connections remain)
- 167 components; ERC 0/0

Checks and docs:
- new check_all.py runs ERC, netlist/board verification, sizing reports,
  BOM export and DRC; --write refreshes review/*_v16 and sheet images
- verify_netlist.py, verify_board.py, analyze_*.py updated for 0.16
- REDESIGN_24V.md -> DESIGN.md (current design only), new CHANGELOG.md,
  superseded 12 V documents in PCB_V1/history/, older reports in
  review/history/, README files rewritten as entry points
- cost estimation paused; v0.15 price audit kept as history

Co-Authored-By: Claude Opus 5.5 <noreply@anthropic.com>
Parts:
- U201: footprint RF_Module:ESP32-WROOM-32E -> GrowBox:ESP32-WROOM-32E_NoVias; LCSC (none) -> C701341; MPN (none) -> ESP32-WROOM-32E-N4; Manufacturer (none) -> Espressif
Changed lines of the file:
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@@
 		(title "02 - ESP32 and programming")
 		(date "2026-09-26")
-		(rev "0.4-DRAFT")
+		(rev "0.16-DRAFT")
 		(company "GrowBox controller")
 		(comment 1 "Draft: input protection and LED drivers pending")
@@
 			)
 		)
-		(property "Footprint" "RF_Module:ESP32-WROOM-32E"
+		(property "Footprint" "GrowBox:ESP32-WROOM-32E_NoVias"
 			(at 101.6 81.28 0)
 			(hide yes)
@@
 			)
 		)
+		(property "LCSC" "C701341"
+			(at 101.6 81.28 0)
+			(effects
+				(font
+					(size 1 1)
+				)
+				(hide yes)
+				(justify left)
+			)
+		)
+		(property "MPN" "ESP32-WROOM-32E-N4"
+			(at 101.6 81.28 0)
+			(effects
+				(font
+					(size 1 1)
+				)
+				(hide yes)
+				(justify left)
+			)
+		)
+		(property "Manufacturer" "Espressif"
+			(at 101.6 81.28 0)
+			(effects
+				(font
+					(size 1 1)
+				)
+				(hide yes)
+				(justify left)
+			)
+		)
