File: pcb/PCB_V1/MCU.kicad_sch (KiCad schematic)
At the start: 19 parts, among them J201 UART / 3V3 logic, SW201 RESET, SW202 BOOT, U201 ESP32-WROOM-32E-N4

Commit message: pcb: simplify passives and microSD circuitry for revision 0.18
Parts:
- C202: value 100n / 16V -> 100n 50V X7R; LCSC (none) -> C1591; MPN (none) -> CL10B104KB8NNNC; Manufacturer (none) -> Samsung
- R204: value 1k / VREF only -> 1k 1%; LCSC (none) -> C21190; MPN (none) -> 0603WAF1001T5E; Manufacturer (none) -> UNI-ROYAL
- R205, R206: value 470 -> 1k 1%; LCSC (none) -> C21190; MPN (none) -> 0603WAF1001T5E; Manufacturer (none) -> UNI-ROYAL
Other:
- note added: "FAN PWM: 25 kHz, inverted by open-drain MOSFET. Reset -> fan full speed. GPIO34/35: input only. GPIO12 held LOW for 3.3 V flash. PCB: antenna keepout on all copper layers per module datasheet. Pump / heater default OFF. R211/R212 hold LIGHT_PWM/ENABLE low."
- note added: "UART: adapter TX -> J201.4; RX -> J201.3; common GND. J201.2 = reference only through 1k; leave open on a simple adapter. Power board from its own 24 V source. No 5 V UART signals. Hold BOOT, pulse RESET, release BOOT to flash. EN / IO0: manual buttons or open-drain programmer outputs."
- note removed: "FAN PWM: 25 kHz, inverted by open-drain MOSFET. Reset -> fan full speed. GPIO34/35: input only. GPIO12 held LOW for 3.3 V flash. PCB: antenna keepout on all copper layers per module datasheet. Pump / heater default OFF. LED drivers not yet implemented."
- note removed: "UART: adapter TX -> J201.4; RX -> J201.3; common GND.\nJ201.2 = reference only through 1k; leave open on a simple adapter.\nPower board from its own 24 V source. No 5 V UART signals.\nHold BOOT, pulse RESET, release BOOT to flash.\nEN / IO0: manual buttons or open-drain programmer outputs."
Changed lines of the file:
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@@
 	(title_block
 		(title "02 - ESP32 and programming")
-		(date "2026-09-28")
-		(rev "0.17-DRAFT")
+		(date "2026-09-29")
+		(rev "0.18-DRAFT")
 		(company "GrowBox controller")
-		(comment 1 "Draft: input protection and LED drivers pending")
+		(comment 1 "Simplified prototype; unrouted; hardware qualification pending")
 	)
-	(text "UART: adapter TX -> J201.4; RX -> J201.3; common GND.\\nJ201.2 = reference only through 1k; leave open on a simple adapter.\\nPower board from its own 24 V source. No 5 V UART signals.\\nHold BOOT, pulse RESET, release BOOT to flash.\\nEN / IO0: manual buttons or open-drain programmer outputs."
+	(text "UART: adapter TX -> J201.4; RX -> J201.3; common GND.\nJ201.2 = reference only through 1k; leave open on a simple adapter.\nPower board from its own 24 V source. No 5 V UART signals.\nHold BOOT, pulse RESET, release BOOT to flash.\nEN / IO0: manual buttons or open-drain programmer outputs."
 		(exclude_from_sim no)
 		(at 177.8 121.92 0)
@@
 		)
 	)
-	(text "FAN PWM: 25 kHz, inverted by open-drain MOSFET. Reset -> fan full speed.\nGPIO34/35: input only. GPIO12 held LOW for 3.3 V flash.\nPCB: antenna keepout on all copper layers per module datasheet.\nPump / heater default OFF. LED drivers not yet implemented."
+	(text "FAN PWM: 25 kHz, inverted by open-drain MOSFET. Reset -> fan full speed.\nGPIO34/35: input only. GPIO12 held LOW for 3.3 V flash.\nPCB: antenna keepout on all copper layers per module datasheet.\nPump / heater default OFF. R211/R212 hold LIGHT_PWM/ENABLE low."
 		(exclude_from_sim no)
 		(at 20.32 180.34 0)
@@
 			)
 		)
-		(property "Value" "1k / VREF only"
+		(property "Value" "1k 1%"
 			(at 185.88 74.93 0)
 			(show_name no)
@@
 			)
 		)
+		(property "Manufacturer" "UNI-ROYAL"
+			(at 182.88 73.66 0)
+			(hide yes)
+			(show_name no)
+			(do_not_autoplace no)
+			(effects
+				(font
+					(size 1 1)
+				)
+				(justify left)
+			)
+		)
+		(property "MPN" "0603WAF1001T5E"
+			(at 182.88 73.66 0)
+			(hide yes)
+			(show_name no)
+			(do_not_autoplace no)
+			(effects
+				(font
+					(size 1 1)
+				)
+				(justify left)
+			)
+		)
+		(property "LCSC" "C21190"
+			(at 182.88 73.66 0)
+			(hide yes)
+			(show_name no)
+			(do_not_autoplace no)
+			(effects
+				(font
+					(size 1 1)
+				)
+				(justify left)
+			)
+		)
 	)
 	(symbol
@@
 			)
 		)
-		(property "Value" "470"
+		(property "Value" "1k 1%"
 			(at 185.88 105.41 0)
 			(show_name no)
@@
 			)
 		)
+		(property "Manufacturer" "UNI-ROYAL"
+			(at 182.88 104.14 0)
+			(hide yes)
+			(show_name no)
+			(do_not_autoplace no)
+			(effects
+				(font
+					(size 1 1)
+				)
+				(justify left)
+			)
+		)
+		(property "MPN" "0603WAF1001T5E"
+			(at 182.88 104.14 0)
+			(hide yes)
+			(show_name no)
+			(do_not_autoplace no)
+			(effects
+				(font
+					(size 1 1)
+				)
+				(justify left)
+			)
+		)
+		(property "LCSC" "C21190"
+			(at 182.88 104.14 0)
+			(hide yes)
+			(show_name no)
+			(do_not_autoplace no)
+			(effects
+				(font
+					(size 1 1)
+				)
+				(justify left)
+			)
+		)
 	)
 	(symbol
@@
 			)
 		)
-		(property "Value" "100n / 16V"
+		(property "Value" "100n 50V X7R"
 			(at 58.88 46.99 0)
 			(show_name no)
@@
 			)
 		)
+		(property "Manufacturer" "Samsung"
+			(at 55.88 45.72 0)
+			(hide yes)
+			(show_name no)
+			(do_not_autoplace no)
+			(effects
+				(font
+					(size 1 1)
+				)
+				(justify left)
+			)
+		)
+		(property "MPN" "CL10B104KB8NNNC"
+			(at 55.88 45.72 0)
+			(hide yes)
+			(show_name no)
+			(do_not_autoplace no)
+			(effects
+				(font
+					(size 1 1)
+				)
+				(justify left)
+			)
+		)
+		(property "LCSC" "C1591"
+			(at 55.88 45.72 0)
+			(hide yes)
+			(show_name no)
+			(do_not_autoplace no)
+			(effects
+				(font
+					(size 1 1)
+				)
+				(justify left)
+			)
+		)
 	)
 	(symbol
@@
 			)
 		)
-		(property "Value" "470"
+		(property "Value" "1k 1%"
 			(at 239.22 105.41 0)
 			(show_name no)
@@
 			)
 		)
+		(property "Manufacturer" "UNI-ROYAL"
+			(at 236.22 104.14 0)
+			(hide yes)
+			(show_name no)
+			(do_not_autoplace no)
+			(effects
+				(font
+					(size 1 1)
+				)
+				(justify left)
+			)
+		)
+		(property "MPN" "0603WAF1001T5E"
+			(at 236.22 104.14 0)
+			(hide yes)
+			(show_name no)
+			(do_not_autoplace no)
+			(effects
+				(font
+					(size 1 1)
+				)
+				(justify left)
+			)
+		)
+		(property "LCSC" "C21190"
+			(at 236.22 104.14 0)
+			(hide yes)
+			(show_name no)
+			(do_not_autoplace no)
+			(effects
+				(font
+					(size 1 1)
+				)
+				(justify left)
+			)
+		)
