File: pcb/cheap-version/InputPower.kicad_sch (KiCad schematic)
At the start: 22 parts, among them J901 XT60PW-M 24V IN, U902 LMR16020PDDAR

Commit message: cheap-version: schematic substitutions from stock parts
tools/make_cheap1.py generates the cheap-1 sheets from the PCB_V1 0.22 baseline:
ST1S14 for LMR16020 (RT resistor removed, EN/FB divider recalculated), IRS4427S and
IRL2505 for the heater, BSC146N10LS5 for the LED boost switches, SS56 diodes,
KF301/FS1.5/KF2510/XH connectors, stock resistors and capacitors (Source field =
stock:<id>). J901 XT60 is replaced by a screw terminal as decided. U101 TPS54202 and
D711/D721 SS5P10 are kept because datasheets for ST1S10 and SBRT15U100SP5 were not
available. ERC: 0 errors (one warning: footprint for the DTMSS-27 inductor pending);
netdiff against PCB_V1: no connectivity differences among untouched pins.

Co-Authored-By: Claude Sonnet 5.5 <noreply@anthropic.com>
Parts:
- removed R906: 47k 1%, Resistor_SMD:R_0603_1608Metric, symbol Device:R
- removed U902: LMR16020PDDAR, Package_SO:SOIC-8-1EP_3.9x4.9mm_P1.27mm_EP2.95x4.9mm_Mask2.71x3.4mm, symbol GrowBox:LMR16020
- added U902: ST1S14PHR, Package_SO:SOIC-8-1EP_3.9x4.9mm_P1.27mm_EP2.41x3.3mm, symbol Regulator_Switching:ST1S14PHR
- C901: value 220u / 50V -> 470u / 63V; footprint Capacitor_SMD:CP_Elec_10x10.5 -> Capacitor_SMD:CP_Elec_16x17.5; LCSC C178549 -> C178728; MPN EEEFK1H221P -> EEVFK1J471M; Source (none) -> stock:13
- C902: value 1u / 50V X7R -> 2.2u 50V X7R; footprint Capacitor_SMD:C_1210_3225Metric -> Capacitor_SMD:C_1206_3216Metric; LCSC C40708 -> (none); MPN CL32B105KBHNNNE -> 12065C225KATM-HW; Manufacturer Samsung Electro-Mechanics -> KYOCERA AVX; Source (none) -> stock:3
- C905, C906: LCSC C386166 -> C92388; MPN UMK325AB7106KMHP -> CL32B106KBJNNNE; Manufacturer Taiyo Yuden -> Samsung Electro-Mechanics; Source (none) -> stock:47
- C907, C908: Source (none) -> stock:54
- C909: value 100u 25V polymer -> 820u 25V; footprint Capacitor_SMD:CP_Elec_8x6.9 -> Capacitor_SMD:CP_Elec_10x10.5; LCSC C136279 -> C178593; MPN 25SVPF100M -> EEEFT1E821AP; Source (none) -> stock:14
- C910: value 22u 25V X7R -> 10u 35V X5R; LCSC C309062 -> C2980162; MPN CL32B226KAJNNNE -> CL32A106KLULNNE; Manufacturer Samsung -> Samsung Electro-Mechanics; Source (none) -> stock:6
- D902: value SS36-E3/57T -> SS56; LCSC C35722 -> (none); MPN SS36-E3/57T -> SS56; Manufacturer Vishay -> (none); Source (none) -> stock:20
- J901: value XT60PW-M 24V IN -> 24V IN (KF301-5.0-2P); footprint GrowBox:AMASS_XT60PW-M_1x02_P7.20mm_Horizontal -> TerminalBlock_Phoenix:TerminalBlock_Phoenix_MKDS-1,5-2_1x02_P5.00mm_Horizontal; LCSC C98732 -> (none); MPN XT60PW-M -> KF301-5.0-2P; Manufacturer Changzhou Amass -> (none); Source (none) -> stock:93
- R904: value 150k 0.1% -> 88.7k 0.1%; LCSC C326734 -> (none); MPN RT0603BRD07150KL -> RT0603BRD0788K7L; Source (none) -> buy: verify MPN on LCSC
- R907: value 560k 1% -> 470k 1%; LCSC C23203 -> (none); MPN 0603WAF5603T5E -> 0603WAF4703T5E
- R908: footprint Resistor_SMD:R_0603_1608Metric -> Resistor_SMD:R_1206_3216Metric; LCSC C105579 -> (none); MPN RC0603FR-0747KL -> (none); Manufacturer Yageo -> (none); Source (none) -> stock:61
Connections:
- net AUX_VIN: now also U902.7 (VIN)
- net BUCK12_BOOT: now also U902.1 (BOOT)
- net BUCK12_EN: now also U902.5 (EN2)
- net BUCK12_FB: now also U902.4 (FB)
- net BUCK12_SW: now also U902.8 (SW)
- net GND: now also U902.3 (~{EN1}), U902.6 (GND), U902.9 (PADGND)
