File: pcb/cheap-version/InputPower.kicad_sch (KiCad schematic)
At the start: 21 parts, among them J901 24V IN (KF301-5.0-2P), U902 ST1S14PHR

Commit message: Turn 24V input terminal toward board edge preserving polarity
Parts:
- J901: footprint TerminalBlock_Phoenix:TerminalBlock_Phoenix_MKDS-1,5-2_1x02_P5.00mm_Horizontal -> GrowBox:TerminalBlock_KF301_1x02_P5.00mm_Horizontal_Input
Changed lines of the file:
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@@
 			)
 		)
-		(property "Footprint" "TerminalBlock_Phoenix:TerminalBlock_Phoenix_MKDS-1,5-2_1x02_P5.00mm_Horizontal"
+		(property "Footprint" "GrowBox:TerminalBlock_KF301_1x02_P5.00mm_Horizontal_Input"
 			(at 38.1 50.8 0)
 			(effects
