File: pcb/cheap-version/InputPower.kicad_sch (KiCad schematic)
At the start: 21 parts, among them J901 24V IN (KF301-5.0-2P), U902 ST1S14PHR

Commit message: cheap-version: local HF bypass C911 at the ST1S14 VIN pin
The route from the input capacitors C905/C906 to U902 pin 7 is about 15 mm
of 0.6 mm copper with two vias, half of it on B.Cu above the +3V3 flood
instead of GND (hot-loop inductance 15 nH or more). C911, 100 nF 0603 from
stock (a copy of C907), now sits on the bottom side right under pins 6/7:
AUX_VIN pad on the existing B.Cu track, GND via beside it into In1, a
second AUX_VIN via next to pin 7 closes the loop (about 5 nH). Schematic
(generator), board (tools/add_c911.py), BOM (161 parts, 94 from stock),
DRC 0 / check_fab 0 FAIL.

Co-Authored-By: Claude Sonnet 5.5 <noreply@anthropic.com>
Parts:
- added C911: 100n 50V X7R, Capacitor_SMD:C_0603_1608Metric, symbol Device:C
Connections:
- net AUX_VIN: now also C911.1
- net GND: now also C911.2
Changed lines of the file:
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@@
+		)
+	)
+	(symbol
+		(lib_id "Device:C")
+		(at 86.36 124.46 0)
+		(unit 1)
+		(exclude_from_sim no)
+		(in_bom yes)
+		(on_board yes)
+		(dnp no)
+		(property "Reference" "C911"
+			(at 90.17 123.19 0)
+			(effects
+				(font
+					(size 1 1)
+				)
+				(justify left)
+			)
+		)
+		(property "Value" "100n 50V X7R"
+			(at 90.17 125.73 0)
+			(effects
+				(font
+					(size 1 1)
+				)
+				(justify left)
+			)
+		)
+		(property "Footprint" "Capacitor_SMD:C_0603_1608Metric"
+			(at 86.36 124.46 0)
+			(effects
+				(font
+					(size 1 1)
+				)
+				(hide yes)
+				(justify left)
+			)
+		)
+		(property "Datasheet" ""
+			(at 86.36 124.46 0)
+			(effects
+				(font
+					(size 1 1)
+				)
+				(hide yes)
+				(justify left)
+			)
+		)
+		(property "Manufacturer" "Samsung"
+			(at 86.36 124.46 0)
+			(effects
+				(font
+					(size 1 1)
+				)
+				(hide yes)
+				(justify left)
+			)
+		)
+		(property "MPN" "CL10B104KB8NNNC"
+			(at 86.36 124.46 0)
+			(effects
+				(font
+					(size 1 1)
+				)
+				(hide yes)
+				(justify left)
+			)
+		)
+		(property "LCSC" "C1591"
+			(at 86.36 124.46 0)
+			(effects
+				(font
+					(size 1 1)
+				)
+				(hide yes)
+				(justify left)
+			)
+		)
+		(property "Source" "stock:54"
+			(at 86.36 124.46 0)
+			(effects
+				(font
+					(size 1 1)
+				)
+				(hide yes)
+				(justify left)
+			)
+		)
+		(pin "1"
+		)
+		(pin "2"
+		)
+		(instances
+			(project "cheap-version"
+				(path "/7c30e6d8-4e60-4647-b4d3-d05e639d6467/13f6ec92-6d25-5cb3-b953-f0854e3d007b"
+					(reference "C911")
+					(unit 1)
+				)
+			)
+		)
+	)
+	(wire
+		(pts
+			(xy 86.36 120.65) (xy 86.36 118.11)
+		)
+		(stroke
+			(width 0)
+			(type default)
+		)
+	)
+	(label "AUX_VIN"
+		(at 86.36 118.11 90)
+		(effects
+			(font
+				(size 1.0 1.0)
+			)
+			(justify left)
+		)
+	)
+	(wire
+		(pts
+			(xy 86.36 128.27) (xy 86.36 130.81)
+		)
+		(stroke
+			(width 0)
+			(type default)
+		)
+	)
+	(global_label "GND"
+		(shape bidirectional)
+		(at 86.36 130.81 270)
+		(effects
+			(font
+				(size 1.0 1.0)
+			)
+			(justify right)
 		)
 	)
