File: pcb/cheap-version/InputPower.kicad_sch (KiCad schematic)
At the start: 22 parts, among them J901 24V IN (KF301-5.0-2P), U902 ST1S14PHR

Commit message: Verify cheap-version purchase parts and require complete release checks
Parts:
- R904: LCSC (none) -> C728599; Source buy: verify MPN on LCSC -> buy
- R907: LCSC (none) -> C23178; Source (none) -> buy
Changed lines of the file:
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@@
 			)
 		)
-		(property "LCSC" ""
+		(property "LCSC" "C23178"
+			(at 91.44 111.76 0)
+			(effects
+				(font
+					(size 1 1)
+				)
+				(hide yes)
+				(justify left)
+			)
+		)
+		(property "Source" "buy"
 			(at 91.44 111.76 0)
 			(effects
@@
 			)
 		)
-		(property "LCSC" ""
+		(property "LCSC" "C728599"
 			(at 220.98 114.3 0)
 			(effects
@@
 			)
 		)
-		(property "Source" "buy: verify MPN on LCSC"
+		(property "Source" "buy"
 			(at 220.98 114.3 0)
 			(effects
