File: pcb/cheap-version/MCU.kicad_sch (KiCad schematic)
At the start: 19 parts, among them J201 UART / 3V3 logic, SW201 RESET, SW202 BOOT, U201 ESP32-WROOM-32E-N4

Commit message: cheap-version: schematic substitutions from stock parts
tools/make_cheap1.py generates the cheap-1 sheets from the PCB_V1 0.22 baseline:
ST1S14 for LMR16020 (RT resistor removed, EN/FB divider recalculated), IRS4427S and
IRL2505 for the heater, BSC146N10LS5 for the LED boost switches, SS56 diodes,
KF301/FS1.5/KF2510/XH connectors, stock resistors and capacitors (Source field =
stock:<id>). J901 XT60 is replaced by a screw terminal as decided. U101 TPS54202 and
D711/D721 SS5P10 are kept because datasheets for ST1S10 and SBRT15U100SP5 were not
available. ERC: 0 errors (one warning: footprint for the DTMSS-27 inductor pending);
netdiff against PCB_V1: no connectivity differences among untouched pins.

Co-Authored-By: Claude Sonnet 5.5 <noreply@anthropic.com>
Parts:
- C201: value 10u / 25V X5R -> 10u 16V X5R; LCSC C15850 -> (none); MPN CL21A106KAYNNNE -> (none); Manufacturer Samsung Electro-Mechanics -> (none); Source (none) -> stock:58
- C202: Source (none) -> stock:54
- C203: value 1u / 16V -> 2.2u 16V X5R; footprint Capacitor_SMD:C_0603_1608Metric -> Capacitor_SMD:C_0805_2012Metric; MPN (none) -> CL21A225KOFNNNE; Manufacturer (none) -> Samsung Electro-Mechanics; Source (none) -> stock:57
- R201, R202, R203, R207, R208, R209, R210, R211, R212: value 10k -> 10k 5%; footprint Resistor_SMD:R_0603_1608Metric -> Resistor_SMD:R_0805_2012Metric; Source (none) -> stock:70
- R204, R205, R206: MPN 0603WAF1001T5E -> RC0603FR-071KL; Manufacturer UNI-ROYAL -> Yageo; Source (none) -> stock:62
- SW201, SW202: footprint Button_Switch_SMD:SW_Push_1P1T_XKB_TS-1187A -> Button_Switch_THT:SW_PUSH_6mm_H9.5mm; LCSC C318884 -> (none); MPN TS-1187A-B-A-B -> 6X6X10MM Tact Switch; Manufacturer XKB Connection -> (none); Source (none) -> stock:95
