File: pcb/cheap-version/Peripherals.kicad_sch (KiCad schematic)
At the start: 33 parts, among them J301 SHT4x / XH 2.50, J302 FLOAT / 3.5 mm, J401 HRO TF-01A, U301 PCF8563T/5, Y301 32.768k 12.5pF

Commit message: cheap-version: schematic substitutions from stock parts
tools/make_cheap1.py generates the cheap-1 sheets from the PCB_V1 0.22 baseline:
ST1S14 for LMR16020 (RT resistor removed, EN/FB divider recalculated), IRS4427S and
IRL2505 for the heater, BSC146N10LS5 for the LED boost switches, SS56 diodes,
KF301/FS1.5/KF2510/XH connectors, stock resistors and capacitors (Source field =
stock:<id>). J901 XT60 is replaced by a screw terminal as decided. U101 TPS54202 and
D711/D721 SS5P10 are kept because datasheets for ST1S10 and SBRT15U100SP5 were not
available. ERC: 0 errors (one warning: footprint for the DTMSS-27 inductor pending);
netdiff against PCB_V1: no connectivity differences among untouched pins.

Co-Authored-By: Claude Sonnet 5.5 <noreply@anthropic.com>
Parts:
- C301, C303, C402: Source (none) -> stock:54
- C302: value 1u / 16V -> 2.2u 16V X5R; footprint Capacitor_SMD:C_0603_1608Metric -> Capacitor_SMD:C_0805_2012Metric; MPN (none) -> CL21A225KOFNNNE; Manufacturer (none) -> Samsung Electro-Mechanics; Source (none) -> stock:57
- C401: LCSC C29277 -> C318688; MPN CL21A226MPQNNNE -> CL21A226KPCLRNC; Source (none) -> stock:7
- J301: footprint Connector_JST:JST_XH_B4B-XH-A_1x04_P2.50mm_Vertical -> Connector_JST:JST_XH_S4B-XH-A_1x04_P2.50mm_Horizontal; MPN (none) -> XH2.54-4P-90; Source (none) -> stock:90
- J302: footprint GrowBox:TerminalBlock_DORABO_DB125-3.5_1x02_P3.50mm_Horizontal -> TerminalBlock_Phoenix:TerminalBlock_Phoenix_PT-1,5-2-3.5-H_1x02_P3.50mm_Horizontal; LCSC C466970 -> (none); MPN DB125-3.5-2P-GN-S -> FS1.5-02-350-2601R; Manufacturer DORABO -> (none); Source (none) -> stock:86
- R301, R302: value 4.7k -> 4.7k 5%; footprint Resistor_SMD:R_0603_1608Metric -> Resistor_SMD:R_0805_2012Metric; Source (none) -> stock:72
- R305, R307: MPN 0603WAF1001T5E -> RC0603FR-071KL; Manufacturer UNI-ROYAL -> Yageo; Source (none) -> stock:62
- R306, R405, R406, R407, R408, R410: value 10k -> 10k 5%; footprint Resistor_SMD:R_0603_1608Metric -> Resistor_SMD:R_0805_2012Metric; Source (none) -> stock:70
