File: pcb/cheap-version/cheap-version.kicad_sch (KiCad schematic)
At the start: 13 parts, among them U101 TPS54202DDCR

Commit message: cheap-version: schematic substitutions from stock parts
tools/make_cheap1.py generates the cheap-1 sheets from the PCB_V1 0.22 baseline:
ST1S14 for LMR16020 (RT resistor removed, EN/FB divider recalculated), IRS4427S and
IRL2505 for the heater, BSC146N10LS5 for the LED boost switches, SS56 diodes,
KF301/FS1.5/KF2510/XH connectors, stock resistors and capacitors (Source field =
stock:<id>). J901 XT60 is replaced by a screw terminal as decided. U101 TPS54202 and
D711/D721 SS5P10 are kept because datasheets for ST1S10 and SBRT15U100SP5 were not
available. ERC: 0 errors (one warning: footprint for the DTMSS-27 inductor pending);
netdiff against PCB_V1: no connectivity differences among untouched pins.

Co-Authored-By: Claude Sonnet 5.5 <noreply@anthropic.com>
Parts:
- C101: value 22u 25V X7R -> 10u 35V X5R; LCSC C309062 -> C2980162; MPN CL32B226KAJNNNE -> CL32A106KLULNNE; Manufacturer Samsung -> Samsung Electro-Mechanics; Source (none) -> stock:6
- C102, C103: Source (none) -> stock:54
- C104, C105: LCSC C29277 -> C318688; MPN CL21A226MPQNNNE -> CL21A226KPCLRNC; Source (none) -> stock:7
- R101: LCSC C25803 -> C14675; MPN 0603WAF1003T5E -> RC0603FR-07100KL; Manufacturer UNI-ROYAL -> Yageo; Source (none) -> stock:55
Changed lines of the file:
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@@
 	(title_block
 		(title "01 - Logic power / 12 V aux to 3.3 V")
-		(date "2026-09-30")
-		(rev "0.22-DRAFT")
+		(date "2026-10-03")
+		(rev "cheap-1-DRAFT")
 		(company "GrowBox controller")
-		(comment 1 "Simplified prototype; unrouted; hardware qualification pending")
+		(comment 1 "cheap-1: one-off board from stock parts, schematic derived from PCB_V1 0.22; unrouted")
 	)
 	(text "Vout = 0.596 x (1 + 100k/22k) = 3.305 V; divider 1%.\nStatic FB + resistor limits: 3.170..3.444 V. Budget <=1 A.\nL101 FXL0630-100-M: 10 uH, Isat 4.9 A, Irms 3.8 A, DCR 68 mOhm max.\nVerify C104/C105 effective capacitance and load-step response.\nC106 is NOT fitted until loop/transient verification."
@@
 			)
 		)
-		(property "Value" "22u 25V X7R"
+		(property "Value" "10u 35V X5R"
 			(at 42.72 69.85 0)
 			(show_name no)
@@
 			)
 		)
-		(property "Manufacturer" "Samsung"
+		(property "Manufacturer" "Samsung Electro-Mechanics"
 			(at 45.72 68.58 0)
 			(hide yes)
@@
 			)
 		)
-		(property "MPN" "CL32B226KAJNNNE"
+		(property "MPN" "CL32A106KLULNNE"
 			(at 45.72 68.58 0)
 			(hide yes)
@@
 			)
 		)
-		(property "LCSC" "C309062"
+		(property "LCSC" "C2980162"
 			(at 45.72 68.58 0)
 			(hide yes)
@@
 					(size 1 1)
 				)
+				(justify left)
+			)
+		)
+		(property "Source" "stock:6"
+			(at 45.72 68.58 0)
+			(effects
+				(font
+					(size 1 1)
+				)
+				(hide yes)
 				(justify left)
 			)
@@
 			)
 		)
-		(property "LCSC" "C29277"
+		(property "LCSC" "C318688"
 			(at 185.42 80.01 0)
 			(effects
@@
 			)
 		)
-		(property "MPN" "CL21A226MPQNNNE"
+		(property "Source" "stock:7"
+			(at 185.42 80.01 0)
+			(effects
+				(font
+					(size 1 1)
+				)
+				(hide yes)
+				(justify left)
+			)
+		)
+		(property "MPN" "CL21A226KPCLRNC"
 			(at 185.42 80.01 0)
 			(effects
@@
 			)
 		)
-		(property "Manufacturer" "UNI-ROYAL"
+		(property "Manufacturer" "Yageo"
 			(at 203.2 76.2 0)
 			(hide yes)
@@
 			)
 		)
-		(property "MPN" "0603WAF1003T5E"
+		(property "MPN" "RC0603FR-07100KL"
 			(at 203.2 76.2 0)
 			(hide yes)
@@
 			)
 		)
-		(property "LCSC" "C25803"
+		(property "LCSC" "C14675"
 			(at 203.2 76.2 0)
 			(hide yes)
@@
 					(size 1 1)
 				)
+				(justify left)
+			)
+		)
+		(property "Source" "stock:55"
+			(at 203.2 76.2 0)
+			(effects
+				(font
+					(size 1 1)
+				)
+				(hide yes)
 				(justify left)
 			)
@@
 			)
 		)
+		(property "Source" "stock:54"
+			(at 60.96 68.58 0)
+			(effects
+				(font
+					(size 1 1)
+				)
+				(hide yes)
+				(justify left)
+			)
+		)
 	)
 	(symbol
@@
 			)
 		)
+		(property "Source" "stock:54"
+			(at 116.84 53.34 90)
+			(effects
+				(font
+					(size 1 1)
+				)
+				(hide yes)
+				(justify left)
+			)
+		)
 	)
 	(symbol
@@
 			)
 		)
-		(property "LCSC" "C29277"
+		(property "LCSC" "C318688"
 			(at 165.1 80.01 0)
 			(effects
@@
 			)
 		)
-		(property "MPN" "CL21A226MPQNNNE"
+		(property "Source" "stock:7"
 			(at 165.1 80.01 0)
 			(effects
+				(font
+					(size 1 1)
+				)
+				(hide yes)
+				(justify left)
+			)
+		)
+		(property "MPN" "CL21A226KPCLRNC"
+			(at 165.1 80.01 0)
+			(effects

Commit message: cheap-version: ST1S10, SBRT15U100SP5, datasheet checks, LED boost estimate
With the datasheets supplied by the user: U101 TPS54202 -> ST1S10PHR (INH to VIN, SYNC to GND,
L101 4.7 uH FXL0630-4R7-M, R102 31.6k, C103 repurposed as the VIN_A bypass); the 3.3 V sheet is
redrawn in the stub-and-label style. D711/D721 -> SBRT15U100SP5 with a new GrowBox:Diodes_PowerDI5
footprint (tools/make_footprints.py). IRS4427S pinout/levels, BSC146N10LS5 and DTMSS-27 data
checked; tools/analyze_led_cheap.py re-runs the PCB_V1 LED boost model with the stock parts
(all checks pass). Datasheet PDFs are not committed (datasheets/.gitignore). ERC: 0 errors,
only the pending DTMSS-27 footprint warning; netdiff vs PCB_V1: no differences.

Co-Authored-By: Claude Sonnet 5.5 <noreply@anthropic.com>
Parts:
- removed U101: TPS54202DDCR, Package_TO_SOT_SMD:SOT-23-6, symbol Regulator_Switching:TPS54202DDC
- added U101: ST1S10PHR, Package_SO:SOIC-8-1EP_3.9x4.9mm_P1.27mm_EP2.41x3.3mm, symbol Regulator_Switching:ST1S10PHR
- C103: value 100n 50V X7R -> 2.2u 16V X5R; footprint Capacitor_SMD:C_0603_1608Metric -> Capacitor_SMD:C_0805_2012Metric; LCSC C1591 -> (none); MPN CL10B104KB8NNNC -> CL21A225KOFNNNE; Manufacturer Samsung -> Samsung Electro-Mechanics; Source stock:54 -> stock:57
- L101: value 10u FXL0630-100-M -> 4.7u FXL0630-4R7-M; LCSC C167223 -> C167220; MPN FXL0630-100-M -> FXL0630-4R7-M
- R102: value 22k 1% -> 31.6k 1%; LCSC C31850 -> (none); MPN 0603WAF2202T5E -> 0603WAF3162T5E; Source (none) -> buy: verify MPN on LCSC
Connections:
- net +12V: now also C103.1, U101.1 (VINA), U101.2 (INH), U101.6 (VINSW)
- net BUCK_FB: now also U101.3 (FB)
- net BUCK_SW: now also U101.7 (SW); no longer C103.2
- net GND: now also C103.2, U101.4 (AGND), U101.5 (SYNC), U101.8 (PGND), U101.9 (PADGND)
- no-connect marks 1 -> 0
Other:
- note added: "INH (EN) соединён с +12V: регулятор включён всегда. SYNC на GND: 900 кГц без внешней синхронизации."
- note added: "Vout = 0.8 V x (1 + 100k/31.6k) = 3.33 V (ST1S10 VFB 0.784..0.816 V); dividers 1%. ST1S10: 2.5..18 V in, 3 A, synchronous, 900 kHz (SYNC to GND), INH tied to VIN (on), no BOOT. L101 FXL0630-4R7-M: 4.7 uH, Isat 9 A, DCR 33 mOhm; C103 is the VIN_A bypass. Cout 3 x 22u/10V X5R (C104, C105, C401); verify load-step response. C106 is NOT fitted."
- note added: "cheap-1 DRAFT: schematic derived from PCB_V1 0.22 with stock-part substitutions; unrouted."
- note removed: "0.22 DRAFT: pre-routing (Murata LED output MLCCs, HRO TF-01A microSD, CLKOUT test pad; stack 1.6 mm, 1 oz outer / 0.5 oz inner); routing and prototype validation pending."
- note removed: "EN оставлен свободным: автоматический запуск по datasheet. Не подключать EN напрямую к 12 V."
- note removed: "Vout = 0.596 x (1 + 100k/22k) = 3.305 V; divider 1%. Static FB + resistor limits: 3.170..3.444 V. Budget <=1 A. L101 FXL0630-100-M: 10 uH, Isat 4.9 A, Irms 3.8 A, DCR 68 mOhm max. Verify C104/C105 effective capacitance and load-step response. C106 is NOT fitted until loop/transient verification."
