File: pcb/cheap-version/cheap-version.kicad_sch (KiCad schematic)
At the start: 13 parts, among them U101 ST1S10PHR

Commit message: Verify cheap-version purchase parts and require complete release checks
Parts:
- R102: LCSC (none) -> C25967; Source buy: verify MPN on LCSC -> buy
Changed lines of the file:
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@@
 			)
 		)
-		(property "LCSC" ""
+		(property "LCSC" "C25967"
 			(at 203.2 101.6 0)
 			(hide yes)
@@
 			)
 		)
-		(property "Source" "buy: verify MPN on LCSC"
+		(property "Source" "buy"
 			(at 203.2 101.6 0)
 			(effects
