File: pcb/cheap-version/LEDDrivers.kicad_sch (KiCad schematic)
At the start: 54 parts, among them J711 LED +/- (return isolated), J721 LED +/- (return isolated), J731 LED +/- (return isolated), Q711 BSC146N10LS5, Q721 BSC146N10LS5, U700 SN74LVC1G08DBVR, U710 AL8853S-13, U720 AL8853S-13

Commit message: cheap-version: CH1 for 80 W and UCC27524 heater driver
R716 0.18 -> 0.12 ohm (1.667 A, 80 W at 48 V; the LED panel is rated up to
120 W and is not fully loaded). analyze_led_cheap.py re-run: input current
up to 4.61 A, inductor peak 6.26 A, OCP headroom 2.06 A, all model checks
pass; about 96 W is the ceiling of this controller/inductor pair.

U601 is the PCB_V1 UCC27524ADR again instead of the IRS4427S (2.5 V input
threshold left 0.14 V of margin at ESP32 VOH): ENA tied to +12V, ENB to
GND. Board side in tools/swap_heater_driver.py; generator, BOM and BUY
lists follow (order estimate USD 34.69). Schematic ERC 0, schematic and
board match pin by pin.

Co-Authored-By: Claude Sonnet 5.5 <noreply@anthropic.com>
Parts:
- R716: value 0.18 1% 2W 50ppm -> 0.12 1% 2W 50ppm; LCSC C48533605 -> (none); MPN FRM252WFR180TM -> FRM252WFR120TM
Other:
- note added: "CH1: 1.667 A nominal = 80 W at 48 V (panel rated up to 120 W)"
- note removed: "CH1: 1.111 A nominal / panel"
Changed lines of the file:
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@@
 		)
 	)
-	(text "CH1: 1.111 A nominal / panel"
+	(text "CH1: 1.667 A nominal = 80 W at 48 V (panel rated up to 120 W)"
 		(exclude_from_sim no)
 		(at 20.32 80.01 0)
@@
 			)
 		)
-		(property "Value" "0.18 1% 2W 50ppm"
+		(property "Value" "0.12 1% 2W 50ppm"
 			(at 448.31 124.46 0)
 			(show_name no)
@@
 			)
 		)
-		(property "MPN" "FRM252WFR180TM"
+		(property "MPN" "FRM252WFR120TM"
 			(at 444.5 123.19 0)
 			(hide yes)
@@
 			)
 		)
-		(property "LCSC" "C48533605"
+		(property "LCSC" ""
 			(at 444.5 123.19 0)
 			(hide yes)
