File: pcb/cheap-version/cheap-version.kicad_pcb (KiCad board)
At the start: 4 copper layers, 100 x 100 mm, 170 parts, among them J201 UART / 3V3 logic, J301 SHT4x / XH 2.50, J302 FLOAT / 3.5 mm, J401 HRO TF-01A, J501 FAN1 / 3.5 mm, J511 FAN2 / 3.5 mm, J521 PUMP 24V / 6W, J601 PTC + / switched - (3.5 mm), J711 LED +/- (return isolated), J721 LED +/- (return isolated), J731 LED +/- (return isolated), J901 24V IN (KF301-5.0-2P), Q501 AO3400A, Q511 AO3400A, Q521 AO3422, Q601 IRL2505, Q711 BSC146N10LS5, Q721 BSC146N10LS5, SW201 RESET, SW202 BOOT, U101 ST1S10PHR, U201 ESP32-WROOM-32E-N4, U301 PCF8563T/5, U601 UCC27524ADR, U700 SN74LVC1G08DBVR, U710 AL8853S-13, U720 AL8853S-13, U902 ST1S14PHR, Y301 32.768k 12.5pF

Commit message: Verify cheap-version purchase parts and require complete release checks
Parts:
- R716: value 0.12 1% 2W 50ppm -> 0.12 1% 3W 50ppm
Changed lines of the file:
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@@
 			)
 		)
-		(property "LCSC" ""
+		(property "LCSC" "C728599"
 			(at 0 0 0)
 			(layer "F.SilkS")
@@
 			)
 		)
-		(property "LCSC" ""
+		(property "LCSC" "C25967"
 			(at 0 0 0)
 			(layer "F.SilkS")
@@
 			)
 		)
-		(property "Value" "0.12 1% 2W 50ppm"
+		(property "Value" "0.12 1% 3W 50ppm"
 			(at 0 2.63 90)
 			(layer "F.Fab")
@@
 			)
 		)
-		(property "Datasheet" "https://datasheet.lcsc.com/datasheet/pdf/b47da348e6587de9f1f028172ba2b8ea.pdf"
+		(property "Datasheet" "https://datasheet.lcsc.com/datasheet/pdf/02ae4b20613551dea68a63964573e262.pdf"
 			(at 0 0 90)
 			(layer "F.Fab")
@@
 			)
 		)
-		(property "Manufacturer" "FOJAN"
+		(property "Manufacturer" "JIERR"
 			(at 0 0 90)
 			(layer "F.SilkS")
@@
 			)
 		)
-		(property "MPN" "FRM252WFR120TM"
+		(property "MPN" "JER2512F3R120"
 			(at 0 0 90)
 			(layer "F.SilkS")
@@
 			)
 		)
-		(property "LCSC" ""
+		(property "LCSC" "C49164917"
 			(at 0 0 90)
 			(layer "F.SilkS")
@@
 			)
 		)
-		(property "LCSC" ""
+		(property "LCSC" "C23178"
 			(at 0 0 0)
 			(layer "F.SilkS")

Commit message: Show key component references on cheap board silkscreen
Changed lines of the file:
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@@
 			(at 0 0 0)
 			(layer "F.Fab")
-			(hide yes)
 			(effects
 				(font
@@
 			(at 0 0 270)
 			(layer "F.Fab")
-			(hide yes)
 			(effects
 				(font
@@
 			(at 0 0 0)
 			(layer "F.Fab")
-			(hide yes)
 			(effects
 				(font
@@
 		(tags "SMD SMT Crystal")
 		(property "Reference" "Y301"
-			(at -3.4 -0.1 0)
+			(at 2.506 4.777143 0)
 			(layer "F.SilkS")
-			(hide yes)
 			(effects
 				(font
 					(size 1 1)
-					(thickness 0.15)
+					(thickness 0.2)
 				)
 			)
@@
 			(at 0 0 0)
 			(layer "F.Fab")
-			(hide yes)
 			(effects
 				(font
@@
 			(at 0 0 0)
 			(layer "F.Fab")
-			(hide yes)
 			(effects
 				(font
@@
 			(at 0 0 0)
 			(layer "F.Fab")
-			(hide yes)
 			(effects
 				(font
@@
 			(at 0 0 0)
 			(layer "F.Fab")
-			(hide yes)
 			(effects
 				(font
@@
 			(at 0 0 0)
 			(layer "F.Fab")
-			(hide yes)
 			(effects
 				(font
@@
 			(at 0 0 180)
 			(layer "F.Fab")
-			(hide yes)
 			(effects
 				(font
@@
 			(at 0 0 0)
 			(layer "F.Fab")
-			(hide yes)
 			(effects
 				(font
@@
 		(tags "power shielded cjiang fxl")
 		(property "Reference" "L101"
-			(at 0 -4.25 0)
+			(at -6.453334 1.094 0)
 			(layer "F.SilkS")
-			(hide yes)
 			(effects
 				(font
 					(size 1 1)
-					(thickness 0.15)
+					(thickness 0.2)
 				)
 			)
@@
 			(at 0 0 0)
 			(layer "F.Fab")
-			(hide yes)
 			(effects
 				(font
@@
 		(tags "SOT TO_SOT_SMD")
 		(property "Reference" "D303"
-			(at 0 -2.7 90)
+			(at -9.031 -2.798572 0)
 			(layer "F.SilkS")
-			(hide yes)
 			(effects
 				(font
 					(size 1 1)
-					(thickness 0.15)
+					(thickness 0.2)
 				)
 			)
@@
 			(at 0 0 0)
 			(layer "F.Fab")
-			(hide yes)
 			(effects
 				(font
@@
 			(at 0 0 0)
 			(layer "F.Fab")
-			(hide yes)
 			(effects
 				(font
@@
 			(at 0 0 270)
 			(layer "F.Fab")
-			(hide yes)
 			(effects
 				(font
@@
 			(at 0 0 0)
 			(layer "F.Fab")
-			(hide yes)
 			(effects
 				(font
@@
 		(tags "power shielded cjiang fxl")
 		(property "Reference" "L902"
-			(at 0 -4.25 0)
+			(at -0.053334 4.706 0)
 			(layer "F.SilkS")
-			(hide yes)
 			(effects
 				(font
 					(size 1 1)
-					(thickness 0.15)
+					(thickness 0.2)
 				)
 			)
@@
 			(at 0 0 180)
 			(layer "F.Fab")
-			(hide yes)
 			(effects
 				(font
@@
 			(at 0 0 0)
 			(layer "F.Fab")
-			(hide yes)
 			(effects
 				(font
@@
 		(tags "microSD TF card socket push-push HRO TF-01A")
 		(property "Reference" "J401"
-			(at 0 -9.5 90)
+			(at 5.116 -10.480524 0)
 			(layer "F.SilkS")
-			(hide yes)
 			(effects
 				(font
-					(size 1.27 1.27)
+					(size 1 1)
+					(thickness 0.2)
 				)
 			)
@@
 			(at 0 0 0)
 			(layer "F.Fab")
-			(hide yes)
 			(effects
 				(font
@@
 			(at 0 0 0)
 			(layer "F.Fab")
-			(hide yes)
 			(effects
 				(font
@@
 			(at 0 0 0)
 			(layer "F.Fab")
-			(hide yes)
 			(effects
 				(font
@@
 			(unlocked yes)
 			(layer "B.Fab")
-			(hide yes)
 			(effects
 				(font
