File: hardware/PCB_EU/InputPower.kicad_sch (KiCad schematic)
At the start: 33 parts, among them J101 24 V IN, U101 L7987 3A

Commit message: hardware: complete EU mechanical footprint assignments and validate pad maps
Parts:
- F101, F102, F103: footprint (none) -> EU_Mechanical:Fuse_Schurter_UST_USI1206_Reflow; Design_note DC fuse package / clearing I2t to be checked before layout -> SCHURTER reflow lands checked; fuse clearing I2t/coordinati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; FootprintStatus PENDING - no approved footprint -> DRAWING CHECKED - physical fit and PCB validation pending
- F104, F105, F106: footprint (none) -> EU_Mechanical:Fuse_Schurter_UMT250; Design_note DC fuse package / clearing I2t to be checked before layout -> SCHURTER reflow lands checked; fuse clearing I2t/coordinati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; FootprintStatus PENDING - no approved footprint -> DRAWING CHECKED - physical fit and PCB validation pending
- J101: footprint (none) -> EU_Mechanical:TerminalBlock_Degson_DG301R-5.0_1x02; Design_note 16 A terminal; exact footprint pending drawing -> DG301R-C02 T1 drawing; UL 15 A / IEC 17.5 A; confirm ordere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; FootprintStatus PENDING - no approved footprint -> DRAWING CHECKED - physical fit and PCB validation pending
- L101: footprint (none) -> EU_Mechanical:L_Jantek_JNRH1207; Design_note Jantek drawing and hot Isat remain layout/prototype checks -> Jantek SP-N251224012 rev A lands checked; hot Isat remains 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; FootprintStatus PENDING - no approved footprint -> DRAWING CHECKED - physical fit and PCB validation pending
- U101: footprint (none) -> EU_Mechanical:HTSSOP-16-1EP_4.4x5mm_P0.65mm_EP3x3mm; Design_note HTSSOP16 EP; exact exposed pad footprint still pending -> ST HTSSOP16 EP17=GND; 3x3 EP and 0.65 pitch; assembly and t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; FootprintStatus PENDING - no approved footprint -> DRAWING CHECKED - physical fit and PCB validation pending
