File: hardware/PCB_EU/Interfaces.kicad_sch (KiCad schematic)
At the start: 29 parts, among them J401 SHT 3V3 / GND, J402 SHT SDA / SCL, J403 FLOAT / GND, J411 FAN1: GND / +12, J412 FAN1: TACH / PWM, J421 FAN2: GND / +12, J422 FAN2: TACH / PWM, Q411 FAN1 AO3422, Q421 FAN2 AO3422, U401 USBLC6-2SC6, U402 USBLC6-2SC6

Commit message: hardware: complete EU mechanical footprint assignments and validate pad maps
Parts:
- F401: footprint (none) -> EU_Mechanical:Fuse_Schurter_UMT250; FootprintStatus PENDING - no approved footprint -> DRAWING CHECKED - physical fit and PCB validation pending
- J401, J402, J403, J411, J412, J421, J422: footprint (none) -> EU_Mechanical:TerminalBlock_Degson_DG306-5.0_1x02; FootprintStatus PENDING - no approved footprint -> DRAWING CHECKED - physical fit and PCB validation pending
Changed lines of the file:
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@@
 (property "Reference" "J401" (at 45.72 137.87 0) (effects (font (size 1.15 1.15)) ))
 (property "Value" "SHT 3V3 / GND" (at 45.72 151.69 0) (effects (font (size 0.98 0.98)) ))
-(property "Footprint" "" (at 45.72 144.78 0) (effects (font (size 1 1)) (hide yes)))
+(property "Footprint" "EU_Mechanical:TerminalBlock_Degson_DG306-5.0_1x02" (at 45.72 144.78 0) (effects (font (size 1 1)) (hide yes)))
 (property "Datasheet" "" (at 45.72 144.78 0) (effects (font (size 1 1)) (hide yes)))
 (property "MPN" "DG306-5.0-2P12" (at 45.72 144.78 0) (effects (font (size 1 1)) (hide yes)))
 (property "Design_note" "" (at 45.72 144.78 0) (effects (font (size 1 1)) (hide yes)))
-(property "FootprintStatus" "PENDING - no approved footprint" (at 45.72 144.78 0) (effects (font (size 1 1)) (hide yes)))
+(property "FootprintStatus" "DRAWING CHECKED - physical fit and PCB validation pending" (at 45.72 144.78 0) (effects (font (size 1 1)) (hide yes)))
 (pin "1")
 (pin "2")
@@
 (property "Reference" "J402" (at 106.68 137.87 0) (effects (font (size 1.15 1.15)) ))
 (property "Value" "SHT SDA / SCL" (at 106.68 151.69 0) (effects (font (size 0.98 0.98)) ))
-(property "Footprint" "" (at 106.68 144.78 0) (effects (font (size 1 1)) (hide yes)))
+(property "Footprint" "EU_Mechanical:TerminalBlock_Degson_DG306-5.0_1x02" (at 106.68 144.78 0) (effects (font (size 1 1)) (hide yes)))
 (property "Datasheet" "" (at 106.68 144.78 0) (effects (font (size 1 1)) (hide yes)))
 (property "MPN" "DG306-5.0-2P12" (at 106.68 144.78 0) (effects (font (size 1 1)) (hide yes)))
 (property "Design_note" "" (at 106.68 144.78 0) (effects (font (size 1 1)) (hide yes)))
-(property "FootprintStatus" "PENDING - no approved footprint" (at 106.68 144.78 0) (effects (font (size 1 1)) (hide yes)))
+(property "FootprintStatus" "DRAWING CHECKED - physical fit and PCB validation pending" (at 106.68 144.78 0) (effects (font (size 1 1)) (hide yes)))
 (pin "1")
 (pin "2")
@@
 (property "Reference" "J403" (at 173.99 137.87 0) (effects (font (size 1.15 1.15)) ))
 (property "Value" "FLOAT / GND" (at 173.99 151.69 0) (effects (font (size 0.98 0.98)) ))
-(property "Footprint" "" (at 173.99 144.78 0) (effects (font (size 1 1)) (hide yes)))
+(property "Footprint" "EU_Mechanical:TerminalBlock_Degson_DG306-5.0_1x02" (at 173.99 144.78 0) (effects (font (size 1 1)) (hide yes)))
 (property "Datasheet" "" (at 173.99 144.78 0) (effects (font (size 1 1)) (hide yes)))
 (property "MPN" "DG306-5.0-2P12" (at 173.99 144.78 0) (effects (font (size 1 1)) (hide yes)))
 (property "Design_note" "" (at 173.99 144.78 0) (effects (font (size 1 1)) (hide yes)))
-(property "FootprintStatus" "PENDING - no approved footprint" (at 173.99 144.78 0) (effects (font (size 1 1)) (hide yes)))
+(property "FootprintStatus" "DRAWING CHECKED - physical fit and PCB validation pending" (at 173.99 144.78 0) (effects (font (size 1 1)) (hide yes)))
 (pin "1")
 (pin "2")
@@
 (property "Reference" "F401" (at 308.61 159.46 0) (effects (font (size 1.15 1.15)) ))
 (property "Value" "2 A slow" (at 308.61 170.74 0) (effects (font (size 0.98 0.98)) ))
-(property "Footprint" "" (at 308.61 165.1 0) (effects (font (size 1 1)) (hide yes)))
+(property "Footprint" "EU_Mechanical:Fuse_Schurter_UMT250" (at 308.61 165.1 0) (effects (font (size 1 1)) (hide yes)))
 (property "Datasheet" "" (at 308.61 165.1 0) (effects (font (size 1 1)) (hide yes)))
 (property "MPN" "3403.0169.11" (at 308.61 165.1 0) (effects (font (size 1 1)) (hide yes)))
 (property "Design_note" "" (at 308.61 165.1 0) (effects (font (size 1 1)) (hide yes)))
-(property "FootprintStatus" "PENDING - no approved footprint" (at 308.61 165.1 0) (effects (font (size 1 1)) (hide yes)))
+(property "FootprintStatus" "DRAWING CHECKED - physical fit and PCB validation pending" (at 308.61 165.1 0) (effects (font (size 1 1)) (hide yes)))
 (pin "1")
 (pin "2")
@@
 (property "Reference" "J411" (at 374.65 158.19 0) (effects (font (size 1.15 1.15)) ))
 (property "Value" "FAN1: GND / +12" (at 374.65 172.01 0) (effects (font (size 0.98 0.98)) ))
-(property "Footprint" "" (at 374.65 165.1 0) (effects (font (size 1 1)) (hide yes)))
+(property "Footprint" "EU_Mechanical:TerminalBlock_Degson_DG306-5.0_1x02" (at 374.65 165.1 0) (effects (font (size 1 1)) (hide yes)))
 (property "Datasheet" "" (at 374.65 165.1 0) (effects (font (size 1 1)) (hide yes)))
 (property "MPN" "DG306-5.0-2P12" (at 374.65 165.1 0) (effects (font (size 1 1)) (hide yes)))
 (property "Design_note" "" (at 374.65 165.1 0) (effects (font (size 1 1)) (hide yes)))
-(property "FootprintStatus" "PENDING - no approved footprint" (at 374.65 165.1 0) (effects (font (size 1 1)) (hide yes)))
+(property "FootprintStatus" "DRAWING CHECKED - physical fit and PCB validation pending" (at 374.65 165.1 0) (effects (font (size 1 1)) (hide yes)))
 (pin "1")
 (pin "2")
@@
 (property "Reference" "J412" (at 45.72 178.51 0) (effects (font (size 1.15 1.15)) ))
 (property "Value" "FAN1: TACH / PWM" (at 45.72 192.33 0) (effects (font (size 0.98 0.98)) ))
-(property "Footprint" "" (at 45.72 185.42 0) (effects (font (size 1 1)) (hide yes)))
+(property "Footprint" "EU_Mechanical:TerminalBlock_Degson_DG306-5.0_1x02" (at 45.72 185.42 0) (effects (font (size 1 1)) (hide yes)))
 (property "Datasheet" "" (at 45.72 185.42 0) (effects (font (size 1 1)) (hide yes)))
 (property "MPN" "DG306-5.0-2P12" (at 45.72 185.42 0) (effects (font (size 1 1)) (hide yes)))
 (property "Design_note" "" (at 45.72 185.42 0) (effects (font (size 1 1)) (hide yes)))
-(property "FootprintStatus" "PENDING - no approved footprint" (at 45.72 185.42 0) (effects (font (size 1 1)) (hide yes)))
+(property "FootprintStatus" "DRAWING CHECKED - physical fit and PCB validation pending" (at 45.72 185.42 0) (effects (font (size 1 1)) (hide yes)))
 (pin "1")
 (pin "2")
@@
 (property "Reference" "J421" (at 374.65 178.51 0) (effects (font (size 1.15 1.15)) ))
 (property "Value" "FAN2: GND / +12" (at 374.65 192.33 0) (effects (font (size 0.98 0.98)) ))
-(property "Footprint" "" (at 374.65 185.42 0) (effects (font (size 1 1)) (hide yes)))
+(property "Footprint" "EU_Mechanical:TerminalBlock_Degson_DG306-5.0_1x02" (at 374.65 185.42 0) (effects (font (size 1 1)) (hide yes)))
 (property "Datasheet" "" (at 374.65 185.42 0) (effects (font (size 1 1)) (hide yes)))
 (property "MPN" "DG306-5.0-2P12" (at 374.65 185.42 0) (effects (font (size 1 1)) (hide yes)))
 (property "Design_note" "" (at 374.65 185.42 0) (effects (font (size 1 1)) (hide yes)))
-(property "FootprintStatus" "PENDING - no approved footprint" (at 374.65 185.42 0) (effects (font (size 1 1)) (hide yes)))
+(property "FootprintStatus" "DRAWING CHECKED - physical fit and PCB validation pending" (at 374.65 185.42 0) (effects (font (size 1 1)) (hide yes)))
 (pin "1")
 (pin "2")
@@
 (property "Reference" "J422" (at 45.72 197.56 0) (effects (font (size 1.15 1.15)) ))
 (property "Value" "FAN2: TACH / PWM" (at 45.72 211.38 0) (effects (font (size 0.98 0.98)) ))
-(property "Footprint" "" (at 45.72 204.47 0) (effects (font (size 1 1)) (hide yes)))
+(property "Footprint" "EU_Mechanical:TerminalBlock_Degson_DG306-5.0_1x02" (at 45.72 204.47 0) (effects (font (size 1 1)) (hide yes)))
 (property "Datasheet" "" (at 45.72 204.47 0) (effects (font (size 1 1)) (hide yes)))
 (property "MPN" "DG306-5.0-2P12" (at 45.72 204.47 0) (effects (font (size 1 1)) (hide yes)))
 (property "Design_note" "" (at 45.72 204.47 0) (effects (font (size 1 1)) (hide yes)))
-(property "FootprintStatus" "PENDING - no approved footprint" (at 45.72 204.47 0) (effects (font (size 1 1)) (hide yes)))
-(pin "1")
-(pin "2")
+(property "FootprintStatus" "DRAWING CHECKED - physical fit and PCB validation pending" (at 45.72 204.47 0) (effects (font (size 1 1)) (hide yes)))
+(pin "1")
+(pin "2")
