File: hardware/PCB_EU/Interfaces.kicad_sch (KiCad schematic)
At the start: 29 parts, among them J401 SHT 3V3 / GND, J402 SHT SDA / SCL, J403 FLOAT / GND, J411 FAN1: GND / +12, J412 FAN1: TACH / PWM, J421 FAN2: GND / +12, J422 FAN2: TACH / PWM, Q411 FAN1 AO3422, Q421 FAN2 AO3422, U401 USBLC6-2SC6, U402 USBLC6-2SC6

Commit message: PCB_EU: all terminals at the board edges, no HS2, fans on KF2510-4A, SHT4x on XH2.54-4P-90
Per Igors (22.10.2026):
- stack stated as 1 oz outer / 0.5 oz inner in DESIGN.md;
- heatsink HS2 removed from the LED2 channel (Q601 runs without a heatsink,
  about 54 C rise, to be measured on the prototype), freed area used for the
  pump terminal J702 and its parts at the right edge;
- J101, J201, J411, J421, J401, J403, J701, J702 moved so that every cable
  entry faces the board edge; J701 changed from DG301R to DG306;
- fan connectors J411/J421 are 4-pin KF2510-4A headers (Molex KK-254
  footprint), J412/J422 removed;
- SHT4x on one right-angle XH2.54-4P-90 header J401 (JST XH S4B-XH-A
  footprint), J402 removed;
- input, trunk and PTC copper re-routed in routing.json; the F101.2 trunk
  now starts with a 2.4 mm neck inside the pad (it was not attached before);
- BOM: quantities and total (82.50 EUR) unchanged, the new rows have no shop
  or price and are flagged for the BOM review.

Checks (KiCad 10.0.7): ERC 0, 56 connectivity checks, 22639 placement checks,
DRC 0 / parity 0 / unconnected 0, rebuild from the repository is byte-identical.
ampacity.py: worst IPC-2221 rise 38 C, three vias above the 2 A rule of thumb.

Co-Authored-By: Claude Sonnet 5.5 <noreply@anthropic.com>
Claude-Session: https://claude.ai/code/session_01AxccZX6Cb4FnRKJMrFYMSX
Parts:
- removed J402: SHT SDA / SCL, EU_Mechanical:TerminalBlock_Degson_DG306-5.0_1x02, symbol EU:J2
- removed J412: FAN1: TACH / PWM, EU_Mechanical:TerminalBlock_Degson_DG306-5.0_1x02, symbol EU:J2
- removed J422: FAN2: TACH / PWM, EU_Mechanical:TerminalBlock_Degson_DG306-5.0_1x02, symbol EU:J2
- J401: value SHT 3V3 / GND -> SHT4x XH2.54-4P-90; footprint EU_Mechanical:TerminalBlock_Degson_DG306-5.0_1x02 -> Connector_JST:JST_XH_S4B-XH-A_1x04_P2.50mm_Horizontal; symbol EU:J2 -> EU:J4; Design_note (none) -> 1 +3V3, 2 GND, 3 SDA, 4 SCL. XH clone, right angle; real pi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; FootprintStatus DRAWING CHECKED - physical fit and PCB validation pending -> PACKAGE ONLY - verify before PCB; MPN DG306-5.0-2P12 -> XH2.54-4P-90
- J411: value FAN1: GND / +12 -> FAN1 2510-4P; footprint EU_Mechanical:TerminalBlock_Degson_DG306-5.0_1x02 -> Connector_Molex:Molex_KK-254_AE-6410-04A_1x04_P2.54mm_Vertical; symbol EU:J2 -> EU:J4; Design_note (none) -> 4-pin PC fan pinout: 1 GND, 2 +12 V, 3 tach, 4 PWM. KF2510 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; FootprintStatus DRAWING CHECKED - physical fit and PCB validation pending -> PACKAGE ONLY - verify before PCB; MPN DG306-5.0-2P12 -> KF2510-4A
- J421: value FAN2: GND / +12 -> FAN2 2510-4P; footprint EU_Mechanical:TerminalBlock_Degson_DG306-5.0_1x02 -> Connector_Molex:Molex_KK-254_AE-6410-04A_1x04_P2.54mm_Vertical; symbol EU:J2 -> EU:J4; Design_note (none) -> 4-pin PC fan pinout: 1 GND, 2 +12 V, 3 tach, 4 PWM. KF2510 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; FootprintStatus DRAWING CHECKED - physical fit and PCB validation pending -> PACKAGE ONLY - verify before PCB; MPN DG306-5.0-2P12 -> KF2510-4A
Connections:
- net FAN1_PWM: now also J411.4
- net FAN1_TACH_EXT: now also J411.3
- net FAN2_PWM: now also J421.4
- net FAN2_TACH_EXT: now also J421.3
- net SHT_SCL: now also J401.4
- net SHT_SDA: now also J401.3
Other:
- moved on the sheet: C401, C402, C403, F401, J403, R401, R402, R403, R404, R411, R412, R413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
