File: hardware/PCB_EU/LED1.kicad_sch (KiCad schematic)
At the start: 29 parts, among them J501 LED1 + / GND, Q501 IRF540ZPBF, U501 LM3429MH/NOPB

Commit message: hardware: complete EU mechanical footprint assignments and validate pad maps
Parts:
- J501: footprint (none) -> EU_Mechanical:TerminalBlock_Degson_DG306-5.0_1x02; FootprintStatus PENDING - no approved footprint -> DRAWING CHECKED - physical fit and PCB validation pending
- L501, L502: footprint (none) -> EU_Mechanical:L_Jantek_JNRH1207; FootprintStatus PENDING - no approved footprint -> DRAWING CHECKED - physical fit and PCB validation pending
- U501: footprint (none) -> EU_Mechanical:TI_PWP0014A_LM3429; Design_note HTSSOP14 EP footprint dimensions must be validated -> TI PWP0014A: EP15=GND; copper 3.4x5, mask 3.155x3.255; ther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; FootprintStatus PENDING - no approved footprint -> DRAWING CHECKED - physical fit and PCB validation pending
Changed lines of the file:
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@@
 (property "Reference" "U501" (at 85.09 45.16 0) (effects (font (size 1.15 1.15)) ))
 (property "Value" "LM3429MH/NOPB" (at 85.09 74.22 0) (effects (font (size 0.98 0.98)) ))
-(property "Footprint" "" (at 85.09 59.69 0) (effects (font (size 1 1)) (hide yes)))
+(property "Footprint" "EU_Mechanical:TI_PWP0014A_LM3429" (at 85.09 59.69 0) (effects (font (size 1 1)) (hide yes)))
 (property "Datasheet" "https://www.ti.com/lit/ds/symlink/lm3429.pdf" (at 85.09 59.69 0) (effects (font (size 1 1)) (hide yes)))
 (property "MPN" "LM3429MH/NOPB" (at 85.09 59.69 0) (effects (font (size 1 1)) (hide yes)))
-(property "Design_note" "HTSSOP14 EP footprint dimensions must be validated" (at 85.09 59.69 0) (effects (font (size 1 1)) (hide yes)))
-(property "FootprintStatus" "PENDING - no approved footprint" (at 85.09 59.69 0) (effects (font (size 1 1)) (hide yes)))
+(property "Design_note" "TI PWP0014A: EP15=GND; copper 3.4x5, mask 3.155x3.255; thermal vias and assembly pending" (at 85.09 59.69 0) (effects (font (size 1 1)) (hide yes)))
+(property "FootprintStatus" "DRAWING CHECKED - physical fit and PCB validation pending" (at 85.09 59.69 0) (effects (font (size 1 1)) (hide yes)))
 (pin "1")
 (pin "2")
@@
 (property "Reference" "L501" (at 45.72 113.74 0) (effects (font (size 1.15 1.15)) ))
 (property "Value" "10u" (at 45.72 125.02 0) (effects (font (size 0.98 0.98)) ))
-(property "Footprint" "" (at 45.72 119.38 0) (effects (font (size 1 1)) (hide yes)))
+(property "Footprint" "EU_Mechanical:L_Jantek_JNRH1207" (at 45.72 119.38 0) (effects (font (size 1 1)) (hide yes)))
 (property "Datasheet" "" (at 45.72 119.38 0) (effects (font (size 1 1)) (hide yes)))
 (property "MPN" "JNRH1207-100N-A" (at 45.72 119.38 0) (effects (font (size 1 1)) (hide yes)))
 (property "Design_note" "" (at 45.72 119.38 0) (effects (font (size 1 1)) (hide yes)))
-(property "FootprintStatus" "PENDING - no approved footprint" (at 45.72 119.38 0) (effects (font (size 1 1)) (hide yes)))
+(property "FootprintStatus" "DRAWING CHECKED - physical fit and PCB validation pending" (at 45.72 119.38 0) (effects (font (size 1 1)) (hide yes)))
 (pin "1")
 (pin "2")
@@
 (property "Reference" "L502" (at 106.68 113.74 0) (effects (font (size 1.15 1.15)) ))
 (property "Value" "10u" (at 106.68 125.02 0) (effects (font (size 0.98 0.98)) ))
-(property "Footprint" "" (at 106.68 119.38 0) (effects (font (size 1 1)) (hide yes)))
+(property "Footprint" "EU_Mechanical:L_Jantek_JNRH1207" (at 106.68 119.38 0) (effects (font (size 1 1)) (hide yes)))
 (property "Datasheet" "" (at 106.68 119.38 0) (effects (font (size 1 1)) (hide yes)))
 (property "MPN" "JNRH1207-100N-A" (at 106.68 119.38 0) (effects (font (size 1 1)) (hide yes)))
 (property "Design_note" "" (at 106.68 119.38 0) (effects (font (size 1 1)) (hide yes)))
-(property "FootprintStatus" "PENDING - no approved footprint" (at 106.68 119.38 0) (effects (font (size 1 1)) (hide yes)))
+(property "FootprintStatus" "DRAWING CHECKED - physical fit and PCB validation pending" (at 106.68 119.38 0) (effects (font (size 1 1)) (hide yes)))
 (pin "1")
 (pin "2")
@@
 (property "Reference" "J501" (at 106.68 192.48 0) (effects (font (size 1.15 1.15)) ))
 (property "Value" "LED1 + / GND" (at 106.68 206.3 0) (effects (font (size 0.98 0.98)) ))
-(property "Footprint" "" (at 106.68 199.39 0) (effects (font (size 1 1)) (hide yes)))
+(property "Footprint" "EU_Mechanical:TerminalBlock_Degson_DG306-5.0_1x02" (at 106.68 199.39 0) (effects (font (size 1 1)) (hide yes)))
 (property "Datasheet" "" (at 106.68 199.39 0) (effects (font (size 1 1)) (hide yes)))
 (property "MPN" "DG306-5.0-2P12" (at 106.68 199.39 0) (effects (font (size 1 1)) (hide yes)))
 (property "Design_note" "" (at 106.68 199.39 0) (effects (font (size 1 1)) (hide yes)))
-(property "FootprintStatus" "PENDING - no approved footprint" (at 106.68 199.39 0) (effects (font (size 1 1)) (hide yes)))
-(pin "1")
-(pin "2")
+(property "FootprintStatus" "DRAWING CHECKED - physical fit and PCB validation pending" (at 106.68 199.39 0) (effects (font (size 1 1)) (hide yes)))
+(pin "1")
+(pin "2")
