File: hardware/PCB_EU/LED2.kicad_sch (KiCad schematic)
At the start: 28 parts, among them J601 LED2 + / GND, J602 BAR2 + / GND, Q601 IRF540ZPBF, U601 LM3429MH/NOPB

Commit message: hardware: complete EU mechanical footprint assignments and validate pad maps
Parts:
- J601, J602: footprint (none) -> EU_Mechanical:TerminalBlock_Degson_DG306-5.0_1x02; FootprintStatus PENDING - no approved footprint -> DRAWING CHECKED - physical fit and PCB validation pending
- L601: footprint (none) -> EU_Mechanical:L_Jantek_JNRH1207; FootprintStatus PENDING - no approved footprint -> DRAWING CHECKED - physical fit and PCB validation pending
- U601: footprint (none) -> EU_Mechanical:TI_PWP0014A_LM3429; Design_note HTSSOP14 EP footprint dimensions must be validated -> TI PWP0014A: EP15=GND; copper 3.4x5, mask 3.155x3.255; ther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; FootprintStatus PENDING - no approved footprint -> DRAWING CHECKED - physical fit and PCB validation pending
Changed lines of the file:
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@@
 (property "Reference" "U601" (at 85.09 45.16 0) (effects (font (size 1.15 1.15)) ))
 (property "Value" "LM3429MH/NOPB" (at 85.09 74.22 0) (effects (font (size 0.98 0.98)) ))
-(property "Footprint" "" (at 85.09 59.69 0) (effects (font (size 1 1)) (hide yes)))
+(property "Footprint" "EU_Mechanical:TI_PWP0014A_LM3429" (at 85.09 59.69 0) (effects (font (size 1 1)) (hide yes)))
 (property "Datasheet" "https://www.ti.com/lit/ds/symlink/lm3429.pdf" (at 85.09 59.69 0) (effects (font (size 1 1)) (hide yes)))
 (property "MPN" "LM3429MH/NOPB" (at 85.09 59.69 0) (effects (font (size 1 1)) (hide yes)))
-(property "Design_note" "HTSSOP14 EP footprint dimensions must be validated" (at 85.09 59.69 0) (effects (font (size 1 1)) (hide yes)))
-(property "FootprintStatus" "PENDING - no approved footprint" (at 85.09 59.69 0) (effects (font (size 1 1)) (hide yes)))
+(property "Design_note" "TI PWP0014A: EP15=GND; copper 3.4x5, mask 3.155x3.255; thermal vias and assembly pending" (at 85.09 59.69 0) (effects (font (size 1 1)) (hide yes)))
+(property "FootprintStatus" "DRAWING CHECKED - physical fit and PCB validation pending" (at 85.09 59.69 0) (effects (font (size 1 1)) (hide yes)))
 (pin "1")
 (pin "2")
@@
 (property "Reference" "L601" (at 45.72 113.74 0) (effects (font (size 1.15 1.15)) ))
 (property "Value" "22u" (at 45.72 125.02 0) (effects (font (size 0.98 0.98)) ))
-(property "Footprint" "" (at 45.72 119.38 0) (effects (font (size 1 1)) (hide yes)))
+(property "Footprint" "EU_Mechanical:L_Jantek_JNRH1207" (at 45.72 119.38 0) (effects (font (size 1 1)) (hide yes)))
 (property "Datasheet" "" (at 45.72 119.38 0) (effects (font (size 1 1)) (hide yes)))
 (property "MPN" "JNRH1207-220M-A" (at 45.72 119.38 0) (effects (font (size 1 1)) (hide yes)))
 (property "Design_note" "" (at 45.72 119.38 0) (effects (font (size 1 1)) (hide yes)))
-(property "FootprintStatus" "PENDING - no approved footprint" (at 45.72 119.38 0) (effects (font (size 1 1)) (hide yes)))
+(property "FootprintStatus" "DRAWING CHECKED - physical fit and PCB validation pending" (at 45.72 119.38 0) (effects (font (size 1 1)) (hide yes)))
 (pin "1")
 (pin "2")
@@
 (property "Reference" "J601" (at 374.65 173.43 0) (effects (font (size 1.15 1.15)) ))
 (property "Value" "LED2 + / GND" (at 374.65 187.25 0) (effects (font (size 0.98 0.98)) ))
-(property "Footprint" "" (at 374.65 180.34 0) (effects (font (size 1 1)) (hide yes)))
+(property "Footprint" "EU_Mechanical:TerminalBlock_Degson_DG306-5.0_1x02" (at 374.65 180.34 0) (effects (font (size 1 1)) (hide yes)))
 (property "Datasheet" "" (at 374.65 180.34 0) (effects (font (size 1 1)) (hide yes)))
 (property "MPN" "DG306-5.0-2P12" (at 374.65 180.34 0) (effects (font (size 1 1)) (hide yes)))
 (property "Design_note" "" (at 374.65 180.34 0) (effects (font (size 1 1)) (hide yes)))
-(property "FootprintStatus" "PENDING - no approved footprint" (at 374.65 180.34 0) (effects (font (size 1 1)) (hide yes)))
+(property "FootprintStatus" "DRAWING CHECKED - physical fit and PCB validation pending" (at 374.65 180.34 0) (effects (font (size 1 1)) (hide yes)))
 (pin "1")
 (pin "2")
@@
 (property "Reference" "J602" (at 45.72 192.48 0) (effects (font (size 1.15 1.15)) ))
 (property "Value" "BAR2 + / GND" (at 45.72 206.3 0) (effects (font (size 0.98 0.98)) ))
-(property "Footprint" "" (at 45.72 199.39 0) (effects (font (size 1 1)) (hide yes)))
+(property "Footprint" "EU_Mechanical:TerminalBlock_Degson_DG306-5.0_1x02" (at 45.72 199.39 0) (effects (font (size 1 1)) (hide yes)))
 (property "Datasheet" "" (at 45.72 199.39 0) (effects (font (size 1 1)) (hide yes)))
 (property "MPN" "DG306-5.0-2P12" (at 45.72 199.39 0) (effects (font (size 1 1)) (hide yes)))
 (property "Design_note" "" (at 45.72 199.39 0) (effects (font (size 1 1)) (hide yes)))
-(property "FootprintStatus" "PENDING - no approved footprint" (at 45.72 199.39 0) (effects (font (size 1 1)) (hide yes)))
-(pin "1")
-(pin "2")
+(property "FootprintStatus" "DRAWING CHECKED - physical fit and PCB validation pending" (at 45.72 199.39 0) (effects (font (size 1 1)) (hide yes)))
+(pin "1")
+(pin "2")
