File: hardware/PCB_EU/Loads.kicad_sch (KiCad schematic)
At the start: 15 parts, among them J701 PTC + / RETURN, J702 PUMP + / RETURN, Q701 BC847B-DIO, Q702 BC857B, Q703 IRF1010ESPBF, Q704 AO3422

Commit message: hardware: complete EU mechanical footprint assignments and validate pad maps
Parts:
- J701: footprint (none) -> EU_Mechanical:TerminalBlock_Degson_DG301R-5.0_1x02; FootprintStatus PENDING - no approved footprint -> DRAWING CHECKED - physical fit and PCB validation pending
- J702: footprint (none) -> EU_Mechanical:TerminalBlock_Degson_DG306-5.0_1x02; FootprintStatus PENDING - no approved footprint -> DRAWING CHECKED - physical fit and PCB validation pending
Changed lines of the file:
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@@
 (property "Reference" "J701" (at 45.72 98.5 0) (effects (font (size 1.15 1.15)) ))
 (property "Value" "PTC + / RETURN" (at 45.72 112.32 0) (effects (font (size 0.98 0.98)) ))
-(property "Footprint" "" (at 45.72 105.41 0) (effects (font (size 1 1)) (hide yes)))
+(property "Footprint" "EU_Mechanical:TerminalBlock_Degson_DG301R-5.0_1x02" (at 45.72 105.41 0) (effects (font (size 1 1)) (hide yes)))
 (property "Datasheet" "" (at 45.72 105.41 0) (effects (font (size 1 1)) (hide yes)))
 (property "MPN" "DG301R-5.0-2P12" (at 45.72 105.41 0) (effects (font (size 1 1)) (hide yes)))
 (property "Design_note" "" (at 45.72 105.41 0) (effects (font (size 1 1)) (hide yes)))
-(property "FootprintStatus" "PENDING - no approved footprint" (at 45.72 105.41 0) (effects (font (size 1 1)) (hide yes)))
+(property "FootprintStatus" "DRAWING CHECKED - physical fit and PCB validation pending" (at 45.72 105.41 0) (effects (font (size 1 1)) (hide yes)))
 (pin "1")
 (pin "2")
@@
 (property "Reference" "J702" (at 106.68 117.55 0) (effects (font (size 1.15 1.15)) ))
 (property "Value" "PUMP + / RETURN" (at 106.68 131.37 0) (effects (font (size 0.98 0.98)) ))
-(property "Footprint" "" (at 106.68 124.46 0) (effects (font (size 1 1)) (hide yes)))
+(property "Footprint" "EU_Mechanical:TerminalBlock_Degson_DG306-5.0_1x02" (at 106.68 124.46 0) (effects (font (size 1 1)) (hide yes)))
 (property "Datasheet" "" (at 106.68 124.46 0) (effects (font (size 1 1)) (hide yes)))
 (property "MPN" "DG306-5.0-2P12" (at 106.68 124.46 0) (effects (font (size 1 1)) (hide yes)))
 (property "Design_note" "" (at 106.68 124.46 0) (effects (font (size 1 1)) (hide yes)))
-(property "FootprintStatus" "PENDING - no approved footprint" (at 106.68 124.46 0) (effects (font (size 1 1)) (hide yes)))
+(property "FootprintStatus" "DRAWING CHECKED - physical fit and PCB validation pending" (at 106.68 124.46 0) (effects (font (size 1 1)) (hide yes)))
 (pin "1")
 (pin "2")
