File: hardware/PCB_EU/MCU.kicad_sch (KiCad schematic)
At the start: 17 parts, among them J201 UART 3V3, SW201 RESET, SW202 BOOT, U201 AP63203WU-7, U202 ESP32-WROOM-32E-N4

Commit message: hardware: complete EU mechanical footprint assignments and validate pad maps
Parts:
- L201: footprint (none) -> EU_Mechanical:L_Bourns_SRN6045; Design_note Bourns SRN6045, exact footprint dimensions to verify -> Bourns SRN6045 lands checked; not the TA variant; stability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; FootprintStatus PENDING - no approved footprint -> DRAWING CHECKED - physical fit and PCB validation pending
- SW201, SW202: footprint (none) -> EU_Mechanical:SW_Ninigi_TACTB-64K-F; FootprintStatus PENDING - no approved footprint -> DRAWING CHECKED - physical fit and PCB validation pending
Changed lines of the file:
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@@
 (property "Reference" "L201" (at 45.72 139.14 0) (effects (font (size 1.15 1.15)) ))
 (property "Value" "6u8" (at 45.72 150.42 0) (effects (font (size 0.98 0.98)) ))
-(property "Footprint" "" (at 45.72 144.78 0) (effects (font (size 1 1)) (hide yes)))
+(property "Footprint" "EU_Mechanical:L_Bourns_SRN6045" (at 45.72 144.78 0) (effects (font (size 1 1)) (hide yes)))
 (property "Datasheet" "" (at 45.72 144.78 0) (effects (font (size 1 1)) (hide yes)))
 (property "MPN" "SRN6045-6R8Y" (at 45.72 144.78 0) (effects (font (size 1 1)) (hide yes)))
-(property "Design_note" "Bourns SRN6045, exact footprint dimensions to verify" (at 45.72 144.78 0) (effects (font (size 1 1)) (hide yes)))
-(property "FootprintStatus" "PENDING - no approved footprint" (at 45.72 144.78 0) (effects (font (size 1 1)) (hide yes)))
+(property "Design_note" "Bourns SRN6045 lands checked; not the TA variant; stability remains prototype check" (at 45.72 144.78 0) (effects (font (size 1 1)) (hide yes)))
+(property "FootprintStatus" "DRAWING CHECKED - physical fit and PCB validation pending" (at 45.72 144.78 0) (effects (font (size 1 1)) (hide yes)))
 (pin "1")
 (pin "2")
@@
 (property "Reference" "SW201" (at 374.65 159.46 0) (effects (font (size 1.15 1.15)) ))
 (property "Value" "RESET" (at 374.65 170.74 0) (effects (font (size 0.98 0.98)) ))
-(property "Footprint" "" (at 374.65 165.1 0) (effects (font (size 1 1)) (hide yes)))
+(property "Footprint" "EU_Mechanical:SW_Ninigi_TACTB-64K-F" (at 374.65 165.1 0) (effects (font (size 1 1)) (hide yes)))
 (property "Datasheet" "" (at 374.65 165.1 0) (effects (font (size 1 1)) (hide yes)))
 (property "MPN" "TACTB-64K-F" (at 374.65 165.1 0) (effects (font (size 1 1)) (hide yes)))
 (property "Design_note" "4 physical button leads form two internally common pairs" (at 374.65 165.1 0) (effects (font (size 1 1)) (hide yes)))
-(property "FootprintStatus" "PENDING - no approved footprint" (at 374.65 165.1 0) (effects (font (size 1 1)) (hide yes)))
+(property "FootprintStatus" "DRAWING CHECKED - physical fit and PCB validation pending" (at 374.65 165.1 0) (effects (font (size 1 1)) (hide yes)))
 (pin "1")
 (pin "2")
@@
 (property "Reference" "SW202" (at 45.72 179.78 0) (effects (font (size 1.15 1.15)) ))
 (property "Value" "BOOT" (at 45.72 191.06 0) (effects (font (size 0.98 0.98)) ))
-(property "Footprint" "" (at 45.72 185.42 0) (effects (font (size 1 1)) (hide yes)))
+(property "Footprint" "EU_Mechanical:SW_Ninigi_TACTB-64K-F" (at 45.72 185.42 0) (effects (font (size 1 1)) (hide yes)))
 (property "Datasheet" "" (at 45.72 185.42 0) (effects (font (size 1 1)) (hide yes)))
 (property "MPN" "TACTB-64K-F" (at 45.72 185.42 0) (effects (font (size 1 1)) (hide yes)))
 (property "Design_note" "" (at 45.72 185.42 0) (effects (font (size 1 1)) (hide yes)))
-(property "FootprintStatus" "PENDING - no approved footprint" (at 45.72 185.42 0) (effects (font (size 1 1)) (hide yes)))
-(pin "1")
-(pin "2")
+(property "FootprintStatus" "DRAWING CHECKED - physical fit and PCB validation pending" (at 45.72 185.42 0) (effects (font (size 1 1)) (hide yes)))
+(pin "1")
+(pin "2")
