File: hardware/PCB_EU/MCU.kicad_sch (KiCad schematic)
At the start: 17 parts, among them J201 UART 3V3, SW201 RESET, SW202 BOOT, U201 AP63203WU-7, U202 ESP32-WROOM-32E-N4

Commit message: hardware: apply PCB_EU review fixes
- R702 100k -> 4k7: ESP32 internal pull-up on GPIO32 (old firmware
  INPUT_PULLUP) could switch the 100 W PTC on.
- C208 100n -> 1u for the Espressif EN delay.
- Remove TC4427A driver and its parts; each LM3429 GATE drives its own
  IRF540Z through 4R7 (driver was 20-25 mm from both MOSFETs).
- Add reverse-polarity protection: Q102 IRF1010ES in the input return
  with a 5k6+5k6 / 10k gate divider.
- F103 label: UST 1206 is time-lag.
- Rebuild PCB via build_board.py + route_power.py, rerun all checks on
  KiCad 10.0.7: ERC 0, DRC 0 / parity 0, 355 unrouted, 51 checks.
- Parts estimate 80.00 -> 78.59 EUR; check ceiling raised to 100 EUR.

Co-Authored-By: Claude Opus 5.5 (1M context) <noreply@anthropic.com>
Claude-Session: https://claude.ai/code/session_01AxccZX6Cb4FnRKJMrFYMSX
Parts:
- C208: value 100n RESET -> 1u RESET; MPN CL21B104KBCNNNC -> CL21B105KBFNNNG
Changed lines of the file:
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@@
 (symbol (lib_id "EU:C") (at 173.99 165.1 0) (unit 1) (in_bom yes) (on_board yes) (dnp no)
 (property "Reference" "C208" (at 173.99 159.46 0) (effects (font (size 1.15 1.15)) ))
-(property "Value" "100n RESET" (at 173.99 170.74 0) (effects (font (size 0.98 0.98)) ))
+(property "Value" "1u RESET" (at 173.99 170.74 0) (effects (font (size 0.98 0.98)) ))
 (property "Footprint" "Capacitor_SMD:C_0805_2012Metric" (at 173.99 165.1 0) (effects (font (size 1 1)) (hide yes)))
 (property "Datasheet" "" (at 173.99 165.1 0) (effects (font (size 1 1)) (hide yes)))
-(property "MPN" "CL21B104KBCNNNC" (at 173.99 165.1 0) (effects (font (size 1 1)) (hide yes)))
+(property "MPN" "CL21B105KBFNNNG" (at 173.99 165.1 0) (effects (font (size 1 1)) (hide yes)))
 (property "Design_note" "" (at 173.99 165.1 0) (effects (font (size 1 1)) (hide yes)))
 (property "FootprintStatus" "PACKAGE ONLY - verify before PCB" (at 173.99 165.1 0) (effects (font (size 1 1)) (hide yes)))
