File: hardware/PCB_EU/Peripherals.kicad_sch (KiCad schematic)
At the start: 18 parts, among them J301 MEM2061 SPI, U301 MCP7940N-I/SN, Y301 32.768k CL7p

Commit message: PCB_EU: C301/C302 KEMET C1206C100J5GACTU at Electrobase, one cooling set
C301/C302 (RTC crystal load, C0G needed): Salvats C1206C100J5GAC, whose
card heading says Y5V, -> KEMET C1206C100J5GACTU (C0G) at Electrobase,
2 x 0.25 instead of 2 x 0.10 EUR (+0.30; price and stock >1000 checked
2026-10-23). Second cooling set removed: RAD-DY-GF/3, TO220-SET and
SMICA-TO220-2 are bought once (-1.38 EUR).

BOM 85.75 -> 84.67 EUR: Electrobase 40.83, Salvats 37.97, shipping 5.87,
two parcels as before.

tools/generate.py rebuilds the schematic, design.json and the BOM (the
generator is idempotent). The MPN of C301/C302 is text-patched in
PCB_EU.kicad_pcb and review/netlist.xml the way a KiCad export and
build_board.py would write it; review/connectivity.txt comes from
tools/verify.py (56 checks pass). README.md and DESIGN.md are updated.

KiCad was not run: ERC, DRC, schematic parity and the other KiCad-based
checks of run_checks.py have NOT been run for this commit.

Co-Authored-By: Claude Sonnet 5.5 <noreply@anthropic.com>
Claude-Session: https://claude.ai/code/session_011GxPyRnAFpBjFQ5VURqV5H
Parts:
- C301, C302: MPN C1206C100J5GAC -> C1206C100J5GACTU
Changed lines of the file:
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@@
 (property "Footprint" "Capacitor_SMD:C_1206_3216Metric" (at 106.68 119.38 0) (effects (font (size 1 1)) (hide yes)))
 (property "Datasheet" "" (at 106.68 119.38 0) (effects (font (size 1 1)) (hide yes)))
-(property "MPN" "C1206C100J5GAC" (at 106.68 119.38 0) (effects (font (size 1 1)) (hide yes)))
+(property "MPN" "C1206C100J5GACTU" (at 106.68 119.38 0) (effects (font (size 1 1)) (hide yes)))
 (property "Design_note" "" (at 106.68 119.38 0) (effects (font (size 1 1)) (hide yes)))
 (property "FootprintStatus" "PACKAGE ONLY - verify before PCB" (at 106.68 119.38 0) (effects (font (size 1 1)) (hide yes)))
@@
 (property "Footprint" "Capacitor_SMD:C_1206_3216Metric" (at 173.99 119.38 0) (effects (font (size 1 1)) (hide yes)))
 (property "Datasheet" "" (at 173.99 119.38 0) (effects (font (size 1 1)) (hide yes)))
-(property "MPN" "C1206C100J5GAC" (at 173.99 119.38 0) (effects (font (size 1 1)) (hide yes)))
+(property "MPN" "C1206C100J5GACTU" (at 173.99 119.38 0) (effects (font (size 1 1)) (hide yes)))
 (property "Design_note" "" (at 173.99 119.38 0) (effects (font (size 1 1)) (hide yes)))
 (property "FootprintStatus" "PACKAGE ONLY - verify before PCB" (at 173.99 119.38 0) (effects (font (size 1 1)) (hide yes)))
